Commit message: added weights and inertia of ec swift sensors

File: urdf/livox_mid360.xacro (robot description, xacro)
@@ -1,4 +1,10 @@
 <?xml version="1.0"?>
 <robot xmlns:xacro="http://ros.org/wiki/xacro">
+	<!-- datasheet: https://terra-1-g.djicdn.com/851d20f7b9f64838a34cd02351370894/Livox/Livox_Mid-360_User_Manual_EN.pdf -->
+	<xacro:property name="livox_mid360_mass" value="0.265"/>
+	<xacro:property name="livox_mid360_length" value="0.065"/>
+	<xacro:property name="livox_mid360_width" value="0.073"/>
+	<xacro:property name="livox_mid360_height" value="0.061"/>
+	<xacro:include filename="$(find hector_xacro_tools)/urdf/inertia_tensors.urdf.xacro" />
 	<xacro:property name="M_PI" value="3.14159"/>
 	<xacro:macro name="livox_mid360" params="name:=default *origin *parent">
@@ -9,4 +15,5 @@
 		</joint>
 		<link name="livox_mid360_${name}_link">
+			<xacro:inertial_cuboid mass="${livox_mid360_mass}" x_length="${livox_mid360_length}" y_length="${livox_mid360_width}" z_length="${livox_mid360_height}"/>
 			<visual>
 				<origin xyz="0 0 0" rpy="0 0 0"/>
@@ -19,5 +26,5 @@
 				<origin xyz="0 0 0.012" rpy="0 0 0" />
 				<geometry>
-					<box size="0.065 0.073 0.061"/>
+					<box size="${livox_mid360_length} ${livox_mid360_width} ${livox_mid360_height}" />
 				</geometry>
 			</collision>

File: urdf/orbbec_astra2.xacro (robot description, xacro)
@@ -1,4 +1,10 @@
 <?xml version="1.0"?>
 <robot xmlns:xacro="http://ros.org/wiki/xacro">
+    <!-- datasheet: https://d1cd332k3pgc17.cloudfront.net/wp-content/uploads/2023/04/ORBBEC_Datasheet_Astra-2.pdf -->
+    <xacro:property name="orbbec_astra2_mass" value="0.195"/>
+    <xacro:property name="orbbec_astra2_length" value="0.037"/>
+    <xacro:property name="orbbec_astra2_width" value="0.147"/>
+    <xacro:property name="orbbec_astra2_height" value="0.035"/>
+    <xacro:include filename="$(find hector_xacro_tools)/urdf/inertia_tensors.urdf.xacro" />
     <xacro:property name="M_PI" value="3.14159"/>
     <xacro:macro name="orbbec_astra2" params="name:=default *origin *parent">
@@ -10,4 +16,5 @@
         <!-- Camera base -->
         <link name="astra2_${name}_base_link">
+            <xacro:inertial_cuboid mass="${orbbec_astra2_mass}" x_length="${orbbec_astra2_length}" y_length="${orbbec_astra2_width}" z_length="${orbbec_astra2_height}" />
             <visual>
                 <origin xyz="0 0 0" rpy="0 0 ${M_PI}" />
@@ -19,5 +26,5 @@
                 <origin xyz="0.018 0 0" rpy="0 0 0" />
                 <geometry>
-                    <box size="0.037 0.147 0.035"/>
+                    <box size="${orbbec_astra2_length} ${orbbec_astra2_width} ${orbbec_astra2_height}" />
                 </geometry>
             </collision>

File: urdf/seek_thermal_xr.xacro (robot description, xacro)
@@ -1,4 +1,10 @@
 <?xml version="1.0"?>
 <robot xmlns:xacro="http://ros.org/wiki/xacro">
+    <!-- datasheet: https://www.thermal.com/uploads/1/0/1/3/101388544/compactxr-sellsheet-usa_web.pdf -->
+    <xacro:property name="seek_thermal_xr_mass" value="0.014"/>
+    <xacro:property name="seek_thermal_xr_length" value="0.027"/>
+    <xacro:property name="seek_thermal_xr_width" value="0.04"/>
+    <xacro:property name="seek_thermal_xr_height" value="0.055"/>
+    <xacro:include filename="$(find hector_xacro_tools)/urdf/inertia_tensors.urdf.xacro" />
     <xacro:property name="M_PI" value="3.14159"/>
     <xacro:macro name="seek_thermal_xr" params="name:=default *origin *parent">
@@ -10,4 +16,5 @@
         <!-- Camera base -->
         <link name="seek_thermal_xr_${name}_base_link">
+            <xacro:inertial_cuboid mass="${seek_thermal_xr_mass}" x_length="${seek_thermal_xr_length}" y_length="${seek_thermal_xr_width}" z_length="${seek_thermal_xr_height}" />
             <visual>
                 <origin xyz="0 0 0" rpy="0 0 0" />
@@ -19,5 +26,5 @@
                 <origin xyz="0.013 0 -0.011" rpy="0 0 0" />
                 <geometry>
-                    <box size="0.027 0.04 0.055"/>
+                    <box size="${seek_thermal_xr_length} ${seek_thermal_xr_width} ${seek_thermal_xr_height}" />
                 </geometry>
             </collision>
