Commit message: corrected "hector_models" path to hector_sensors_description

File: urdf/astra_stereo_s_u3.xacro (robot description, xacro)
@@ -13,5 +13,5 @@
                 <origin xyz="0 0 0" rpy="0 0 0" />
                 <geometry>
-                    <mesh filename="package://hector_models/meshes/orbbec_astra_stereo_s_u3/orbbec_astra_stereo_s_u3.dae"/>
+                    <mesh filename="package://hector_sensors_description/meshes/orbbec_astra_stereo_s_u3/orbbec_astra_stereo_s_u3.dae"/>
                 </geometry>
             </visual>

File: urdf/livox_mid360.xacro (robot description, xacro)
@@ -12,5 +12,5 @@
 				<origin xyz="0 0 0" rpy="0 0 0"/>
 				<geometry>
-					<mesh filename="package://hector_models/meshes/livox_mid360/livox_mid360.dae">
+					<mesh filename="package://hector_sensors_description/meshes/livox_mid360/livox_mid360.dae">
 					</mesh>
 				</geometry>

File: urdf/orbbec_astra2.xacro (robot description, xacro)
@@ -13,5 +13,5 @@
                 <origin xyz="0 0 0" rpy="0 0 ${M_PI}" />
                 <geometry>
-                    <mesh filename="package://hector_models/meshes/orbbec_astra2/orbbec_astra2.dae"/>
+                    <mesh filename="package://hector_sensors_description/meshes/orbbec_astra2/orbbec_astra2.dae"/>
                 </geometry>
             </visual>

File: urdf/seek_thermal_xr.xacro (robot description, xacro)
@@ -13,5 +13,5 @@
                 <origin xyz="0 0 0" rpy="0 0 0" />
                 <geometry>
-                    <mesh filename="package://hector_models/meshes/seek_thermal_xr/seek_thermal_xr.dae"/>
+                    <mesh filename="package://hector_sensors_description/meshes/seek_thermal_xr/seek_thermal_xr.dae"/>
                 </geometry>
             </visual>

Commit message: corrected the frame names

File: urdf/astra_stereo_s_u3.xacro (robot description, xacro)
@@ -1,13 +1,20 @@
 <?xml version="1.0"?>
+<!-- datasheet: https://www.sodavision.com/wp-content/uploads/2023/12/2023.07-astra-stereo-s-u3-datasheet-_v2.0_en.pdf -->
 <robot xmlns:xacro="http://ros.org/wiki/xacro">
     <xacro:property name="M_PI" value="3.14159"/>
-    <xacro:macro name="orbbec_astra_stereo_s_u3" params="name:=default *origin *parent">
-        <joint name="astra_stereo_s_${name}_base_joint" type="fixed">
-            <child link="astra_stereo_s_${name}_base_link"/>
+    <xacro:property name="orbbec_astra_stereo_s_u3_mass" value="0.05"/> <!-- estimated, needs to be checked -->
+    <xacro:property name="orbbec_astra_stereo_s_u3_length" value="0.0653"/>
+    <xacro:property name="orbbec_astra_stereo_s_u3_width" value="0.0123"/>
+    <xacro:property name="orbbec_astra_stereo_s_u3_height" value="0.0225"/>
+    <xacro:include filename="$(find hector_xacro_tools)/urdf/inertia_tensors.urdf.xacro" />
+    <xacro:macro name="${name}" params="name:=default *origin *parent">
+        <joint name="${name}_joint" type="fixed">
+            <child link="${name}_link"/>
             <xacro:insert_block name="origin"/>
             <xacro:insert_block name="parent"/>
         </joint>
         <!-- Camera base -->
-        <link name="astra_stereo_s_${name}_base_link">
+        <link name="${name}_link">
+            <xacro:inertial_cuboid mass="${orbbec_astra2_mass}" x_length="${orbbec_astra2_length}" y_length="${orbbec_astra2_width}" z_length="${orbbec_astra2_height}" />
             <visual>
                 <origin xyz="0 0 0" rpy="0 0 0" />
@@ -24,9 +31,31 @@
         </link>
         <!-- Camera RGB sensor -->
-        <link name="astra_stereo_s_${name}_link"/>
-        <joint name="astra_stereo_s_${name}_sensor_joint" type="fixed">
+        <link name="${name}_rgb_link"/>
+        <joint name="${name}_rgb_joint" type="fixed">
             <origin xyz="0.014 0.01 0" rpy="0 0 0" />
-            <parent link="astra_stereo_s_${name}_base_link" />
-            <child link="astra_stereo_s_${name}_link" />
+            <parent link="${name}_link" />
+            <child link="${name}_rgb_link" />
+        </joint>
+        <!-- Camera Depth sensor -->
+        <!-- Assuming the depth image is published in the same frame as the rgb image -->
+        <link name="${name}_depth_link"/>
+        <joint name="${name}_depth_joint" type="fixed">
+            <origin xyz="0.014 0.01 0" rpy="0 0 0" />
+            <parent link="${name}_link" />
+            <child link="${name}_depth_link" />
+        </joint>
+        <!-- Camera Optical Frame -->
+        <link name="${name}_rgb_optical_frame"/>
+        <joint name="${name}_rgb_optical_joint" type="fixed">
+            <origin xyz="0 0 0" rpy="-${M_PI/2.0} 0 -${M_PI/2.0}" />
+            <parent link="${name}_rgb_link" />
+            <child link="${name}_rgb_optical_frame" />
+        </joint>
+        <!-- Camera Depth Optical Frame -->
+        <link name="${name}_depth_optical_frame"/>
+        <joint name="${name}_depth_optical_joint" type="fixed">
+            <origin xyz="0 0 0" rpy="-${M_PI/2.0} 0 -${M_PI/2.0}" />
+            <parent link="${name}_depth_link" />
+            <child link="${name}_depth_optical_frame" />
         </joint>
     </xacro:macro>

File: urdf/insta360_air.xacro (robot description, xacro)
@@ -2,16 +2,23 @@
 <robot xmlns:xacro="http://ros.org/wiki/xacro">
     <xacro:property name="M_PI" value="3.14159"/>
-    <xacro:macro name="insta360_air" params="name:=default *origin *parent">
-        <joint name="insta360_air_${name}_base_joint" type="fixed">
-            <child link="insta360_air_${name}_base_link"/>
+    <!-- TODO: check datasheet -->
+    <xacro:property name="insta360_air_mass" value="0.05"/>
+    <xacro:property name="insta360_air_length" value="0.021"/>
+    <xacro:property name="insta360_air_width" value="0.07"/>
+    <xacro:property name="insta360_air_height" value="0.025"/>
+    <xacro:include filename="$(find hector_xacro_tools)/urdf/inertia_tensors.urdf.xacro" />
+    <xacro:macro name="${name}" params="name:=default *origin *parent">
+        <joint name="${name}_joint" type="fixed">
+            <child link="${name}_link"/>
             <xacro:insert_block name="origin"/>
             <xacro:insert_block name="parent"/>
         </joint>
         <!-- Camera base -->
-        <link name="insta360_air_${name}_base_link">
+        <link name="${name}_link">
+            <xacro:inertial_cuboid mass="${insta360_air_mass}" x_length="${insta360_air_length}" y_length="${insta360_air_width}" z_length="${insta360_air_height}" />
             <visual>
                 <origin xyz="0 0 0" rpy="0 0 0" />
                 <geometry>
-                    <box size="0.021 0.07 0.025"/>
+                    <box size="${insta360_air_length} ${insta360_air_width} ${insta360_air_height}"/>
                 </geometry>
             </visual>
@@ -19,17 +26,17 @@
                 <origin xyz="0 0 0" rpy="0 0 0" />
                 <geometry>
-                    <box size="0.021 0.07 0.025"/>
+                    <box size="${insta360_air_length} ${insta360_air_width} ${insta360_air_height}"/>
                 </geometry>
             </collision>
         </link>
         <!-- Camera RGB sensor -->
-        <link name="insta360_air_${name}_left_optical_frame"/>
-        <joint name="insta360_air_${name}_left_optical_joint" type="fixed">
+        <link name="${name}_rgb_left"/>
+        <joint name="${name}_rgb_left_joint" type="fixed">
             <origin xyz="0 0 0" rpy="0 0 0" />
             <parent link="insta360_air_${name}_base_link" />
-            <child link="insta360_air_${name}_left_optical_frame" />
+            <child link="insta360_air_${name}_rgb_left" />
         </joint>
-        <link name="insta360_air_${name}_right_optical_frame"/>
-        <joint name="insta360_air_${name}_right_optical_joint" type="fixed">
+        <link name="${name}_right_optical_frame"/>
+        <joint name="${name}_right_optical_joint" type="fixed">
             <origin xyz="0 0 0" rpy="0 0 ${M_PI}" />
             <parent link="insta360_air_${name}_base_link" />

File: urdf/livox_mid360.xacro (robot description, xacro)
@@ -2,4 +2,5 @@
 <robot xmlns:xacro="http://ros.org/wiki/xacro">
 	<!-- datasheet: https://terra-1-g.djicdn.com/851d20f7b9f64838a34cd02351370894/Livox/Livox_Mid-360_User_Manual_EN.pdf -->
+	<xacro:property name="M_PI" value="3.14159"/>
 	<xacro:property name="livox_mid360_mass" value="0.265"/>
 	<xacro:property name="livox_mid360_length" value="0.065"/>
@@ -7,18 +8,16 @@
 	<xacro:property name="livox_mid360_height" value="0.061"/>
 	<xacro:include filename="$(find hector_xacro_tools)/urdf/inertia_tensors.urdf.xacro" />
-	<xacro:property name="M_PI" value="3.14159"/>
-	<xacro:macro name="livox_mid360" params="name:=default *origin *parent">
-		<joint name="livox_mid360_${name}_joint" type="fixed">
-			<child link="livox_mid360_${name}_link"/>
+	<xacro:macro name="${name}" params="name:=default *origin *parent">
+		<joint name="${name}_joint" type="fixed">
+			<child link="${name}_link"/>
 			<xacro:insert_block name="origin"/>
 			<xacro:insert_block name="parent"/>
 		</joint>
-		<link name="livox_mid360_${name}_link">
+		<link name="${name}_link">
 			<xacro:inertial_cuboid mass="${livox_mid360_mass}" x_length="${livox_mid360_length}" y_length="${livox_mid360_width}" z_length="${livox_mid360_height}"/>
 			<visual>
 				<origin xyz="0 0 0" rpy="0 0 0"/>
 				<geometry>
-					<mesh filename="package://hector_sensors_description/meshes/livox_mid360/livox_mid360.dae">
-					</mesh>
+					<mesh filename="package://hector_sensors_description/meshes/livox_mid360/livox_mid360.dae"/>
 				</geometry>
 			</visual>

File: urdf/orbbec_astra2.xacro (robot description, xacro)
@@ -2,4 +2,5 @@
 <robot xmlns:xacro="http://ros.org/wiki/xacro">
     <!-- datasheet: https://d1cd332k3pgc17.cloudfront.net/wp-content/uploads/2023/04/ORBBEC_Datasheet_Astra-2.pdf -->
+    <xacro:property name="M_PI" value="3.14159"/>
     <xacro:property name="orbbec_astra2_mass" value="0.195"/>
     <xacro:property name="orbbec_astra2_length" value="0.037"/>
@@ -7,13 +8,12 @@
     <xacro:property name="orbbec_astra2_height" value="0.035"/>
     <xacro:include filename="$(find hector_xacro_tools)/urdf/inertia_tensors.urdf.xacro" />
-    <xacro:property name="M_PI" value="3.14159"/>
-    <xacro:macro name="orbbec_astra2" params="name:=default *origin *parent">
-		<joint name="astra2_${name}_base_joint" type="fixed">
-			<child link="astra2_${name}_base_link"/>
-			<xacro:insert_block name="origin"/>
-			<xacro:insert_block name="parent"/>
-		</joint>
+    <xacro:macro name="${name}" params="name:=default *origin *parent">
+        <joint name="${name}_joint" type="fixed">
+            <child link="${name}_link"/>
+            <xacro:insert_block name="origin"/>
+            <xacro:insert_block name="parent"/>
+        </joint>
         <!-- Camera base -->
-        <link name="astra2_${name}_base_link">
+        <link name="${name}_link">
             <xacro:inertial_cuboid mass="${orbbec_astra2_mass}" x_length="${orbbec_astra2_length}" y_length="${orbbec_astra2_width}" z_length="${orbbec_astra2_height}" />
             <visual>
@@ -30,10 +30,10 @@
             </collision>
         </link>
-        <!-- Camera RGB sensor - Frame for gazebo (in x direction) -->
-        <link name="astra2_${name}_link"/>
-        <joint name="astra2_${name}_sensor_joint" type="fixed">
+        <!-- Camera RGB sensor -->
+        <link name="${name}_rgb_link"/>
+        <joint name="${name}_rgb_joint" type="fixed">
             <origin xyz="0.033 0.022 0" rpy="0 0 0" />
-            <parent link="astra2_${name}_base_link" />
-            <child link="astra2_${name}_link" />
+            <parent link="${name}_link" />
+            <child link="${name}_rgb_link" />
         </joint>
         <!-- Optical Frame for ros (in z direction) -->

File: urdf/seek_thermal_xr.xacro (robot description, xacro)
@@ -2,4 +2,5 @@
 <robot xmlns:xacro="http://ros.org/wiki/xacro">
     <!-- datasheet: https://www.thermal.com/uploads/1/0/1/3/101388544/compactxr-sellsheet-usa_web.pdf -->
+    <xacro:property name="M_PI" value="3.14159"/>
     <xacro:property name="seek_thermal_xr_mass" value="0.014"/>
     <xacro:property name="seek_thermal_xr_length" value="0.027"/>
@@ -7,13 +8,12 @@
     <xacro:property name="seek_thermal_xr_height" value="0.055"/>
     <xacro:include filename="$(find hector_xacro_tools)/urdf/inertia_tensors.urdf.xacro" />
-    <xacro:property name="M_PI" value="3.14159"/>
-    <xacro:macro name="seek_thermal_xr" params="name:=default *origin *parent">
-        <joint name="seek_thermal_xr_${name}_base_joint" type="fixed">
-            <child link="seek_thermal_xr_${name}_base_link"/>
+    <xacro:macro name="${name}" params="name:=default *origin *parent">
+        <joint name="${name}_joint" type="fixed">
+            <child link="${name}_link"/>
             <xacro:insert_block name="origin"/>
             <xacro:insert_block name="parent"/>
         </joint>
         <!-- Camera base -->
-        <link name="seek_thermal_xr_${name}_base_link">
+        <link name="${name}_link">
             <xacro:inertial_cuboid mass="${seek_thermal_xr_mass}" x_length="${seek_thermal_xr_length}" y_length="${seek_thermal_xr_width}" z_length="${seek_thermal_xr_height}" />
             <visual>
@@ -30,10 +30,10 @@
             </collision>
         </link>
-        <!-- Camera sensor -->
-        <link name="seek_thermal_xr_${name}_link"/>
-        <joint name="seek_thermal_xr_${name}_sensor_joint" type="fixed">
-            <origin xyz="0.025 0 0" rpy="0 0 0" />
-            <parent link="seek_thermal_xr_${name}_base_link" />
-            <child link="seek_thermal_xr_${name}_link" />
+        <!-- Camera optical frame -->
+        <link name="${name}_optical_frame"/>
+        <joint name="${name}_optical_joint" type="fixed">
+            <origin xyz="0.025 0 0" rpy="-${M_PI/2} 0 -${M_PI/2}" />
+            <parent link="${name}_link" />
+            <child link="${name}_optical_frame" />
         </joint>
     </xacro:macro>
