Commit message: corrected the frame names (#2)
* corrected the frame names

* integrated feedback and made naming consistent

* fixed lidar issue

---------

Co-authored-by: Markus Kramer <kramer@sim.tu-darmstadt.de>

File: urdf/generic_camera.urdf.xacro (robot description, xacro)
@@ -37,5 +37,3 @@
     </joint>
     <link name="${name}_optical_frame"/>
-    <xacro:generic_camera_gazebo name="${name}" update_rate="${update_rate}" res_x="${res_x}" res_y="${res_y}" hfov="${hfov}" image_format="${image_format}"/>
-  </xacro:macro>
 </robot>

Commit message: changed sensors to use arg robot_name and unified topics to be $(arg robot_name)/topic
Additionally added xacro.arg for the robot_name.

This allows to initialize the robots as standalone without providing a
robot_name (for default topics /topic) and to namespace them by
providing the arg robot_name, which is done in our robot urdfs anyways.

File: urdf/generic_camera.urdf.xacro (robot description, xacro)
@@ -37,3 +37,5 @@
     </joint>
     <link name="${name}_optical_frame"/>
+    <xacro:generic_camera_gazebo name="${name}" update_rate="${update_rate}" res_x="${res_x}" res_y="${res_y}" hfov="${hfov}" image_format="${image_format}"/>
+  </xacro:macro>
 </robot>

Commit message: adjusted urdf file

File: urdf/generic_camera.urdf.xacro (robot description, xacro)
@@ -3,5 +3,5 @@
   <xacro:include filename="$(find hector_sensors_description)/gazebo/generic_camera.gazebo.xacro"/>
   <xacro:property name="M_PI" value="3.1415926535897931" />
-  <xacro:macro name="generic_camera" params="name parent robot_name *origin ros_topic cam_info_topic update_rate res_x res_y image_format hfov">
+  <xacro:macro name="generic_camera" params="name parent robot_name *origin ros_topic cam_info_topic update_rate res_x res_y image_format hfov wide_angle=false">
     <joint name="${name}_joint" type="fixed">
       <xacro:insert_block name="origin" />
@@ -31,4 +31,5 @@
       </collision>-->
     </link>
+    <link name="${name}_optical_frame"/>
     <joint name="${name}_optical_joint" type="fixed">
       <origin xyz="0 0 0" rpy="${-M_PI/2} 0.0 ${-M_PI/2}" />
@@ -36,4 +37,5 @@
       <child link="${name}_optical_frame"/>
     </joint>
-    <link name="${name}_optical_frame"/>
+    <xacro:generic_camera_gazebo name="${name}" robot_name="${robot_name}" update_rate="${update_rate}" res_x="${res_x}" res_y="${res_y}" hfov="${hfov}" image_format="${image_format}" wide_angle="${wide_angle}"/>
+  </xacro:macro>
 </robot>
