Commit message: fixed frames of gemini2

File: urdf/orbbec_gemini2.urdf.xacro (robot description, xacro)
@@ -20,5 +20,5 @@
             <xacro:inertial_cuboid mass="${orbbec_gemini2_mass}" x_length="${orbbec_gemini2_length}" y_length="${orbbec_gemini2_width}" z_length="${orbbec_gemini2_height}" />
             <visual>
-                <origin xyz="0 0 0" rpy="${M_PI} 0 0" />
+                <origin xyz="0 0 0" rpy="0 0 0" />
                 <geometry>
                     <mesh filename="package://hector_sensors_description/meshes/orbbec_gemini2/orbbec_gemini2.stl"/>
@@ -36,5 +36,5 @@
         <link name="${name}_rgb_link"/>
         <joint name="${name}_rgb_joint" type="fixed">
-            <origin xyz="0.01682 0.010995 0.012505" rpy="0 0 0" />
+            <origin xyz="0.01682 0.010995 0" rpy="0 0 0" />
             <parent link="${name}_link" />
             <child link="${name}_rgb_link" />
@@ -44,10 +44,10 @@
         <joint name="${name}_rgb_optical_joint" type="fixed">
             <origin xyz="0 0 0" rpy="-${M_PI/2.0} 0 -${M_PI/2.0}" />
-            <parent link="${name}_link" />
+            <parent link="${name}_rgb_link" />
             <child link="${name}_rgb_optical_frame" />
         </joint>
         <link name="${name}_depth_link"/>
         <joint name="${name}_depth_joint" type="fixed">
-            <origin xyz="0.01491 0.025 0.0125" rpy="0 0 0" />
+            <origin xyz="0.01491 0.025 0" rpy="0 0 0" />
             <parent link="${name}_link" />
             <child link="${name}_depth_link" />
@@ -56,5 +56,5 @@
         <joint name="${name}_depth_optical_joint" type="fixed">
             <origin xyz="0 0 0" rpy="-${M_PI/2.0} 0 -${M_PI/2.0}" />
-            <parent link="${name}_link" />
+            <parent link="${name}_depth_link" />
             <child link="${name}_depth_optical_frame" />
         </joint>

Commit message: Optimized models for the d435, d455 and gemini2

File: urdf/orbbec_gemini2.urdf.xacro (robot description, xacro)
@@ -22,7 +22,6 @@
                 <origin xyz="0 0 0" rpy="0 0 0" />
                 <geometry>
-                    <mesh filename="package://hector_sensors_description/meshes/orbbec_gemini2/orbbec_gemini2.stl"/>
+                    <mesh filename="package://hector_sensors_description/meshes/orbbec_gemini2/orbbec_gemini2.dae"/>
                 </geometry>
-                <material name="black"/>
             </visual>
             <collision>

Commit message: fixed the collision for the orbbec gemini2

File: urdf/orbbec_gemini2.urdf.xacro (robot description, xacro)
@@ -26,5 +26,5 @@
             </visual>
             <collision>
-                <origin xyz="0.018 0 0" rpy="0 0 0" />
+                <origin xyz="0.0051 0 0" rpy="0 0 0" />
                 <geometry>
                     <box size="${orbbec_gemini2_length} ${orbbec_gemini2_width} ${orbbec_gemini2_height}" />
