Commit message: Port ec_scout sensors to gazebor harmonic. Move gazebo refs to dedicated files. Include proper robot namespacing in sensor topics

File: urdf/flir_a65_camera.urdf.xacro (robot description, xacro)
@@ -2,4 +2,5 @@
 <robot xmlns:xacro="http://www.ros.org/wiki/xacro">
   <xacro:include filename="$(find hector_xacro_tools)/urdf/sensor_macros.urdf.xacro" />
+  <xacro:include filename="$(find hector_sensors_description)/gazebo/flir_a65_camera.gazebo.xacro"/>
   <!--Dimensions taken from http://www.flir.com/automation/display/?id=56341-->
   <xacro:macro name="flir_a65_camera_model" params="name parent *origin">
@@ -29,33 +30,9 @@
     </gazebo>
   </xacro:macro>
-  <xacro:macro name="flir_a65_camera" params="name parent *origin">
+  <xacro:macro name="flir_a65_camera" params="name parent robot_name *origin">
     <xacro:flir_a65_camera_model name="${name}" parent="${parent}">
       <xacro:insert_block name="origin" />
     </xacro:flir_a65_camera_model>
-    <gazebo reference="${name}_frame">
-      <sensor type="camera" name="thermal_camera_sensor">
-        <update_rate>9</update_rate>
-        <camera>
-          <horizontal_fov>${45.0*pi/180.0}</horizontal_fov>
-          <image>
-            <format>R8G8B8</format>
-            <width>640</width>
-            <height>512</height>
-          </image>
-          <clip>
-            <near>0.01</near>
-            <far>10</far>
-          </clip>
-        </camera>
-        <plugin name="thermal_camera_controller" filename="libgazebo_ros_thermal_camera.so">
-          <alwaysOn>true</alwaysOn>
-          <updateRate>9</updateRate>
-          <cameraName>${name}</cameraName>
-          <imageTopicName>image_raw</imageTopicName>
-          <cameraInfoTopicName>camera_info</cameraInfoTopicName>
-          <frameName>${name}_optical_frame</frameName>
-        </plugin>
-      </sensor>
-    </gazebo>
+    <xacro:flir_a65_camera_gazebo robot_name="${robot_name}"/>
   </xacro:macro>
 </robot>

File: urdf/generic_camera.urdf.xacro (robot description, xacro)
@@ -1,6 +1,7 @@
 <?xml version="1.0"?>
 <robot xmlns:xacro="http://www.ros.org/wiki/xacro">
+  <xacro:include filename="$(find hector_sensors_description)/gazebo/generic_camera.gazebo.xacro"/>
   <xacro:property name="M_PI" value="3.1415926535897931" />
-  <xacro:macro name="generic_camera" params="name parent *origin ros_topic cam_info_topic update_rate res_x res_y image_format hfov">
+  <xacro:macro name="generic_camera" params="name parent robot_name *origin ros_topic cam_info_topic update_rate res_x res_y image_format hfov">
     <joint name="${name}_joint" type="fixed">
       <xacro:insert_block name="origin" />
@@ -36,27 +37,5 @@
     </joint>
     <link name="${name}_optical_frame"/>
-    <gazebo reference="${name}_link">
-      <sensor type="camera" name="${name}_camera_sensor">
-        <update_rate>${update_rate}</update_rate>
-        <camera>
-          <horizontal_fov>${hfov * M_PI/180.0}</horizontal_fov>
-          <image>
-            <format>${image_format}</format>
-            <width>${res_x}</width>
-            <height>${res_y}</height>
-          </image>
-          <clip>
-            <near>0.01</near>
-            <far>100</far>
-          </clip>
-        </camera>
-        <plugin name="${name}_camera_controller" filename="libgazebo_ros_camera.so">
-          <cameraName>${name}</cameraName>
-          <imageTopicName>${ros_topic}</imageTopicName>
-          <cameraInfoTopicName>${cam_info_topic}</cameraInfoTopicName>
-          <frameName>${name}_optical_frame</frameName>
-        </plugin>
-      </sensor>
-    </gazebo>
+    <xacro:generic_camera_gazebo name="${name}" robot_name="${robot_name}" update_rate="${update_rate}" res_x="${res_x}" res_y="${res_y}" hfov="${hfov}" image_format="${image_format}"/>
   </xacro:macro>
 </robot>

File: urdf/insta360_pro2.urdf.xacro (robot description, xacro)
@@ -1,9 +1,10 @@
 <?xml version="1.0"?>
 <robot xmlns:xacro="http://www.ros.org/wiki/xacro">
+  <xacro:include filename="$(find hector_sensors_description)/gazebo/insta360_pro2.gazebo.xacro"/>
   <xacro:property name="camera_frame_center_distance" value="0.06" />
   <material name="Grey">
     <color rgba="0.5 0.5 0.5 1" />
   </material>
-  <xacro:macro name="insta360_pro2" params="name parent *origin ros_topic update_rate res_x res_y image_format fov">
+  <xacro:macro name="insta360_pro2" params="name parent robot_name *origin ros_topic update_rate res_x res_y image_format fov">
     <joint name="${name}_center_joint" type="fixed">
       <xacro:insert_block name="origin" />
@@ -52,5 +53,5 @@
     </xacro:insta360_pro2_camera>
   </xacro:macro>
-  <xacro:macro name="insta360_pro2_with_calibration" params="name parent *origin *calibration1 *calibration2 *calibration3 *calibration4 *calibration5 *calibration6 ros_topic update_rate res_x res_y image_format fov">
+  <xacro:macro name="insta360_pro2_with_calibration" params="name parent robot_name *origin *calibration1 *calibration2 *calibration3 *calibration4 *calibration5 *calibration6 ros_topic update_rate res_x res_y image_format fov">
     <joint name="${name}_center_joint" type="fixed">
       <xacro:insert_block name="origin" />
@@ -80,24 +81,24 @@
       </collision>
     </link>
-    <xacro:insta360_pro2_camera parent="${name}_origin2_optical_frame" camera_number="1" ros_topic="${ros_topic}" update_rate="${update_rate}" res_x="${res_x}" res_y="${res_y}" image_format="${image_format}" fov="${fov}">
+    <xacro:insta360_pro2_camera parent="${name}_origin2_optical_frame" robot_name="${robot_name}" camera_number="1" ros_topic="${ros_topic}" update_rate="${update_rate}" res_x="${res_x}" res_y="${res_y}" image_format="${image_format}" fov="${fov}">
       <xacro:insert_block name="calibration1" />
     </xacro:insta360_pro2_camera>
-    <xacro:insta360_pro2_camera parent="${name}_origin3_optical_frame" camera_number="2" ros_topic="${ros_topic}" update_rate="${update_rate}" res_x="${res_x}" res_y="${res_y}" image_format="${image_format}" fov="${fov}">
+    <xacro:insta360_pro2_camera parent="${name}_origin3_optical_frame" robot_name="${robot_name}" camera_number="2" ros_topic="${ros_topic}" update_rate="${update_rate}" res_x="${res_x}" res_y="${res_y}" image_format="${image_format}" fov="${fov}">
       <xacro:insert_block name="calibration2" />
     </xacro:insta360_pro2_camera>
-    <xacro:insta360_pro2_camera parent="${name}_origin4_optical_frame" camera_number="3" ros_topic="${ros_topic}" update_rate="${update_rate}" res_x="${res_x}" res_y="${res_y}" image_format="${image_format}" fov="${fov}">
+    <xacro:insta360_pro2_camera parent="${name}_origin4_optical_frame" robot_name="${robot_name}" camera_number="3" ros_topic="${ros_topic}" update_rate="${update_rate}" res_x="${res_x}" res_y="${res_y}" image_format="${image_format}" fov="${fov}">
       <xacro:insert_block name="calibration3" />
     </xacro:insta360_pro2_camera>
-    <xacro:insta360_pro2_camera parent="${name}_origin5_optical_frame" camera_number="4" ros_topic="${ros_topic}" update_rate="${update_rate}" res_x="${res_x}" res_y="${res_y}" image_format="${image_format}" fov="${fov}">
+    <xacro:insta360_pro2_camera parent="${name}_origin5_optical_frame" robot_name="${robot_name}" camera_number="4" ros_topic="${ros_topic}" update_rate="${update_rate}" res_x="${res_x}" res_y="${res_y}" image_format="${image_format}" fov="${fov}">
       <xacro:insert_block name="calibration4" />
     </xacro:insta360_pro2_camera>
-    <xacro:insta360_pro2_camera parent="${name}_origin6_optical_frame" camera_number="5" ros_topic="${ros_topic}" update_rate="${update_rate}" res_x="${res_x}" res_y="${res_y}" image_format="${image_format}" fov="${fov}">
+    <xacro:insta360_pro2_camera parent="${name}_origin6_optical_frame" robot_name="${robot_name}" camera_number="5" ros_topic="${ros_topic}" update_rate="${update_rate}" res_x="${res_x}" res_y="${res_y}" image_format="${image_format}" fov="${fov}">
       <xacro:insert_block name="calibration5" />
     </xacro:insta360_pro2_camera>
-    <xacro:insta360_pro2_camera parent="${name}_center_link" camera_number="6" ros_topic="${ros_topic}" update_rate="${update_rate}" res_x="${res_x}" res_y="${res_y}" image_format="${image_format}" fov="${fov}">
+    <xacro:insta360_pro2_camera parent="${name}_center_link" robot_name="${robot_name}" camera_number="6" ros_topic="${ros_topic}" update_rate="${update_rate}" res_x="${res_x}" res_y="${res_y}" image_format="${image_format}" fov="${fov}">
       <xacro:insert_block name="calibration6" />
     </xacro:insta360_pro2_camera>
   </xacro:macro>
-  <xacro:macro name="insta360_pro2_camera" params="camera_number parent *calibration ros_topic update_rate res_x res_y image_format fov">
+  <xacro:macro name="insta360_pro2_camera" params="camera_number robot_name parent *calibration ros_topic update_rate res_x res_y image_format fov">
     <xacro:property name="camera_name" value="${name}_origin${camera_number}" />
     <joint name="${camera_name}_optical_joint" type="fixed">
@@ -113,34 +114,5 @@
     <link name="${camera_name}_link" />
     <link name="${camera_name}_optical_frame" />
-    <gazebo reference="${camera_name}_link">
-      <sensor type="wideanglecamera" name="${camera_name}_camera_sensor">
-        <update_rate>${update_rate}</update_rate>
-        <camera>
-          <!--<horizontal_fov>${hfov * pi/180.0}</horizontal_fov>-->
-          <horizontal_fov>${fov}</horizontal_fov>
-          <image>
-            <format>${image_format}</format>
-            <width>${res_x}</width>
-            <height>${res_y}</height>
-          </image>
-          <clip>
-            <near>0.01</near>
-            <far>100</far>
-          </clip>
-          <lens>
-            <type>stereographic</type>
-            <scale_to_hfov>true</scale_to_hfov>
-            <cutoff_angle>1.5707</cutoff_angle>
-            <env_texture_size>512</env_texture_size>
-          </lens>
-        </camera>
-        <plugin name="${camera_name}_camera_controller" filename="libgazebo_ros_camera.so">
-          <cameraName>${name}/origin${camera_number}</cameraName>
-          <imageTopicName>${ros_topic}</imageTopicName>
-          <cameraInfoTopicName>not_used</cameraInfoTopicName>
-          <frameName>${camera_name}_optical_frame</frameName>
-        </plugin>
-      </sensor>
-    </gazebo>
+    <xacro:insta360_pro2_gazebo camera_name="${camera_name}" robot_name="${robot_name}" ros_topic="${ros_topic}" update_rate="${update_rate}" fov="${fov}" image_format="${image_format}" res_x="${res_x}" res_y="${res_y}" />
   </xacro:macro>
 </robot>

File: urdf/realsense_d435_camera.urdf.xacro (robot description, xacro)
@@ -18,4 +18,5 @@
   <xacro:property name="realsense_d435_case_offset_y" value="-0.0175"/> <!-- mounting hole to depth frame, Intel_RealSense_D400_Family_Datasheet_Jan2019.pdf, page 66 -->
   <xacro:property name="realsense_d435_case_offset_z" value="0.0"/>
+  <xacro:include filename="$(find hector_sensors_description)/gazebo/realsense_d435_camera.gazebo.xacro"/>
     <!--
      This macro only adds the model, it does not also add the openni gazebo plugin.
@@ -73,35 +74,6 @@
       </link>
     </xacro:macro>
-    <xacro:macro name="realsense_d435_camera_gazebo_plugin_macro" params="name parent image_topic depth_topic:=image_raw depth_points_topic frame_name:=color min_range max_range update_rate">
-      <gazebo reference="${name}_link">
-        <sensor type="depth" name="${name}">
-          <update_rate>${update_rate}</update_rate>
-          <camera>
-            <horizontal_fov>${69.4 * M_PI/180.0}</horizontal_fov>
-            <image>
-              <format>B8G8R8</format>
-              <width>640</width>
-              <height>480</height>
-            </image>
-            <clip>
-              <near>${min_range}</near>
-              <far>${max_range}</far>
-            </clip>
-          </camera>
-          <plugin name="${name}_camera_controller" filename="libgazebo_ros_openni_kinect.so">
-            <cameraName>${name}</cameraName>
-            <imageTopicName>color/${image_topic}</imageTopicName>
-            <cameraInfoTopicName>color/camera_info</cameraInfoTopicName>
-            <depthImageTopicName>depth/${depth_topic}</depthImageTopicName>
-            <depthImageCameraInfoTopicName>depth/camera_info</depthImageCameraInfoTopicName>
-            <pointCloudTopicName>${depth_points_topic}</pointCloudTopicName>
-            <frameName>${name}_${frame_name}_optical_frame</frameName>
-            <!-- Important information about frames: Currently, this plugin only supports simulation of color image and depth image/cloud from a single frame.
-            This frame is given in the <gazebo reference=""> tag above and is set to the ${name}_link which coincides with the depth camera frame. The camera axis is the X-axis. ROS requires an optical frame
-            with the Z-axis as camera axis. It is advised to use the depth_optical_frame for this purpose (frame_name="depth"), even though camera images will have the same frame.
-            The color_optical_frame does not coincide with the depth_optical_frame, so depth image/cloud will be misaligned! -->
-          </plugin>
-        </sensor>
-      </gazebo>
+    <xacro:macro name="realsense_d435_camera_gazebo_plugin_macro" params="name robot_name parent frame_name:=color min_range max_range update_rate">
+      <xacro:realsense_d435_camera_gazebo name="${name}" robot_name="${robot_name}" parent="${parent}" frame_name="color" min_range="${min_range}" max_range="${max_range}" update_rate="${update_rate}"/>
     </xacro:macro>
     <!--
@@ -109,18 +81,18 @@
       The origin is the left infrared (depth) camera, which is also the origin of the depth image
     -->
-    <xacro:macro name="realsense_d435_camera" params="name parent *origin">
+    <xacro:macro name="realsense_d435_camera" params="name robot_name parent *origin">
       <xacro:realsense_d435_camera_model name="${name}" parent="${parent}">
         <xacro:insert_block name="origin" />
       </xacro:realsense_d435_camera_model>
-      <xacro:realsense_d435_camera_gazebo_plugin_macro name="${name}" parent="${parent}" image_topic="image_raw" depth_points_topic="depth/points" min_range="0.3" max_range="9.0" update_rate="20"/>
+      <xacro:realsense_d435_camera_gazebo_plugin_macro name="${name}" robot_name="${robot_name}" parent="${parent}" min_range="0.3" max_range="9.0" update_rate="20"/>
     </xacro:macro>
     <!--
       Insert the realsense with link geometry. Origin is the mounting hole at the back of the camera.
     -->
-    <xacro:macro name="realsense_d435_camera_with_mount" params="name parent *origin">
+    <xacro:macro name="realsense_d435_camera_with_mount" params="name robot_name parent *origin">
       <xacro:realsense_d435_camera_model_with_mount name="${name}" parent="${parent}">
         <xacro:insert_block name="origin" />
       </xacro:realsense_d435_camera_model_with_mount>
-      <xacro:realsense_d435_camera_gazebo_plugin_macro name="${name}" parent="${parent}" image_topic="image_raw" depth_points_topic="depth/points" min_range="0.3" max_range="9.0" update_rate="20"/>
+      <xacro:realsense_d435_camera_gazebo_plugin_macro name="${name}" robot_name="${robot_name}" parent="${parent}" min_range="0.3" max_range="9.0" update_rate="20"/>
     </xacro:macro>
     <!--
@@ -128,27 +100,27 @@
       e.g. if the sensor is added into preexisting geometry
     -->
-    <xacro:macro name="realsense_camera_no_geom" params="name parent *origin">
+    <xacro:macro name="realsense_camera_no_geom" params="name robot_name parent *origin">
       <xacro:realsense_d435_camera_model_no_geom name="${name}" parent="${parent}">
         <xacro:insert_block name="origin" />
       </xacro:realsense_d435_camera_model_no_geom>
-      <xacro:realsense_camera_gazebo_plugin_macro name="${name}" parent="${parent}" image_topic="image_raw" depth_points_topic="depth/points" min_range="0.3" max_range="9.0" update_rate="20"/>
+      <xacro:realsense_camera_gazebo_plugin_macro name="${name}" robot_name="${robot_name}" parent="${parent}" min_range="0.3" max_range="9.0" update_rate="20"/>
     </xacro:macro>
-    <xacro:macro name="realsense_d435_camera_no_geom_comprehensive_params" params="name parent *origin image_topic depth_topic:=image_raw depth_points_topic frame_name:=color min_range max_range update_rate">
+    <xacro:macro name="realsense_d435_camera_no_geom_comprehensive_params" params="name robot_name parent *origin frame_name:=color min_range max_range update_rate">
       <xacro:realsense_d435_camera_model_no_geom name="${name}" parent="${parent}">
         <xacro:insert_block name="origin" />
       </xacro:realsense_d435_camera_model_no_geom>
-      <xacro:realsense_camera_gazebo_plugin_macro name="${name}" parent="${parent}" image_topic="${image_topic}" depth_topic="${depth_topic}" depth_points_topic="${depth_points_topic}" frame_name="${frame_name}" min_range="${min_range}" max_range="${max_range}" update_rate="${update_rate}"/>
+      <xacro:realsense_camera_gazebo_plugin_macro name="${name}" robot_name="${robot_name}" parent="${parent}" image_topic="${image_topic}" depth_topic="${depth_topic}" depth_points_topic="${depth_points_topic}" frame_name="${frame_name}" min_range="${min_range}" max_range="${max_range}" update_rate="${update_rate}"/>
     </xacro:macro>
-    <xacro:macro name="realsense_d435_camera_comprehensive_params" params="name parent *origin image_topic:=image_raw depth_topic:=image_raw depth_points_topic:=depth/color/points frame_name:=color min_range:=0.3 max_range:=9.0 update_rate:=20">
+    <xacro:macro name="realsense_d435_camera_comprehensive_params" params="name robot_name parent *origin frame_name:=color min_range:=0.3 max_range:=9.0 update_rate:=20">
       <xacro:realsense_d435_camera_model name="${name}" parent="${parent}">
         <xacro:insert_block name="origin" />
       </xacro:realsense_d435_camera_model>
-      <xacro:realsense_d435_camera_gazebo_plugin_macro name="${name}" parent="${parent}" image_topic="${image_topic}" depth_topic="${depth_topic}" depth_points_topic="${depth_points_topic}" frame_name="${frame_name}" min_range="${min_range}" max_range="${max_range}" update_rate="${update_rate}"/>
+      <xacro:realsense_d435_camera_gazebo_plugin_macro name="${name}" robot_name="${robot_name}" parent="${parent}" frame_name="${frame_name}" min_range="${min_range}" max_range="${max_range}" update_rate="${update_rate}"/>
     </xacro:macro>
-    <xacro:macro name="realsense_d435_camera_with_mount_comprehensive_params" params="name parent *origin image_topic:=image_raw depth_topic:=image_raw depth_points_topic:=depth/color/points frame_name:=color min_range:=0.3 max_range:=9.0 update_rate:=20">
+    <xacro:macro name="realsense_d435_camera_with_mount_comprehensive_params" params="name robot_name parent *origin frame_name:=color min_range:=0.3 max_range:=9.0 update_rate:=20">
       <xacro:realsense_d435_camera_model_with_mount name="${name}" parent="${parent}">
         <xacro:insert_block name="origin" />
       </xacro:realsense_d435_camera_model_with_mount>
-      <xacro:realsense_d435_camera_gazebo_plugin_macro name="${name}" parent="${parent}" image_topic="${image_topic}" depth_topic="${depth_topic}" depth_points_topic="${depth_points_topic}" frame_name="${frame_name}" min_range="${min_range}" max_range="${max_range}" update_rate="${update_rate}"/>
+      <xacro:realsense_d435_camera_gazebo_plugin_macro name="${name}" robot_name="${robot_name}" parent="${parent}" frame_name="${frame_name}" min_range="${min_range}" max_range="${max_range}" update_rate="${update_rate}"/>
     </xacro:macro>
   </robot>

File: urdf/tis_zoom_cam.urdf.xacro (robot description, xacro)
@@ -35,9 +35,9 @@
     </gazebo>
   </xacro:macro>
-  <xacro:macro name="tis_zoom_camera" params="name parent *origin">
+  <xacro:macro name="tis_zoom_camera" params="name robot_name parent *origin">
     <xacro:tis_zoom_camera_model name="${name}" parent="${parent}">
       <xacro:insert_block name="origin" />
     </xacro:tis_zoom_camera_model>
-    <xacro:generic_camera name="${name}" parent="${name}_housing_frame" ros_topic="image_raw" cam_info_topic="camera_info" update_rate="5" res_x="1920" res_y="1080" image_format="R8G8B8" hfov="70">
+    <xacro:generic_camera name="${name}" robot_name="${robot_name}" parent="${name}_housing_frame" ros_topic="image_raw" cam_info_topic="camera_info" update_rate="5" res_x="1920" res_y="1080" image_format="R8G8B8" hfov="70">
       <origin xyz="0 0 0" rpy="0 0 0"/>
     </xacro:generic_camera>
