Commit message: Added models for the scout's head mounted cameras

File: urdf/flir_a65_camera.urdf.xacro (robot description, xacro)
@@ -13,13 +13,13 @@
       <xacro:inertial_sphere mass="0.21" diameter="0.07" />
       <visual>
-        <origin xyz="${0.1041*-0.5} 0 0" rpy="0 0 0" />
+        <origin xyz="0 0 0" rpy="0 0 0" />
         <geometry>
-          <box size="0.1041 0.0496 0.0466" />
+          <mesh filename="package://hector_sensors_description/meshes/flir_ax5_camera/flir_ax5_housing.glb" />
         </geometry>
       </visual>
       <collision>
-        <origin xyz="${0.1041*-0.5} 0 0" rpy="0 0 0" />
+        <origin xyz="-0.05205 0 -0.0015" rpy="0 0 0" />
         <geometry>
-          <box size="0.1041 0.0496 0.0466" />
+          <box size="0.1041 0.04 0.043" />
         </geometry>
       </collision>

File: urdf/insta360_pro2.urdf.xacro (robot description, xacro)
@@ -16,7 +16,6 @@
       <visual>
         <geometry>
-          <mesh filename="package://hector_sensors_description/meshes/insta360_pro2/insta_pro2.stl" scale="0.001 0.001 0.001" />
+          <mesh filename="package://hector_sensors_description/meshes/insta360_pro2/insta_pro2.glb" />
         </geometry>
-        <material name="Grey" />
       </visual>
       <collision>
@@ -63,7 +62,6 @@
       <visual>
         <geometry>
-          <mesh filename="package://hector_sensors_description/meshes/insta360_pro2/insta_pro2.stl" scale="0.001 0.001 0.001" />
+          <mesh filename="package://hector_sensors_description/meshes/insta360_pro2/insta_pro2.glb" />
         </geometry>
-        <material name="Grey" />
       </visual>
       <collision>

File: urdf/tis_zoom_cam.urdf.xacro (robot description, xacro)
@@ -5,7 +5,7 @@
   <xacro:include filename="$(find hector_sensors_description)/urdf/generic_camera.urdf.xacro" />
   <!-- Dimensions from https://s1-dl.theimagingsource.com/api/2.5/packages/documentation/factsheets-single/fsdfkz30gp031/5e87e13f-c891-50c8-93c1-7bffd94642a1/fsdfkz30gp031.de_DE.pdf -->
-  <xacro:property name="tis_zoom_cam_housing_width" value="0.0606" />
-  <xacro:property name="tis_zoom_cam_housing_height" value="0.0606" />
-  <xacro:property name="tis_zoom_cam_housing_length" value="0.117" />
+  <xacro:property name="tis_zoom_cam_housing_width" value="0.0706" />
+  <xacro:property name="tis_zoom_cam_housing_height" value="0.0706" />
+  <xacro:property name="tis_zoom_cam_housing_length" value="0.146" />
   <xacro:macro name="tis_zoom_camera_model" params="name parent *origin">
     <joint name="${name}_mount_joint" type="fixed">
@@ -15,16 +15,20 @@
     </joint>
     <link name="${name}_housing_frame">
-      <xacro:inertial_cuboid mass="0.02" x_length="0.0285" y_length="0.07" z_length="0.034"/>
+      <xacro:inertial_cuboid_with_pose
+        mass="0.02"
+        x_length="0.0285"
+        y_length="0.07"
+        z_length="0.034" >
+        <origin xyz="-0.073 0 0" rpy="0 0 0" />
+      </xacro:inertial_cuboid_with_pose>
       <visual>
         <geometry>
-          <mesh filename="package://hector_sensors_description/meshes/tis_zoom_cam/zoom_cam_housing.stl" scale="1.0 1.0 1.0"/>
+          <mesh filename="package://hector_sensors_description/meshes/tis_zoom_cam/tis_zoom_cam.glb" />
         </geometry>
-        <material name="DarkGrey">
-          <color rgba="0.3 0.3 0.3 1"/>
-        </material>
       </visual>
       <collision>
+        <origin xyz="-0.073 0 0" rpy="0 0 0" />
         <geometry>
-          <box size="${tis_zoom_cam_housing_length} ${tis_zoom_cam_housing_width} ${tis_zoom_cam_housing_height}" />
+          <box size="0.146 0.0706 0.0706" />
         </geometry>
       </collision>
@@ -40,5 +44,5 @@
     </xacro:tis_zoom_camera_model>
     <xacro:generic_camera name="${name}" robot_name="${robot_name}" parent="${name}_housing_frame" ros_topic="image_raw" cam_info_topic="camera_info" update_rate="5" res_x="1920" res_y="1080" image_format="R8G8B8" hfov="70">
-      <origin xyz="0.04 0.0 0.0" rpy="0 0 0"/>
+      <origin xyz="0 0 0" rpy="0 0 0"/>
     </xacro:generic_camera>
   </xacro:macro>

Commit message: Updated model for ouster os0_128

File: urdf/flir_a65_camera.urdf.xacro (robot description, xacro)
@@ -15,5 +15,5 @@
         <origin xyz="0 0 0" rpy="0 0 0" />
         <geometry>
-          <mesh filename="package://hector_sensors_description/meshes/flir_ax5_camera/flir_ax5_housing.glb" />
+          <mesh filename="package://hector_sensors_description/meshes/flir_ax5_camera/flir_ax5_camera.glb" />
         </geometry>
       </visual>

File: urdf/os0_128.urdf.xacro (robot description, xacro)
@@ -12,13 +12,6 @@
             <xacro:inertial_sphere mass="0.992" diameter="0.08082"/>
             <visual>
-                <origin xyz="0 0 -0.062825" rpy="0 0 0" />
                 <geometry>
-                    <mesh filename="package://hector_sensors_description/meshes/ouster_os0/os0_baseplate.dae" scale="0.001 0.001 0.001"/>
-                </geometry>
-            </visual>
-            <visual>
-                <origin xyz="0 0 -0.040825" rpy="0 0 0" />
-                <geometry>
-                    <mesh filename="package://hector_sensors_description/meshes/ouster_os0/os0.dae" scale="0.001 0.001 0.001"/>
+                    <mesh filename="package://hector_sensors_description/meshes/os0_128/os0_128.glb" />
                 </geometry>
             </visual>

File: urdf/tis_zoom_cam.urdf.xacro (robot description, xacro)
@@ -4,8 +4,4 @@
   <xacro:include filename="$(find hector_xacro_tools)/urdf/inertia_tensors.urdf.xacro" />
   <xacro:include filename="$(find hector_sensors_description)/urdf/generic_camera.urdf.xacro" />
-  <!-- Dimensions from https://s1-dl.theimagingsource.com/api/2.5/packages/documentation/factsheets-single/fsdfkz30gp031/5e87e13f-c891-50c8-93c1-7bffd94642a1/fsdfkz30gp031.de_DE.pdf -->
-  <xacro:property name="tis_zoom_cam_housing_width" value="0.0706" />
-  <xacro:property name="tis_zoom_cam_housing_height" value="0.0706" />
-  <xacro:property name="tis_zoom_cam_housing_length" value="0.146" />
   <xacro:macro name="tis_zoom_camera_model" params="name parent *origin">
     <joint name="${name}_mount_joint" type="fixed">
