Commit message: integrated feedback and made naming consistent

File: urdf/astra_stereo_s_u3.urdf.xacro (robot description, xacro)
@@ -3,10 +3,10 @@
 <robot xmlns:xacro="http://ros.org/wiki/xacro">
     <xacro:property name="M_PI" value="3.14159"/>
-    <xacro:property name="orbbec_astra_stereo_s_u3_mass" value="0.05"/> <!-- estimated, needs to be checked -->
-    <xacro:property name="orbbec_astra_stereo_s_u3_length" value="0.0653"/>
-    <xacro:property name="orbbec_astra_stereo_s_u3_width" value="0.0123"/>
-    <xacro:property name="orbbec_astra_stereo_s_u3_height" value="0.0225"/>
     <xacro:include filename="$(find hector_xacro_tools)/urdf/inertia_tensors.urdf.xacro" />
-    <xacro:macro name="${name}" params="name:=default *origin *parent">
+    <xacro:macro name="orbbec_astra_stereo_s_u3" params="name *origin *parent">
+        <xacro:property name="orbbec_astra_stereo_s_u3_mass" value="0.05"/> <!-- estimated, needs to be checked -->
+        <xacro:property name="orbbec_astra_stereo_s_u3_length" value="0.0653"/>
+        <xacro:property name="orbbec_astra_stereo_s_u3_width" value="0.0123"/>
+        <xacro:property name="orbbec_astra_stereo_s_u3_height" value="0.0225"/>
         <joint name="${name}_joint" type="fixed">
             <child link="${name}_link"/>
@@ -16,5 +16,5 @@
         <!-- Camera base -->
         <link name="${name}_link">
-            <xacro:inertial_cuboid mass="${orbbec_astra2_mass}" x_length="${orbbec_astra2_length}" y_length="${orbbec_astra2_width}" z_length="${orbbec_astra2_height}" />
+            <xacro:inertial_cuboid mass="${orbbec_astra_stereo_s_u3_mass}" x_length="${orbbec_astra_stereo_s_u3_length}" y_length="${orbbec_astra_stereo_s_u3_width}" z_length="${orbbec_astra_stereo_s_u3_height}" />
             <visual>
                 <origin xyz="0 0 0" rpy="0 0 0" />

File: urdf/generic_camera.urdf.xacro (robot description, xacro)
@@ -37,5 +37,3 @@
     </joint>
     <link name="${name}_optical_frame"/>
-    <xacro:generic_camera_gazebo name="${name}" robot_name="${robot_name}" update_rate="${update_rate}" res_x="${res_x}" res_y="${res_y}" hfov="${hfov}" image_format="${image_format}"/>
-  </xacro:macro>
 </robot>

File: urdf/insta360_air.urdf.xacro (robot description, xacro)
@@ -2,11 +2,11 @@
 <robot xmlns:xacro="http://ros.org/wiki/xacro">
     <xacro:property name="M_PI" value="3.14159"/>
-    <!-- TODO: check datasheet -->
-    <xacro:property name="insta360_air_mass" value="0.05"/>
+    <!-- TODO: datsheet: https://www.insta360.com/product/insta360-air -->
+    <xacro:property name="insta360_air_mass" value="0.05"/> <!-- estimated value -->
     <xacro:property name="insta360_air_length" value="0.021"/>
     <xacro:property name="insta360_air_width" value="0.07"/>
     <xacro:property name="insta360_air_height" value="0.025"/>
     <xacro:include filename="$(find hector_xacro_tools)/urdf/inertia_tensors.urdf.xacro" />
-    <xacro:macro name="${name}" params="name:=default *origin *parent">
+    <xacro:macro name="insta360_air" params="name *origin *parent">
         <joint name="${name}_joint" type="fixed">
             <child link="${name}_link"/>
@@ -34,12 +34,25 @@
         <joint name="${name}_rgb_left_joint" type="fixed">
             <origin xyz="0 0 0" rpy="0 0 0" />
-            <parent link="insta360_air_${name}_base_link" />
-            <child link="insta360_air_${name}_rgb_left" />
+            <parent link="${name}_link" />
+            <child link="${name}_rgb_left" />
+        </joint>
+        <link name="${name}_rgb_right"/>
+        <joint name="${name}_rgb_right_joint" type="fixed">
+            <origin xyz="0 0 0" rpy="0 0 ${M_PI}" />
+            <parent link="${name}_link" />
+            <child link="${name}_rgb_right" />
+        </joint>
+        <!-- Camera Optical Frame -->
+        <link name="${name}_left_optical_frame"/>
+        <joint name="${name}_left_optical_joint" type="fixed">
+            <origin xyz="0 0 0" rpy="-${M_PI/2} 0 -${M_PI/2}" />
+            <parent link="${name}_rgb_left" />
+            <child link="${name}_left_optical_frame" />
         </joint>
         <link name="${name}_right_optical_frame"/>
         <joint name="${name}_right_optical_joint" type="fixed">
-            <origin xyz="0 0 0" rpy="0 0 ${M_PI}" />
-            <parent link="insta360_air_${name}_base_link" />
-            <child link="insta360_air_${name}_right_optical_frame" />
+            <origin xyz="0 0 0" rpy="-${M_PI/2} 0 -${M_PI/2}" />
+            <parent link="${name}_rgb_right" />
+            <child link="${name}_right_optical_frame" />
         </joint>
     </xacro:macro>

File: urdf/livox_mid360.urdf.xacro (robot description, xacro)
@@ -8,11 +8,11 @@
 	<xacro:property name="livox_mid360_height" value="0.061"/>
 	<xacro:include filename="$(find hector_xacro_tools)/urdf/inertia_tensors.urdf.xacro" />
-	<xacro:macro name="${name}" params="name:=default *origin *parent">
-		<joint name="${name}_joint" type="fixed">
-			<child link="${name}_link"/>
+	<xacro:macro name="livox_mid360" params="name *origin *parent">
+		<joint name="${name}_lidar_joint" type="fixed">
+			<child link="${name}_lidar_link"/>
 			<xacro:insert_block name="origin"/>
 			<xacro:insert_block name="parent"/>
 		</joint>
-		<link name="${name}_link">
+		<link name="${name}_lidar_link">
 			<xacro:inertial_cuboid mass="${livox_mid360_mass}" x_length="${livox_mid360_length}" y_length="${livox_mid360_width}" z_length="${livox_mid360_height}"/>
 			<visual>

File: urdf/orbbec_astra2.urdf.xacro (robot description, xacro)
@@ -3,10 +3,10 @@
     <!-- datasheet: https://d1cd332k3pgc17.cloudfront.net/wp-content/uploads/2023/04/ORBBEC_Datasheet_Astra-2.pdf -->
     <xacro:property name="M_PI" value="3.14159"/>
-    <xacro:property name="orbbec_astra2_mass" value="0.195"/>
-    <xacro:property name="orbbec_astra2_length" value="0.037"/>
-    <xacro:property name="orbbec_astra2_width" value="0.147"/>
-    <xacro:property name="orbbec_astra2_height" value="0.035"/>
     <xacro:include filename="$(find hector_xacro_tools)/urdf/inertia_tensors.urdf.xacro" />
-    <xacro:macro name="${name}" params="name:=default *origin *parent">
+    <xacro:macro name="orbbec_astra2" params="name *origin *parent">
+        <xacro:property name="orbbec_astra2_mass" value="0.195"/>
+        <xacro:property name="orbbec_astra2_length" value="0.037"/>
+        <xacro:property name="orbbec_astra2_width" value="0.147"/>
+        <xacro:property name="orbbec_astra2_height" value="0.035"/>
         <joint name="${name}_joint" type="fixed">
             <child link="${name}_link"/>
@@ -38,9 +38,21 @@
         </joint>
         <!-- Optical Frame for ros (in z direction) -->
-        <link name="astra2_${name}_optical_frame"/>
-        <joint name="astra2_${name}_sensor_joint_optical_frame" type="fixed">
+        <link name="${name}_rgb_optical_frame"/>
+        <joint name="${name}_rgb_optical_joint" type="fixed">
             <origin xyz="0 0 0" rpy="-${M_PI/2.0} 0 -${M_PI/2.0}" />
-            <parent link="astra2_${name}_link" />
-            <child link="astra2_${name}_optical_frame" />
+            <parent link="${name}_link" />
+            <child link="${name}_rgb_optical_frame" />
+        </joint>
+        <link name="${name}_depth_link"/>
+        <joint name="${name}_depth_joint" type="fixed">
+            <origin xyz="0.033 0.022 0" rpy="0 0 0" />
+            <parent link="${name}_link" />
+            <child link="${name}_depth_link" />
+        </joint>
+        <link name="${name}_depth_optical_frame"/>
+        <joint name="${name}_depth_optical_joint" type="fixed">
+            <origin xyz="0 0 0" rpy="-${M_PI/2.0} 0 -${M_PI/2.0}" />
+            <parent link="${name}_link" />
+            <child link="${name}_depth_optical_frame" />
         </joint>
     </xacro:macro>

File: urdf/seek_thermal_xr.urdf.xacro (robot description, xacro)
@@ -8,5 +8,5 @@
     <xacro:property name="seek_thermal_xr_height" value="0.055"/>
     <xacro:include filename="$(find hector_xacro_tools)/urdf/inertia_tensors.urdf.xacro" />
-    <xacro:macro name="${name}" params="name:=default *origin *parent">
+    <xacro:macro name="seek_thermal_xr" params="name *origin *parent">
         <joint name="${name}_joint" type="fixed">
             <child link="${name}_link"/>
@@ -30,9 +30,15 @@
             </collision>
         </link>
+        <link name="${name}_thermal_link"/>
+        <joint name="${name}_thermal_joint" type="fixed">
+            <origin xyz="0.025 0 0" rpy="0 0 0" />
+            <parent link="${name}_link" />
+            <child link="${name}_thermal_link" />
+        </joint>
         <!-- Camera optical frame -->
         <link name="${name}_optical_frame"/>
         <joint name="${name}_optical_joint" type="fixed">
-            <origin xyz="0.025 0 0" rpy="-${M_PI/2} 0 -${M_PI/2}" />
-            <parent link="${name}_link" />
+            <origin xyz="0 0 0" rpy="-${M_PI/2} 0 -${M_PI/2}" />
+            <parent link="${name}_thermal_link" />
             <child link="${name}_optical_frame" />
         </joint>

Commit message: Publish frames for orbbecs in simulation using static tf publishers (#11)
this renames the frames to match the driver and removes them from the urdf to make the real robot urdf match the simulation

File: urdf/astra_stereo_s_u3.urdf.xacro (robot description, xacro)
@@ -32,33 +32,5 @@
             </collision>
         </link>
-        <!-- Camera RGB sensor -->
-        <link name="${name}_rgb_link"/>
-        <joint name="${name}_rgb_joint" type="fixed">
-            <origin xyz="0.014 0.01 0" rpy="0 0 0" />
-            <parent link="${name}_link" />
-            <child link="${name}_rgb_link" />
-        </joint>
-        <!-- Camera Depth sensor -->
-        <!-- Assuming the depth image is published in the same frame as the rgb image -->
-        <link name="${name}_depth_link"/>
-        <joint name="${name}_depth_joint" type="fixed">
-            <origin xyz="0.014 0.01 0" rpy="0 0 0" />
-            <parent link="${name}_link" />
-            <child link="${name}_depth_link" />
-        </joint>
-        <!-- Camera Optical Frame -->
-        <link name="${name}_rgb_optical_frame"/>
-        <joint name="${name}_rgb_optical_joint" type="fixed">
-            <origin xyz="0 0 0" rpy="-${M_PI/2.0} 0 -${M_PI/2.0}" />
-            <parent link="${name}_rgb_link" />
-            <child link="${name}_rgb_optical_frame" />
-        </joint>
-        <!-- Camera Depth Optical Frame -->
-        <link name="${name}_depth_optical_frame"/>
-        <joint name="${name}_depth_optical_joint" type="fixed">
-            <origin xyz="0 0 0" rpy="-${M_PI/2.0} 0 -${M_PI/2.0}" />
-            <parent link="${name}_depth_link" />
-            <child link="${name}_depth_optical_frame" />
-        </joint>
+    <!-- optical frames are published by driver, use launch file for simulation -->
     </xacro:macro>
 </robot>

Commit message: changed the inertia of the wide angle camera and orbbec astra s u3

File: urdf/astra_stereo_s_u3.urdf.xacro (robot description, xacro)
@@ -18,5 +18,5 @@
         <!-- Camera base -->
         <link name="${name}_link">
-            <xacro:inertial_cuboid mass="${orbbec_astra_stereo_s_u3_mass}" x_length="${orbbec_astra_stereo_s_u3_length}" y_length="${orbbec_astra_stereo_s_u3_width}" z_length="${orbbec_astra_stereo_s_u3_height}" />
+            <xacro:inertial_cuboid mass="${orbbec_astra_stereo_s_u3_mass}" x_length="${orbbec_astra_stereo_s_u3_width}" y_length="${orbbec_astra_stereo_s_u3_length}" z_length="${orbbec_astra_stereo_s_u3_height}" />
             <visual>
                 <origin xyz="0 0 0" rpy="0 0 0" />

File: urdf/generic_wide_angle_camera.urdf.xacro (robot description, xacro)
@@ -11,7 +11,7 @@
     <link name="${name}_link">
       <inertial>
-        <mass value="0.001" />
+        <mass value="0.01" />
         <origin xyz="0 0 0" rpy="0 0 0" />
-        <inertia ixx="0.0001" ixy="0" ixz="0" iyy="0.0001" iyz="0" izz="0.0001" />
+        <inertia ixx="0.000001" ixy="0" ixz="0" iyy="0.000001" iyz="0" izz="0.000001" />
       </inertial>
       <visual>
