Commit message: added visual and collision for the wide angle camera

File: urdf/generic_wide_angle_camera.urdf.xacro (robot description, xacro)
@@ -10,5 +10,5 @@
     </joint>
     <link name="${name}_link">
-<!--      <inertial>
+      <inertial>
         <mass value="0.001" />
         <origin xyz="0 0 0" rpy="0 0 0" />
@@ -16,18 +16,27 @@
       </inertial>
       <visual>
-        <origin xyz="0 0 0" rpy="0 0 0" />
+	    <origin xyz="0 0 0" rpy="0 0 0" />
         <geometry>
-          <box size="0.01 0.01 0.01" />
+          <box size="0.0017 0.032 0.032"/>
         </geometry>
-        <material name="Blue">
-          <color rgba="0.0 0.0 0.8 1"/>
+        <material name="Black">
+          <color rgba="0.0 0.0 0.0 1"/>
+        </material>
+      </visual>
+      <visual>
+        <origin xyz="0.00725 0 0" rpy="0 ${pi/2} 0" />
+        <geometry>
+          <cylinder radius="0.0086" length="0.0145" />
+        </geometry>
+        <material name="Black">
+          <color rgba="0.0 0.0 0.0 1"/>
         </material>
       </visual>
       <collision>
-        <origin xyz="0 0 0" rpy="0 0 0" />
+        <origin xyz="0.00725 0 0" rpy="0 0 0" />
         <geometry>
-          <box size="0.01 0.01 0.01" />
+          <box size="0.016 0.032 0.032" />
         </geometry>
-      </collision>-->
+      </collision>
     </link>
     <link name="${name}_optical_frame"/>

Commit message: added visual and collision for the wide angle camera (#16)
* added visual and collision for the wide angle camera

* added sphere collider to the livox mid360

* changed the inertia of the wide angle camera and orbbec astra s u3

File: urdf/generic_wide_angle_camera.urdf.xacro (robot description, xacro)
@@ -10,24 +10,33 @@
     </joint>
     <link name="${name}_link">
-<!--      <inertial>
-        <mass value="0.001" />
+      <inertial>
+        <mass value="0.01" />
         <origin xyz="0 0 0" rpy="0 0 0" />
-        <inertia ixx="0.0001" ixy="0" ixz="0" iyy="0.0001" iyz="0" izz="0.0001" />
+        <inertia ixx="0.000001" ixy="0" ixz="0" iyy="0.000001" iyz="0" izz="0.000001" />
       </inertial>
       <visual>
-        <origin xyz="0 0 0" rpy="0 0 0" />
+	    <origin xyz="0 0 0" rpy="0 0 0" />
         <geometry>
-          <box size="0.01 0.01 0.01" />
+          <box size="0.0017 0.032 0.032"/>
         </geometry>
-        <material name="Blue">
-          <color rgba="0.0 0.0 0.8 1"/>
+        <material name="Black">
+          <color rgba="0.0 0.0 0.0 1"/>
+        </material>
+      </visual>
+      <visual>
+        <origin xyz="0.00725 0 0" rpy="0 ${pi/2} 0" />
+        <geometry>
+          <cylinder radius="0.0086" length="0.0145" />
+        </geometry>
+        <material name="Black">
+          <color rgba="0.0 0.0 0.0 1"/>
         </material>
       </visual>
       <collision>
-        <origin xyz="0 0 0" rpy="0 0 0" />
+        <origin xyz="0.00725 0 0" rpy="0 0 0" />
         <geometry>
-          <box size="0.01 0.01 0.01" />
+          <box size="0.016 0.032 0.032" />
         </geometry>
-      </collision>-->
+      </collision>
     </link>
     <link name="${name}_optical_frame"/>
