Commit message: Updated Seek Thermal Xr camera

File: urdf/seek_thermal_xr.urdf.xacro (robot description, xacro)
@@ -20,5 +20,5 @@
                 <origin xyz="0 0 0" rpy="0 0 0" />
                 <geometry>
-                    <mesh filename="package://hector_sensors_description/meshes/seek_thermal_xr/seek_thermal_xr.dae"/>
+                    <mesh filename="package://hector_sensors_description/meshes/seek_thermal_xr/seek_thermal_xr.glb"/>
                 </geometry>
             </visual>
