Commit message: integrated feedback and made naming consistent

File: urdf/livox_mid360.urdf.xacro (robot description, xacro)
@@ -14,5 +14,5 @@
 			<xacro:insert_block name="parent"/>
 		</joint>
-		<link name="${name}_link">
+		<link name="${name}_lidar_link">
 			<xacro:inertial_cuboid mass="${livox_mid360_mass}" x_length="${livox_mid360_length}" y_length="${livox_mid360_width}" z_length="${livox_mid360_height}"/>
 			<visual>

Commit message: fixed lidar issue

File: urdf/livox_mid360.urdf.xacro (robot description, xacro)
@@ -9,10 +9,10 @@
 	<xacro:include filename="$(find hector_xacro_tools)/urdf/inertia_tensors.urdf.xacro" />
 	<xacro:macro name="livox_mid360" params="name *origin *parent">
-		<joint name="${name}_lidar_joint" type="fixed">
-			<child link="${name}_lidar_base_link"/>
+		<joint name="${name}_joint" type="fixed">
+			<child link="${name}_link"/>
 			<xacro:insert_block name="origin"/>
 			<xacro:insert_block name="parent"/>
 		</joint>
-		<link name="${name}_lidar_base_link">
+		<link name="${name}_link">
 			<xacro:inertial_cuboid mass="${livox_mid360_mass}" x_length="${livox_mid360_length}" y_length="${livox_mid360_width}" z_length="${livox_mid360_height}"/>
 			<visual>
@@ -29,9 +29,9 @@
 			</collision>
 		</link>
-		<link name="livox_mid360_${name}_laser_frame"/>
-		<joint name="livox_mid360_${name}_sensor_joint_laser_frame" type="fixed">
+		<link name="${name}_laser_frame"/>
+		<joint name="${name}_sensor_joint_laser_frame" type="fixed">
 			<origin xyz="0 0 0" rpy="0 0 ${M_PI/2.0}" />
-            <parent link="livox_mid360_${name}_base_link" />
-            <child link="livox_mid360_${name}_laser_frame" />
+            <parent link="${name}_link" />
+            <child link="${name}_laser_frame" />
         </joint>
 	</xacro:macro>

Commit message: corrected the frame names (#2)
* corrected the frame names

* integrated feedback and made naming consistent

* fixed lidar issue

---------

Co-authored-by: Markus Kramer <kramer@sim.tu-darmstadt.de>

File: urdf/livox_mid360.urdf.xacro (robot description, xacro)
@@ -2,4 +2,5 @@
 <robot xmlns:xacro="http://ros.org/wiki/xacro">
 	<!-- datasheet: https://terra-1-g.djicdn.com/851d20f7b9f64838a34cd02351370894/Livox/Livox_Mid-360_User_Manual_EN.pdf -->
+	<xacro:property name="M_PI" value="3.14159"/>
 	<xacro:property name="livox_mid360_mass" value="0.265"/>
 	<xacro:property name="livox_mid360_length" value="0.065"/>
@@ -7,18 +8,16 @@
 	<xacro:property name="livox_mid360_height" value="0.061"/>
 	<xacro:include filename="$(find hector_xacro_tools)/urdf/inertia_tensors.urdf.xacro" />
-	<xacro:property name="M_PI" value="3.14159"/>
-	<xacro:macro name="livox_mid360" params="name:=default *origin *parent">
-		<joint name="livox_mid360_${name}_joint" type="fixed">
-			<child link="livox_mid360_${name}_base_link"/>
+	<xacro:macro name="livox_mid360" params="name *origin *parent">
+		<joint name="${name}_joint" type="fixed">
+			<child link="${name}_link"/>
 			<xacro:insert_block name="origin"/>
 			<xacro:insert_block name="parent"/>
 		</joint>
-		<link name="livox_mid360_${name}_base_link">
+		<link name="${name}_link">
 			<xacro:inertial_cuboid mass="${livox_mid360_mass}" x_length="${livox_mid360_length}" y_length="${livox_mid360_width}" z_length="${livox_mid360_height}"/>
 			<visual>
 				<origin xyz="0 0 0" rpy="0 0 0"/>
 				<geometry>
-					<mesh filename="package://hector_sensors_description/meshes/livox_mid360/livox_mid360.dae">
-					</mesh>
+					<mesh filename="package://hector_sensors_description/meshes/livox_mid360/livox_mid360.dae"/>
 				</geometry>
 			</visual>
@@ -30,9 +29,9 @@
 			</collision>
 		</link>
-		<link name="livox_mid360_${name}_laser_frame"/>
-		<joint name="livox_mid360_${name}_sensor_joint_laser_frame" type="fixed">
+		<link name="${name}_laser_frame"/>
+		<joint name="${name}_sensor_joint_laser_frame" type="fixed">
 			<origin xyz="0 0 0" rpy="0 0 ${M_PI/2.0}" />
-            <parent link="livox_mid360_${name}_base_link" />
-            <child link="livox_mid360_${name}_laser_frame" />
+            <parent link="${name}_link" />
+            <child link="${name}_laser_frame" />
         </joint>
 	</xacro:macro>

File: urdf/seek_thermal_xr.urdf.xacro (robot description, xacro)
@@ -2,4 +2,5 @@
 <robot xmlns:xacro="http://ros.org/wiki/xacro">
     <!-- datasheet: https://www.thermal.com/uploads/1/0/1/3/101388544/compactxr-sellsheet-usa_web.pdf -->
+    <xacro:property name="M_PI" value="3.14159"/>
     <xacro:property name="seek_thermal_xr_mass" value="0.014"/>
     <xacro:property name="seek_thermal_xr_length" value="0.027"/>
@@ -7,13 +8,12 @@
     <xacro:property name="seek_thermal_xr_height" value="0.055"/>
     <xacro:include filename="$(find hector_xacro_tools)/urdf/inertia_tensors.urdf.xacro" />
-    <xacro:property name="M_PI" value="3.14159"/>
-    <xacro:macro name="seek_thermal_xr" params="name:=default *origin *parent">
-        <joint name="seek_thermal_xr_${name}_base_joint" type="fixed">
-            <child link="seek_thermal_xr_${name}_base_link"/>
+    <xacro:macro name="seek_thermal_xr" params="name *origin *parent">
+        <joint name="${name}_joint" type="fixed">
+            <child link="${name}_link"/>
             <xacro:insert_block name="origin"/>
             <xacro:insert_block name="parent"/>
         </joint>
         <!-- Camera base -->
-        <link name="seek_thermal_xr_${name}_base_link">
+        <link name="${name}_link">
             <xacro:inertial_cuboid mass="${seek_thermal_xr_mass}" x_length="${seek_thermal_xr_length}" y_length="${seek_thermal_xr_width}" z_length="${seek_thermal_xr_height}" />
             <visual>
@@ -30,10 +30,16 @@
             </collision>
         </link>
-        <!-- Camera sensor -->
-        <link name="seek_thermal_xr_${name}_link"/>
-        <joint name="seek_thermal_xr_${name}_sensor_joint" type="fixed">
+        <link name="${name}_thermal_link"/>
+        <joint name="${name}_thermal_joint" type="fixed">
             <origin xyz="0.025 0 0" rpy="0 0 0" />
-            <parent link="seek_thermal_xr_${name}_base_link" />
-            <child link="seek_thermal_xr_${name}_link" />
+            <parent link="${name}_link" />
+            <child link="${name}_thermal_link" />
+        </joint>
+        <!-- Camera optical frame -->
+        <link name="${name}_optical_frame"/>
+        <joint name="${name}_optical_joint" type="fixed">
+            <origin xyz="0 0 0" rpy="-${M_PI/2} 0 -${M_PI/2}" />
+            <parent link="${name}_thermal_link" />
+            <child link="${name}_optical_frame" />
         </joint>
     </xacro:macro>

Commit message: Fixed livox laser frame orientation.

File: urdf/livox_mid360.urdf.xacro (robot description, xacro)
@@ -33,5 +33,5 @@
 		<link name="${name}_laser_frame"/>
 		<joint name="${name}_sensor_joint_laser_frame" type="fixed">
-			<origin xyz="0 0 0" rpy="0 0 ${M_PI/2.0}" />
+			<origin xyz="0 0 0" rpy="0 0 ${-M_PI/2.0}" />
             <parent link="${name}_link" />
             <child link="${name}_laser_frame" />

Commit message: adjusted position of livox laser_frame

File: urdf/livox_mid360.urdf.xacro (robot description, xacro)
@@ -33,5 +33,5 @@
 		<link name="${name}_laser_frame"/>
 		<joint name="${name}_sensor_joint_laser_frame" type="fixed">
-			<origin xyz="0 0 0" rpy="0 0 ${-M_PI/2.0}" />
+			<origin xyz="0 0 0.03" rpy="0 0 ${-M_PI/2.0}" />
             <parent link="${name}_link" />
             <child link="${name}_laser_frame" />

Commit message: adjusted livox laser frame to correct z-offset

File: urdf/livox_mid360.urdf.xacro (robot description, xacro)
@@ -33,5 +33,5 @@
 		<link name="${name}_laser_frame"/>
 		<joint name="${name}_sensor_joint_laser_frame" type="fixed">
-			<origin xyz="0 0 0.03" rpy="0 0 ${-M_PI/2.0}" />
+			<origin xyz="0 0 0.047" rpy="0 0 ${-M_PI/2.0}" />
             <parent link="${name}_link" />
             <child link="${name}_laser_frame" />

Commit message: added sphere collider to the livox mid360

File: urdf/livox_mid360.urdf.xacro (robot description, xacro)
@@ -30,4 +30,10 @@
 				</geometry>
 			</collision>
+			<collision>
+                <origin xyz="0 0 0.039" rpy="0 0 0" />
+                <geometry>
+                    <sphere radius="0.03" />
+                </geometry>
+            </collision>
 		</link>
 		<link name="${name}_laser_frame"/>

Commit message: Changed livox_360 collision to a single sphere

File: urdf/livox_mid360.urdf.xacro (robot description, xacro)
@@ -27,5 +27,5 @@
         <origin xyz="0 0.0002 0.03" rpy="0 0 0"/>
         <geometry>
-          <box size="${livox_mid360_length} ${livox_mid360_width} ${livox_mid360_height}"/>
+          <sphere radius="0.0545"/>
         </geometry>
       </collision>

Commit message: added imu frame for livox mid 360

File: urdf/livox_mid360.urdf.xacro (robot description, xacro)
@@ -37,4 +37,10 @@
       <child link="${name}_laser_frame"/>
     </joint>
+    <link name="${name}_imu_frame"/>
+    <joint name="${name}_sensor_joint_imu_frame" type="fixed">
+      <origin xyz="-0.011 -0.02329 0.04412" rpy="0 0 0"/>
+      <parent link="${name}_link"/>
+      <child link="${name}_imu_frame"/>
+    </joint>
   </xacro:macro>
 </robot>
