Commit message: swapped size axis

File: urdf/seek_thermal_nano.urdf.xacro (robot description, xacro)
@@ -3,6 +3,6 @@
   <!-- datasheet: https://cdn-reichelt.de/documents/datenblatt/D100/NANO_DB-EN.pdf -->
   <xacro:property name="seek_thermal_nano_mass" value="0.013"/>
-  <xacro:property name="seek_thermal_nano_length" value="0.025"/>
-  <xacro:property name="seek_thermal_nano_width" value="0.022"/>
+  <xacro:property name="seek_thermal_nano_length" value="0.022"/>
+  <xacro:property name="seek_thermal_nano_width" value="0.025"/>
   <xacro:property name="seek_thermal_nano_height" value="0.025"/>
   <xacro:include filename="$(find hector_xacro_tools)/urdf/inertia_tensors.urdf.xacro"/>
@@ -24,5 +24,5 @@
       </visual>
       <collision>
-        <origin xyz="0.013 0 -0.011" rpy="0 0 0"/>
+        <origin xyz="0.0 0 0.0" rpy="0 0 0"/>
         <geometry>
           <box size="${seek_thermal_nano_length} ${seek_thermal_nano_width} ${seek_thermal_nano_height}"/>
@@ -30,15 +30,9 @@
       </collision>
     </link>
-    <link name="${name}_thermal_link"/>
-    <joint name="${name}_thermal_joint" type="fixed">
-      <origin xyz="0.025 0 0" rpy="0 0 0"/>
-      <parent link="${name}_link"/>
-      <child link="${name}_thermal_link"/>
-    </joint>
     <!-- Camera optical frame -->
     <link name="${name}_optical_frame"/>
     <joint name="${name}_optical_joint" type="fixed">
       <origin xyz="0 0 0" rpy="-${pi/2} 0 -${pi/2}"/>
-      <parent link="${name}_thermal_link"/>
+      <parent link="${name}_link"/>
       <child link="${name}_optical_frame"/>
     </joint>

Commit message: Added model for seek thermal nano

File: urdf/seek_thermal_nano.urdf.xacro (robot description, xacro)
@@ -19,6 +19,5 @@
         <origin xyz="0 0 0" rpy="0 0 0"/>
         <geometry>
-          <!--mesh filename="package://hector_sensors_description/meshes/seek_thermal_nano/seek_thermal_nano.glb"/-->
-          <box size="${seek_thermal_nano_length} ${seek_thermal_nano_width} ${seek_thermal_nano_height}"/>
+          <mesh filename="package://hector_sensors_description/meshes/seek_thermal_nano/seek_thermal_nano.glb"/>
         </geometry>
       </visual>
