Commit message: updated generic camera and fixed the corrupted file. Also updated it to nclude a parameter for wide angle cameras

File: gazebo/generic_camera.gazebo.xacro (robot description, xacro)
@@ -2,7 +2,13 @@
 <robot xmlns:xacro="http://ros.org/wiki/xacro">
     <xacro:property name="M_PI" value="3.14159"/>
-    <xacro:macro name="generic_camera_gazebo" params="name robot_name update_rate res_x res_y hfov image_format">
+    <xacro:macro name="generic_camera_gazebo" params="name robot_name update_rate res_x res_y hfov image_format wide_angle=false">
+        <xacro:if value="${wide_angle}">
+            <xacro:property name="camera_type" value="wideanglecamera"/>
+        </xacro:if>
+        <xacro:unless value="${wide_angle}">
+            <xacro:property name="camera_type" value="camera"/>
+        </xacro:unless>
         <gazebo reference="${name}_link">
-            <sensor type="camera" name="${name}_camera_sensor">
+            <sensor type="${camera_type}" name="${name}_camera_sensor">
                 <update_rate>${update_rate}</update_rate>
                 <topic>${robot_name}/${name}/image_raw</topic>
