Commit message: Updated wide angle camera

File: gazebo/generic_wide_angle_camera.gazebo.xacro (robot description, xacro)
@@ -2,7 +2,7 @@
 <robot xmlns:xacro="http://ros.org/wiki/xacro">
     <xacro:property name="M_PI" value="3.14159"/>
-    <xacro:macro name="generic_camera_gazebo" params="name robot_name update_rate res_x res_y hfov image_format">
+    <xacro:macro name="generic_wide_angle_camera_gazebo" params="name robot_name update_rate res_x res_y hfov image_format">
         <gazebo reference="${name}_link">
-            <sensor type="camera" name="${name}_camera_sensor">
+            <sensor type="wideanglecamera" name="${name}_camera_sensor">
                 <update_rate>${update_rate}</update_rate>
                 <topic>${robot_name}/${name}/image_raw</topic>
@@ -20,4 +20,10 @@
                         <far>100</far>
                     </clip>
+                     <lens>
+                        <type>equidistant</type>
+                        <cutoff_angle>${hfov * M_PI/180.0 / 2.0}</cutoff_angle>
+                        <scale_to_hfov>true</scale_to_hfov>
+                        <env_texture_size>512</env_texture_size>
+                    </lens>
                 </camera>
                 <!--frameName>${name}_optical_frame</frameName-->

File: urdf/generic_wide_angle_camera.urdf.xacro (robot description, xacro)
@@ -1,7 +1,7 @@
 <?xml version="1.0"?>
 <robot xmlns:xacro="http://www.ros.org/wiki/xacro">
-  <xacro:include filename="$(find hector_sensors_description)/gazebo/generic_camera.gazebo.xacro"/>
+  <xacro:include filename="$(find hector_sensors_description)/gazebo/generic_wide_angle_camera.gazebo.xacro"/>
   <xacro:property name="M_PI" value="3.1415926535897931" />
-  <xacro:macro name="generic_camera" params="name parent robot_name *origin ros_topic cam_info_topic update_rate res_x res_y image_format hfov">
+  <xacro:macro name="generic_wide_angle_camera" params="name parent robot_name *origin ros_topic cam_info_topic update_rate res_x res_y image_format hfov">
     <joint name="${name}_joint" type="fixed">
       <xacro:insert_block name="origin" />
@@ -37,5 +37,5 @@
       <child link="${name}_optical_frame"/>
     </joint>
-    <xacro:generic_camera_gazebo name="${name}" robot_name="${robot_name}" update_rate="${update_rate}" res_x="${res_x}" res_y="${res_y}" hfov="${hfov}" image_format="${image_format}"/>
+    <xacro:generic_wide_angle_camera_gazebo name="${name}" robot_name="${robot_name}" update_rate="${update_rate}" res_x="${res_x}" res_y="${res_y}" hfov="${hfov}" image_format="${image_format}"/>
   </xacro:macro>
 </robot>
