Commit message: updated intel_realsense_d435

File: gazebo/intel_realsense_d435.gazebo.xacro (robot description, xacro)
@@ -1,8 +1,8 @@
 <?xml version="1.0"?>
 <robot xmlns:xacro="http://ros.org/wiki/xacro">
-	<xacro:property name="M_PI" value="3.14159"/>
-	<xacro:arg name="semantic_segmentation" default="false"/>
-	<xacro:macro name="orbbec_astra_stereo_s_u3_gazebo" params="name:=default semantic_segmentation:=false">
-	    <gazebo reference="${name}_link">
+    <xacro:property name="M_PI" value="3.14159"/>
+    <xacro:arg name="semantic_segmentation" default="false"/>
+    <xacro:macro name="intel_realsense_d435_gazebo" params="name:=default semantic_segmentation:=false">
+        <gazebo reference="${name}_link">
 			<sensor type="camera" name="${name}_rgb">
 				<always_on>true</always_on>
@@ -14,13 +14,13 @@
 					<camera_info_topic>/$(arg robot_name)/${name}/rgb/camera_info</camera_info_topic>
 					<optical_frame_id>${name}_rgb_optical_frame</optical_frame_id>
-					<horizontal_fov>${90.0 * M_PI/180.0}</horizontal_fov>
+					<horizontal_fov>${91.2 * M_PI/180.0}</horizontal_fov>
 					<image>
 						<format>R8G8B8</format>
-						<width>720</width>
+						<width>640</width>
 						<height>480</height>
 					</image>
 					<clip>
-						<near>0.05</near>
-						<far>10</far>
+						<near>0.3</near>
+						<far>3</far>
 					</clip>
 				</camera>
@@ -35,5 +35,5 @@
 					<camera_info_topic>/$(arg robot_name)/${name}/depth/camera_info</camera_info_topic>
 					<optical_frame_id>${name}_depth_optical_frame</optical_frame_id>
-					<horizontal_fov>1.047</horizontal_fov>
+					<horizontal_fov>${91.2 * M_PI/180.0}</horizontal_fov>
 					<image>
 						<format>R_FLOAT32</format>
@@ -43,6 +43,6 @@
 					<depth_camera>
 						<clip>
-							<near>0.1</near>
-							<far>10.0</far>
+							<near>0.3</near>
+							<far>3</far>
 						</clip>
 					</depth_camera>
@@ -54,25 +54,5 @@
 				</camera>
 			</sensor>
-			<xacro:if value="$(arg semantic_segmentation)">
-				<sensor name="astra2_${name}_segmentation_camera" type="segmentation">
-					<topic>/$(arg robot_name)/${name}/segmentation</topic>
-					<gz_frame_id>${name}_link</gz_frame_id>
-					<camera>
-						<optical_frame_id>${name}_optical_frame</optical_frame_id>
-						<segmentation_type>instance</segmentation_type>
-						<horizontal_fov>${90.0 * M_PI/180.0}</horizontal_fov>
-						<image>
-							<width>720</width>
-							<height>480</height>
-						</image>
-						<clip>
-							<near>0.1</near>
-							<far>10</far>
-						</clip>
-					</camera>
-					<update_rate>5</update_rate>
-				</sensor>
-			</xacro:if>
-		</gazebo>
-	</xacro:macro>
+        </gazebo>
+    </xacro:macro>
 </robot>
