Commit message: changed sensors to use arg robot_name and unified topics to be $(arg robot_name)/topic
Additionally added xacro.arg for the robot_name.

This allows to initialize the robots as standalone without providing a
robot_name (for default topics /topic) and to namespace them by
providing the arg robot_name, which is done in our robot urdfs anyways.

File: gazebo/astra_stereo_s_u3.gazebo.xacro (robot description, xacro)
@@ -2,4 +2,5 @@
 <robot xmlns:xacro="http://ros.org/wiki/xacro">
 	<xacro:property name="M_PI" value="3.14159"/>
+	<xacro:arg name="robot_name" default=""/>
 	<xacro:macro name="orbbec_astra_stereo_s_u3_gazebo" params="name:=default">
 		<gazebo reference="astra_stereo_s_${name}_link">
@@ -8,8 +9,8 @@
 				<visualize>true</visualize>
 				<update_rate>15</update_rate>
-				<topic>/$(arg robot_name)/astra_stereo_s_${name}/rgb/image_raw</topic>
+				<topic>$(arg robot_name)/astra_stereo_s_${name}/rgb/image_raw</topic>
 				<gz_frame_id>astra2_${name}_link</gz_frame_id>
 				<camera name="astra_stereo_s_u3_${name}_camera">
-					<camera_info_topic>/$(arg robot_name)/astra2_${name}/rgb/camera_info</camera_info_topic>
+					<camera_info_topic>$(arg robot_name)/astra2_${name}/rgb/camera_info</camera_info_topic>
 					<optical_frame_id>astra2_${name}_optical_frame</optical_frame_id>
 					<horizontal_fov>${90.0 * M_PI/180.0}</horizontal_fov>
@@ -29,8 +30,8 @@
 				<visualize>true</visualize>
 				<update_rate>15</update_rate>
-				<topic>/$(arg robot_name)/astra2_${name}/depth/image_raw</topic>
+				<topic>$(arg robot_name)/astra2_${name}/depth/image_raw</topic>
 				<gz_frame_id>astra2_${name}_link</gz_frame_id>
 				<camera>
-					<camera_info_topic>/$(arg robot_name)/astra2_${name}/depth/camera_info</camera_info_topic>
+					<camera_info_topic>$(arg robot_name)/astra2_${name}/depth/camera_info</camera_info_topic>
 					<optical_frame_id>astra2_${name}_optical_frame</optical_frame_id>
 					<horizontal_fov>1.047</horizontal_fov>
@@ -55,5 +56,5 @@
 			<xacro:if value="$(arg semantic_segmentation)">
 				<sensor name="astra2_${name}_segmentation_camera" type="segmentation">
-					<topic>/$(arg robot_name)/astra2_${name}/segmentation</topic>
+					<topic>$(arg robot_name)/astra2_${name}/segmentation</topic>
 					<gz_frame_id>astra2_${name}_link</gz_frame_id>
 					<camera>

File: gazebo/flir_a65_camera.gazebo.xacro (robot description, xacro)
@@ -1,13 +1,14 @@
 <?xml version="1.0"?>
 <robot xmlns:xacro="http://ros.org/wiki/xacro">
-    <xacro:macro name="flir_a65_camera_gazebo" params="robot_name">
+    <xacro:arg name="robot_name" default=""/>
+    <xacro:macro name="flir_a65_camera_gazebo" params="name">
         <gazebo reference="${name}_frame">
             <sensor type="thermal" name="${name}_thermal_cam">
                 <update_rate>9</update_rate>
                 <always_on>true</always_on>
-                <topic>${robot_name}/thermal_camera/image_raw</topic>
+                <topic>$(arg robot_name)/thermal_camera/image_raw</topic>
                 <gz_frame_id>${name}_optical_frame</gz_frame_id>
                 <camera name="${name}">
-                    <camera_info_topic>${robot_name}/${name}/camera_info</camera_info_topic>
+                    <camera_info_topic>$(arg robot_name)/${name}/camera_info</camera_info_topic>
                     <horizontal_fov>${45.0*pi/180.0}</horizontal_fov>
                     <image>

File: gazebo/generic_camera.gazebo.xacro (robot description, xacro)
@@ -1,13 +1,14 @@
 <?xml version="1.0"?>
 <robot xmlns:xacro="http://ros.org/wiki/xacro">
+    <xacro:arg name="robot_name" default=""/>
     <xacro:property name="M_PI" value="3.14159"/>
-    <xacro:macro name="generic_camera_gazebo" params="name robot_name update_rate res_x res_y hfov image_format">
+    <xacro:macro name="generic_camera_gazebo" params="name update_rate res_x res_y hfov image_format">
         <gazebo reference="${name}_link">
             <sensor type="camera" name="${name}_camera_sensor">
                 <update_rate>${update_rate}</update_rate>
-                <topic>${robot_name}/${name}/image_raw</topic>
+                <topic>$(arg robot_name)/${name}/image_raw</topic>
                 <gz_frame_id>${name}_optical_frame</gz_frame_id>
                 <camera name="${name}">
-                    <camera_info_topic>${robot_name}/${name}/camera_info</camera_info_topic>
+                    <camera_info_topic>$(arg robot_name)/${name}/camera_info</camera_info_topic>
                     <horizontal_fov>${hfov * M_PI/180.0}</horizontal_fov>
                     <image>

File: gazebo/insta360_air.gazebo.xacro (robot description, xacro)
@@ -2,4 +2,5 @@
 <robot xmlns:xacro="http://ros.org/wiki/xacro">
     <xacro:property name="M_PI" value="3.14159"/>
+    <xacro:arg name="robot_name" default=""/>
     <xacro:macro name="insta360_air_gazebo" params="name:=default">
         <gazebo reference="insta360_air_${name}_left_optical_frame">
@@ -8,8 +9,8 @@
                 <visualize>true</visualize>
                 <update_rate>15</update_rate>
-                <topic>/$(arg robot_name)/insta360_air_${name}_left/rgb/image_raw</topic>
+                <topic>$(arg robot_name)/insta360_air_${name}_left/rgb/image_raw</topic>
                 <gz_frame_id>insta360_air_${name}_left_optical_frame</gz_frame_id>
                 <camera>
-                    <camera_info_topic>/$(arg robot_name)/insta360_air_${name}_left/rgb/camera_info</camera_info_topic>
+                    <camera_info_topic>$(arg robot_name)/insta360_air_${name}_left/rgb/camera_info</camera_info_topic>
                     <horizontal_fov>${M_PI}</horizontal_fov>
                     <image>
@@ -36,8 +37,8 @@
                 <visualize>true</visualize>
                 <update_rate>15</update_rate>
-                <topic>/$(arg robot_name)/insta360_air_${name}_right/rgb/image_raw</topic>
+                <topic>$(arg robot_name)/insta360_air_${name}_right/rgb/image_raw</topic>
                 <gz_frame_id>insta360_air_${name}_right_optical_frame</gz_frame_id>
                 <camera>
-                    <camera_info_topic>/$(arg robot_name)/insta360_air_${name}_right/rgb/camera_info</camera_info_topic>
+                    <camera_info_topic>$(arg robot_name)/insta360_air_${name}_right/rgb/camera_info</camera_info_topic>
                     <optical_frame_id>insta360_air_${name}_right_optical_frame</optical_frame_id>
                     <horizontal_fov>${M_PI}</horizontal_fov>

File: gazebo/insta360_pro2.gazebo.xacro (robot description, xacro)
@@ -2,13 +2,14 @@
 <robot xmlns:xacro="http://ros.org/wiki/xacro">
     <xacro:property name="M_PI" value="3.14159"/>
-    <xacro:macro name="insta360_pro2_gazebo" params="camera_name robot_name ros_topic update_rate fov image_format res_x res_y">
+    <xacro:arg name="robot_name" default=""/>
+    <xacro:macro name="insta360_pro2_gazebo" params="camera_name ros_topic update_rate fov image_format res_x res_y">
         <gazebo reference="${camera_name}_link">
             <sensor type="wideanglecamera" name="${camera_name}_camera_sensor">
                 <update_rate>${update_rate}</update_rate>
-                <topic>${robot_name}/${camera_name}/${ros_topic}</topic>
+                <topic>$(arg robot_name)/${camera_name}/${ros_topic}</topic>
                 <gz_frame_id>${camera_name}_optical_frame</gz_frame_id>
                 <camera name="${name}">
                 <!--<horizontal_fov>${hfov * pi/180.0}</horizontal_fov>-->
-                    <camera_info_topic>${robot_name}/${camera_name}/camera_info</camera_info_topic>
+                    <camera_info_topic>$(arg robot_name)/${camera_name}/camera_info</camera_info_topic>
                     <horizontal_fov>${fov}</horizontal_fov>
                     <image>

File: gazebo/livox_mid360.gazebo.xacro (robot description, xacro)
@@ -2,9 +2,10 @@
 <robot xmlns:xacro="http://ros.org/wiki/xacro">
 	<xacro:property name="M_PI" value="3.14159"/>
+	<xacro:arg name="robot_name" default=""/>
 	<xacro:macro name="livox_mid360_gazebo" params="visualize:=True name:=default">
 		<gazebo reference="livox_mid360_${name}_laser_frame">
 			<sensor name='gpu_lidar_${name}' type='gpu_lidar'>"
 				<pose relative_to='livox_mid360_${name}_laser_frame'>0 0 0 0 0 0</pose>
-				<topic>/$(arg robot_name)/livox_mid360_${name}</topic>
+				<topic>$(arg robot_name)/livox_mid360_${name}</topic>
 				<update_rate>10</update_rate>
 				<gz_frame_id>livox_mid360_${name}_laser_frame</gz_frame_id>

File: gazebo/orbbec_astra2.gazebo.xacro (robot description, xacro)
@@ -2,4 +2,5 @@
 <robot xmlns:xacro="http://ros.org/wiki/xacro">
 	<xacro:property name="M_PI" value="3.14159"/>
+	<xacro:arg name="robot_name" default=""/>
 	<xacro:macro name="orbbec_astra2_gazebo" params="name:=default semantic_segmentation:=false">
 		<gazebo reference="astra2_${name}_link">
@@ -8,8 +9,8 @@
 				<visualize>true</visualize>
 				<update_rate>15</update_rate>
-				<topic>/$(arg robot_name)/astra2_${name}/rgb/image_raw</topic>
+				<topic>$(arg robot_name)/astra2_${name}/rgb/image_raw</topic>
 				<gz_frame_id>astra2_${name}_link</gz_frame_id>
 				<camera name="astra2_${name}_camera">
-					<camera_info_topic>/$(arg robot_name)/astra2_${name}/rgb/camera_info</camera_info_topic>
+					<camera_info_topic>$(arg robot_name)/astra2_${name}/rgb/camera_info</camera_info_topic>
 					<optical_frame_id>astra2_${name}_optical_frame</optical_frame_id>
 					<horizontal_fov>${90.0 * M_PI/180.0}</horizontal_fov>
@@ -29,5 +30,5 @@
 				<visualize>true</visualize>
 				<update_rate>15</update_rate>
-				<topic>/$(arg robot_name)/astra2_${name}/depth/image_raw</topic>
+				<topic>$(arg robot_name)/astra2_${name}/depth/image_raw</topic>
 				<gz_frame_id>astra2_${name}_link</gz_frame_id>
 				<camera>
@@ -55,5 +56,5 @@
 			<xacro:if value="$(arg semantic_segmentation)">
 				<sensor name="astra2_${name}_segmentation_camera" type="segmentation">
-					<topic>/$(arg robot_name)/astra2_${name}/segmentation</topic>
+					<topic>$(arg robot_name)/astra2_${name}/segmentation</topic>
 					<gz_frame_id>astra2_${name}_link</gz_frame_id>
 					<camera>

File: gazebo/os0_128.gazebo.xacro (robot description, xacro)
@@ -1,5 +1,6 @@
 <?xml version="1.0"?>
 <robot xmlns:xacro="http://ros.org/wiki/xacro">
-    <xacro:macro name="os0_128_gazebo" params="name robot_name update_rate horizontal_samples vertical_samples min_range max_range">
+    <xacro:arg name="robot_name" default=""/>
+    <xacro:macro name="os0_128_gazebo" params="name update_rate horizontal_samples vertical_samples min_range max_range">
         <gazebo reference="${name}_frame">
             <sensor name="${name}-OS0-128" type="gpu_lidar">
@@ -7,5 +8,5 @@
                 <always_on>true</always_on>
                 <update_rate>${update_rate}</update_rate>
-                <topic>${robot_name}/${name}/scan</topic>
+                <topic>$(arg robot_name)/${name}/scan</topic>
                 <!--gz_frame_id>${name}_frame</gz_frame_id-->
                 <lidar>

File: gazebo/realsense_d435_camera.gazebo.xacro (robot description, xacro)
@@ -2,14 +2,15 @@
 <robot xmlns:xacro="http://ros.org/wiki/xacro">
     <xacro:property name="M_PI" value="3.14159"/>
-    <xacro:macro name="realsense_d435_camera_gazebo" params="name robot_name parent frame_name:=color min_range max_range update_rate">
+    <xacro:arg name="robot_name" default=""/>
+    <xacro:macro name="realsense_d435_camera_gazebo" params="name parent frame_name:=color min_range max_range update_rate">
         <gazebo reference="${name}_link">
             <sensor type="rgbd_camera" name="${name}">
             <!-- Camera-specific parameters -->
             <update_rate>${update_rate}</update_rate>
-            <topic>${robot_name}/${name}</topic>
+            <topic>$(arg robot_name)/${name}</topic>
             <gz_frame_id>${name}_${frame_name}_optical_frame</gz_frame_id>
             <!-- frameName>${name}_${frame_name}_optical_frame</frameName-->
             <camera name="${name}_color">
-                <camera_info_topic>${robot_name}/${name}/camera_info</camera_info_topic>
+                <camera_info_topic>$(arg robot_name)/${name}/camera_info</camera_info_topic>
                 <horizontal_fov>${69.4 * M_PI/180.0}</horizontal_fov>
                 <image>

File: urdf/flir_a65_camera.urdf.xacro (robot description, xacro)
@@ -30,9 +30,9 @@
     </gazebo>
   </xacro:macro>
-  <xacro:macro name="flir_a65_camera" params="name parent robot_name *origin">
+  <xacro:macro name="flir_a65_camera" params="name parent *origin">
     <xacro:flir_a65_camera_model name="${name}" parent="${parent}">
       <xacro:insert_block name="origin" />
     </xacro:flir_a65_camera_model>
-    <xacro:flir_a65_camera_gazebo robot_name="${robot_name}"/>
+    <xacro:flir_a65_camera_gazebo name="${name}"/>
   </xacro:macro>
 </robot>

File: urdf/generic_camera.urdf.xacro (robot description, xacro)
@@ -3,5 +3,5 @@
   <xacro:include filename="$(find hector_sensors_description)/gazebo/generic_camera.gazebo.xacro"/>
   <xacro:property name="M_PI" value="3.1415926535897931" />
-  <xacro:macro name="generic_camera" params="name parent robot_name *origin ros_topic cam_info_topic update_rate res_x res_y image_format hfov">
+  <xacro:macro name="generic_camera" params="name parent *origin ros_topic cam_info_topic update_rate res_x res_y image_format hfov">
     <joint name="${name}_joint" type="fixed">
       <xacro:insert_block name="origin" />
@@ -37,5 +37,5 @@
     </joint>
     <link name="${name}_optical_frame"/>
-    <xacro:generic_camera_gazebo name="${name}" robot_name="${robot_name}" update_rate="${update_rate}" res_x="${res_x}" res_y="${res_y}" hfov="${hfov}" image_format="${image_format}"/>
+    <xacro:generic_camera_gazebo name="${name}" update_rate="${update_rate}" res_x="${res_x}" res_y="${res_y}" hfov="${hfov}" image_format="${image_format}"/>
   </xacro:macro>
 </robot>

File: urdf/insta360_pro2.urdf.xacro (robot description, xacro)
@@ -6,5 +6,5 @@
     <color rgba="0.5 0.5 0.5 1" />
   </material>
-  <xacro:macro name="insta360_pro2" params="name parent robot_name *origin ros_topic update_rate res_x res_y image_format fov">
+  <xacro:macro name="insta360_pro2" params="name parent *origin ros_topic update_rate res_x res_y image_format fov">
     <joint name="${name}_center_joint" type="fixed">
       <xacro:insert_block name="origin" />
@@ -53,5 +53,5 @@
     </xacro:insta360_pro2_camera>
   </xacro:macro>
-  <xacro:macro name="insta360_pro2_with_calibration" params="name parent robot_name *origin *calibration1 *calibration2 *calibration3 *calibration4 *calibration5 *calibration6 ros_topic update_rate res_x res_y image_format fov">
+  <xacro:macro name="insta360_pro2_with_calibration" params="name parent *origin *calibration1 *calibration2 *calibration3 *calibration4 *calibration5 *calibration6 ros_topic update_rate res_x res_y image_format fov">
     <joint name="${name}_center_joint" type="fixed">
       <xacro:insert_block name="origin" />
@@ -81,24 +81,24 @@
       </collision>
     </link>
-    <xacro:insta360_pro2_camera parent="${name}_origin2_optical_frame" robot_name="${robot_name}" camera_number="1" ros_topic="${ros_topic}" update_rate="${update_rate}" res_x="${res_x}" res_y="${res_y}" image_format="${image_format}" fov="${fov}">
+    <xacro:insta360_pro2_camera parent="${name}_origin2_optical_frame" camera_number="1" ros_topic="${ros_topic}" update_rate="${update_rate}" res_x="${res_x}" res_y="${res_y}" image_format="${image_format}" fov="${fov}">
       <xacro:insert_block name="calibration1" />
     </xacro:insta360_pro2_camera>
-    <xacro:insta360_pro2_camera parent="${name}_origin3_optical_frame" robot_name="${robot_name}" camera_number="2" ros_topic="${ros_topic}" update_rate="${update_rate}" res_x="${res_x}" res_y="${res_y}" image_format="${image_format}" fov="${fov}">
+    <xacro:insta360_pro2_camera parent="${name}_origin3_optical_frame" camera_number="2" ros_topic="${ros_topic}" update_rate="${update_rate}" res_x="${res_x}" res_y="${res_y}" image_format="${image_format}" fov="${fov}">
       <xacro:insert_block name="calibration2" />
     </xacro:insta360_pro2_camera>
-    <xacro:insta360_pro2_camera parent="${name}_origin4_optical_frame" robot_name="${robot_name}" camera_number="3" ros_topic="${ros_topic}" update_rate="${update_rate}" res_x="${res_x}" res_y="${res_y}" image_format="${image_format}" fov="${fov}">
+    <xacro:insta360_pro2_camera parent="${name}_origin4_optical_frame" camera_number="3" ros_topic="${ros_topic}" update_rate="${update_rate}" res_x="${res_x}" res_y="${res_y}" image_format="${image_format}" fov="${fov}">
       <xacro:insert_block name="calibration3" />
     </xacro:insta360_pro2_camera>
-    <xacro:insta360_pro2_camera parent="${name}_origin5_optical_frame" robot_name="${robot_name}" camera_number="4" ros_topic="${ros_topic}" update_rate="${update_rate}" res_x="${res_x}" res_y="${res_y}" image_format="${image_format}" fov="${fov}">
+    <xacro:insta360_pro2_camera parent="${name}_origin5_optical_frame" camera_number="4" ros_topic="${ros_topic}" update_rate="${update_rate}" res_x="${res_x}" res_y="${res_y}" image_format="${image_format}" fov="${fov}">
       <xacro:insert_block name="calibration4" />
     </xacro:insta360_pro2_camera>
-    <xacro:insta360_pro2_camera parent="${name}_origin6_optical_frame" robot_name="${robot_name}" camera_number="5" ros_topic="${ros_topic}" update_rate="${update_rate}" res_x="${res_x}" res_y="${res_y}" image_format="${image_format}" fov="${fov}">
+    <xacro:insta360_pro2_camera parent="${name}_origin6_optical_frame" camera_number="5" ros_topic="${ros_topic}" update_rate="${update_rate}" res_x="${res_x}" res_y="${res_y}" image_format="${image_format}" fov="${fov}">
       <xacro:insert_block name="calibration5" />
     </xacro:insta360_pro2_camera>
-    <xacro:insta360_pro2_camera parent="${name}_center_link" robot_name="${robot_name}" camera_number="6" ros_topic="${ros_topic}" update_rate="${update_rate}" res_x="${res_x}" res_y="${res_y}" image_format="${image_format}" fov="${fov}">
+    <xacro:insta360_pro2_camera parent="${name}_center_link" camera_number="6" ros_topic="${ros_topic}" update_rate="${update_rate}" res_x="${res_x}" res_y="${res_y}" image_format="${image_format}" fov="${fov}">
       <xacro:insert_block name="calibration6" />
     </xacro:insta360_pro2_camera>
   </xacro:macro>
-  <xacro:macro name="insta360_pro2_camera" params="camera_number robot_name parent *calibration ros_topic update_rate res_x res_y image_format fov">
+  <xacro:macro name="insta360_pro2_camera" params="camera_number parent *calibration ros_topic update_rate res_x res_y image_format fov">
     <xacro:property name="camera_name" value="${name}_origin${camera_number}" />
     <joint name="${camera_name}_optical_joint" type="fixed">
@@ -114,5 +114,5 @@
     <link name="${camera_name}_link" />
     <link name="${camera_name}_optical_frame" />
-    <xacro:insta360_pro2_gazebo camera_name="${camera_name}" robot_name="${robot_name}" ros_topic="${ros_topic}" update_rate="${update_rate}" fov="${fov}" image_format="${image_format}" res_x="${res_x}" res_y="${res_y}" />
+    <xacro:insta360_pro2_gazebo camera_name="${camera_name}" ros_topic="${ros_topic}" update_rate="${update_rate}" fov="${fov}" image_format="${image_format}" res_x="${res_x}" res_y="${res_y}" />
   </xacro:macro>
 </robot>

File: urdf/os0_128.urdf.xacro (robot description, xacro)
@@ -37,14 +37,14 @@
     </link>
   </xacro:macro>
-  <xacro:macro name="os0_128" params="name robot_name parent *origin ros_topic">
-    <xacro:os0_128_advanced_parameters name="${name}" robot_name="${robot_name}" parent="${parent}" update_rate="10" horizontal_samples="512" vertical_samples="128" min_range="0.45" max_range="100">
+  <xacro:macro name="os0_128" params="name parent *origin ros_topic">
+    <xacro:os0_128_advanced_parameters name="${name}" parent="${parent}" update_rate="10" horizontal_samples="512" vertical_samples="128" min_range="0.45" max_range="100">
       <xacro:insert_block name="origin"/>
     </xacro:os0_128_advanced_parameters>
   </xacro:macro>
-  <xacro:macro name="os0_128_advanced_parameters" params="name robot_name parent *origin update_rate horizontal_samples vertical_samples min_range max_range">
+  <xacro:macro name="os0_128_advanced_parameters" params="name parent *origin update_rate horizontal_samples vertical_samples min_range max_range">
     <xacro:os0_128_model name="${name}" parent="${parent}">
       <xacro:insert_block name="origin"/>
     </xacro:os0_128_model>
-    <xacro:os0_128_gazebo name="${name}" robot_name="${robot_name}" update_rate="${update_rate}" horizontal_samples="${horizontal_samples}" vertical_samples="${vertical_samples}" min_range="${min_range}" max_range="${max_range}"/>
+    <xacro:os0_128_gazebo name="${name}" update_rate="${update_rate}" horizontal_samples="${horizontal_samples}" vertical_samples="${vertical_samples}" min_range="${min_range}" max_range="${max_range}"/>
   </xacro:macro>
 </robot>
