Commit message: changed sensors to use arg robot_name and unified topics to be $(arg robot_name)/topic
Additionally added xacro.arg for the robot_name.

This allows to initialize the robots as standalone without providing a
robot_name (for default topics /topic) and to namespace them by
providing the arg robot_name, which is done in our robot urdfs anyways.

File: urdf/realsense_d435_camera.urdf.xacro (robot description, xacro)
@@ -74,6 +74,6 @@
       </link>
     </xacro:macro>
-    <xacro:macro name="realsense_d435_camera_gazebo_plugin_macro" params="name robot_name parent frame_name:=color min_range max_range update_rate">
-      <xacro:realsense_d435_camera_gazebo name="${name}" robot_name="${robot_name}" parent="${parent}" frame_name="color" min_range="${min_range}" max_range="${max_range}" update_rate="${update_rate}"/>
+    <xacro:macro name="realsense_d435_camera_gazebo_plugin_macro" params="name parent frame_name:=color min_range max_range update_rate">
+      <xacro:realsense_d435_camera_gazebo name="${name}" parent="${parent}" frame_name="color" min_range="${min_range}" max_range="${max_range}" update_rate="${update_rate}"/>
     </xacro:macro>
     <!--
@@ -81,18 +81,18 @@
       The origin is the left infrared (depth) camera, which is also the origin of the depth image
     -->
-    <xacro:macro name="realsense_d435_camera" params="name robot_name parent *origin">
+    <xacro:macro name="realsense_d435_camera" params="name  parent *origin">
       <xacro:realsense_d435_camera_model name="${name}" parent="${parent}">
         <xacro:insert_block name="origin" />
       </xacro:realsense_d435_camera_model>
-      <xacro:realsense_d435_camera_gazebo_plugin_macro name="${name}" robot_name="${robot_name}" parent="${parent}" min_range="0.3" max_range="9.0" update_rate="20"/>
+      <xacro:realsense_d435_camera_gazebo_plugin_macro name="${name}" parent="${parent}" min_range="0.3" max_range="9.0" update_rate="20"/>
     </xacro:macro>
     <!--
       Insert the realsense with link geometry. Origin is the mounting hole at the back of the camera.
     -->
-    <xacro:macro name="realsense_d435_camera_with_mount" params="name robot_name parent *origin">
+    <xacro:macro name="realsense_d435_camera_with_mount" params="name parent *origin">
       <xacro:realsense_d435_camera_model_with_mount name="${name}" parent="${parent}">
         <xacro:insert_block name="origin" />
       </xacro:realsense_d435_camera_model_with_mount>
-      <xacro:realsense_d435_camera_gazebo_plugin_macro name="${name}" robot_name="${robot_name}" parent="${parent}" min_range="0.3" max_range="9.0" update_rate="20"/>
+      <xacro:realsense_d435_camera_gazebo_plugin_macro name="${name}" parent="${parent}" min_range="0.3" max_range="9.0" update_rate="20"/>
     </xacro:macro>
     <!--
@@ -100,27 +100,27 @@
       e.g. if the sensor is added into preexisting geometry
     -->
-    <xacro:macro name="realsense_camera_no_geom" params="name robot_name parent *origin">
+    <xacro:macro name="realsense_camera_no_geom" params="name parent *origin">
       <xacro:realsense_d435_camera_model_no_geom name="${name}" parent="${parent}">
         <xacro:insert_block name="origin" />
       </xacro:realsense_d435_camera_model_no_geom>
-      <xacro:realsense_camera_gazebo_plugin_macro name="${name}" robot_name="${robot_name}" parent="${parent}" min_range="0.3" max_range="9.0" update_rate="20"/>
+      <xacro:realsense_camera_gazebo_plugin_macro name="${name}" parent="${parent}" min_range="0.3" max_range="9.0" update_rate="20"/>
     </xacro:macro>
-    <xacro:macro name="realsense_d435_camera_no_geom_comprehensive_params" params="name robot_name parent *origin frame_name:=color min_range max_range update_rate">
+    <xacro:macro name="realsense_d435_camera_no_geom_comprehensive_params" params="name parent *origin frame_name:=color min_range max_range update_rate">
       <xacro:realsense_d435_camera_model_no_geom name="${name}" parent="${parent}">
         <xacro:insert_block name="origin" />
       </xacro:realsense_d435_camera_model_no_geom>
-      <xacro:realsense_camera_gazebo_plugin_macro name="${name}" robot_name="${robot_name}" parent="${parent}" image_topic="${image_topic}" depth_topic="${depth_topic}" depth_points_topic="${depth_points_topic}" frame_name="${frame_name}" min_range="${min_range}" max_range="${max_range}" update_rate="${update_rate}"/>
+      <xacro:realsense_camera_gazebo_plugin_macro name="${name}" parent="${parent}" image_topic="${image_topic}" depth_topic="${depth_topic}" depth_points_topic="${depth_points_topic}" frame_name="${frame_name}" min_range="${min_range}" max_range="${max_range}" update_rate="${update_rate}"/>
     </xacro:macro>
-    <xacro:macro name="realsense_d435_camera_comprehensive_params" params="name robot_name parent *origin frame_name:=color min_range:=0.3 max_range:=9.0 update_rate:=20">
+    <xacro:macro name="realsense_d435_camera_comprehensive_params" params="name parent *origin frame_name:=color min_range:=0.3 max_range:=9.0 update_rate:=20">
       <xacro:realsense_d435_camera_model name="${name}" parent="${parent}">
         <xacro:insert_block name="origin" />
       </xacro:realsense_d435_camera_model>
-      <xacro:realsense_d435_camera_gazebo_plugin_macro name="${name}" robot_name="${robot_name}" parent="${parent}" frame_name="${frame_name}" min_range="${min_range}" max_range="${max_range}" update_rate="${update_rate}"/>
+      <xacro:realsense_d435_camera_gazebo_plugin_macro name="${name}" parent="${parent}" frame_name="${frame_name}" min_range="${min_range}" max_range="${max_range}" update_rate="${update_rate}"/>
     </xacro:macro>
-    <xacro:macro name="realsense_d435_camera_with_mount_comprehensive_params" params="name robot_name parent *origin frame_name:=color min_range:=0.3 max_range:=9.0 update_rate:=20">
+    <xacro:macro name="realsense_d435_camera_with_mount_comprehensive_params" params="name parent *origin frame_name:=color min_range:=0.3 max_range:=9.0 update_rate:=20">
       <xacro:realsense_d435_camera_model_with_mount name="${name}" parent="${parent}">
         <xacro:insert_block name="origin" />
       </xacro:realsense_d435_camera_model_with_mount>
-      <xacro:realsense_d435_camera_gazebo_plugin_macro name="${name}" robot_name="${robot_name}" parent="${parent}" frame_name="${frame_name}" min_range="${min_range}" max_range="${max_range}" update_rate="${update_rate}"/>
+      <xacro:realsense_d435_camera_gazebo_plugin_macro name="${name}" parent="${parent}" frame_name="${frame_name}" min_range="${min_range}" max_range="${max_range}" update_rate="${update_rate}"/>
     </xacro:macro>
   </robot>

Commit message: added default value for semantic segmentation

File: gazebo/astra_stereo_s_u3.gazebo.xacro (robot description, xacro)
@@ -2,4 +2,5 @@
 <robot xmlns:xacro="http://ros.org/wiki/xacro">
 	<xacro:property name="M_PI" value="3.14159"/>
+	<xacro:arg name="semantic_segmentation" default="false"/>
 	<xacro:macro name="orbbec_astra_stereo_s_u3_gazebo" params="name:=default">
 		<gazebo reference="${name}_link">

File: gazebo/orbbec_astra2.gazebo.xacro (robot description, xacro)
@@ -2,5 +2,6 @@
 <robot xmlns:xacro="http://ros.org/wiki/xacro">
 	<xacro:property name="M_PI" value="3.14159"/>
-	<xacro:macro name="orbbec_astra2_gazebo" params="name:=default">
+	<xacro:arg name="semantic_segmentation" default="false"/>
+	<xacro:macro name="orbbec_astra2_gazebo" params="name:=default semantic_segmentation:=false">
 		<gazebo reference="${name}_link">
 			<sensor type="camera" name="${name}_rgb">

Commit message: changed sensors to use arg robot_name and unified topics to be $(arg robot_name)/topic
Additionally added xacro.arg for the robot_name.

This allows to initialize the robots as standalone without providing a
robot_name (for default topics /topic) and to namespace them by
providing the arg robot_name, which is done in our robot urdfs anyways.

File: gazebo/astra_stereo_s_u3.gazebo.xacro (robot description, xacro)
@@ -3,4 +3,5 @@
 	<xacro:property name="M_PI" value="3.14159"/>
 	<xacro:arg name="semantic_segmentation" default="false"/>
+	<xacro:arg name="robot_name" default=""/>
 	<xacro:macro name="orbbec_astra_stereo_s_u3_gazebo" params="name:=default">
 		<gazebo reference="${name}_link">
@@ -56,6 +57,6 @@
 			<xacro:if value="$(arg semantic_segmentation)">
 				<sensor name="astra2_${name}_segmentation_camera" type="segmentation">
-					<topic>/$(arg robot_name)/${name}/segmentation</topic>
-					<gz_frame_id>${name}_link</gz_frame_id>
+					<topic>$(arg robot_name)/astra2_${name}/segmentation</topic>
+					<gz_frame_id>astra2_${name}_link</gz_frame_id>
 					<camera>
 						<optical_frame_id>${name}_optical_frame</optical_frame_id>

File: gazebo/insta360_air.gazebo.xacro (robot description, xacro)
@@ -2,4 +2,5 @@
 <robot xmlns:xacro="http://ros.org/wiki/xacro">
     <xacro:property name="M_PI" value="3.14159"/>
+    <xacro:arg name="robot_name" default=""/>
     <xacro:macro name="insta360_air_gazebo" params="name:=default">
         <gazebo reference="${name}_left_optical_frame">

File: gazebo/livox_mid360.gazebo.xacro (robot description, xacro)
@@ -2,4 +2,5 @@
 <robot xmlns:xacro="http://ros.org/wiki/xacro">
 	<xacro:property name="M_PI" value="3.14159"/>
+	<xacro:arg name="robot_name" default=""/>
 	<xacro:macro name="livox_mid360_gazebo" params="visualize:=True name:=default">
 		<gazebo reference="${name}_laser_frame">

File: gazebo/orbbec_astra2.gazebo.xacro (robot description, xacro)
@@ -3,4 +3,5 @@
 	<xacro:property name="M_PI" value="3.14159"/>
 	<xacro:arg name="semantic_segmentation" default="false"/>
+	<xacro:arg name="robot_name" default=""/>
 	<xacro:macro name="orbbec_astra2_gazebo" params="name:=default semantic_segmentation:=false">
 		<gazebo reference="${name}_link">

File: urdf/flir_a65_camera.urdf.xacro (robot description, xacro)
@@ -30,9 +30,9 @@
     </gazebo>
   </xacro:macro>
-  <xacro:macro name="flir_a65_camera" params="name parent robot_name *origin">
+  <xacro:macro name="flir_a65_camera" params="name parent *origin">
     <xacro:flir_a65_camera_model name="${name}" parent="${parent}">
       <xacro:insert_block name="origin" />
     </xacro:flir_a65_camera_model>
-    <xacro:flir_a65_camera_gazebo robot_name="${robot_name}"/>
+    <xacro:flir_a65_camera_gazebo name="${name}"/>
   </xacro:macro>
 </robot>

File: urdf/generic_camera.urdf.xacro (robot description, xacro)
@@ -3,5 +3,5 @@
   <xacro:include filename="$(find hector_sensors_description)/gazebo/generic_camera.gazebo.xacro"/>
   <xacro:property name="M_PI" value="3.1415926535897931" />
-  <xacro:macro name="generic_camera" params="name parent robot_name *origin ros_topic cam_info_topic update_rate res_x res_y image_format hfov">
+  <xacro:macro name="generic_camera" params="name parent *origin ros_topic cam_info_topic update_rate res_x res_y image_format hfov">
     <joint name="${name}_joint" type="fixed">
       <xacro:insert_block name="origin" />
@@ -37,3 +37,5 @@
     </joint>
     <link name="${name}_optical_frame"/>
+    <xacro:generic_camera_gazebo name="${name}" update_rate="${update_rate}" res_x="${res_x}" res_y="${res_y}" hfov="${hfov}" image_format="${image_format}"/>
+  </xacro:macro>
 </robot>

Commit message: new feature to publish frames via static tf publishers

File: gazebo/astra_stereo_s_u3.gazebo.xacro (robot description, xacro)
@@ -4,5 +4,5 @@
 	<xacro:arg name="semantic_segmentation" default="false"/>
 	<xacro:macro name="orbbec_astra_stereo_s_u3_gazebo" params="name:=default">
-		<gazebo reference="${name}_link">
+	  <gazebo reference="${name}_link">
 			<sensor type="camera" name="${name}_rgb">
 				<always_on>true</always_on>
@@ -10,8 +10,8 @@
 				<update_rate>15</update_rate>
 				<topic>/$(arg robot_name)/${name}/rgb/image_raw</topic>
-				<gz_frame_id>${name}_rgb_link</gz_frame_id>
+				<gz_frame_id>${name}_color_frame</gz_frame_id>
 				<camera name="astra_stereo_s_u3_${name}_camera">
 					<camera_info_topic>/$(arg robot_name)/${name}/rgb/camera_info</camera_info_topic>
-					<optical_frame_id>${name}_rgb_optical_frame</optical_frame_id>
+					<optical_frame_id>${name}_color_optical_frame</optical_frame_id>
 					<horizontal_fov>${90.0 * M_PI/180.0}</horizontal_fov>
 					<image>
@@ -31,5 +31,5 @@
 				<update_rate>15</update_rate>
 				<topic>/$(arg robot_name)/${name}/depth/image_raw</topic>
-				<gz_frame_id>${name}_depth_link</gz_frame_id>
+				<gz_frame_id>${name}_depth_frame</gz_frame_id>
 				<camera>
 					<camera_info_topic>/$(arg robot_name)/${name}/depth/camera_info</camera_info_topic>
@@ -59,5 +59,5 @@
 					<gz_frame_id>${name}_link</gz_frame_id>
 					<camera>
-						<optical_frame_id>${name}_optical_frame</optical_frame_id>
+						<optical_frame_id>${name}_color_optical_frame</optical_frame_id>
 						<segmentation_type>instance</segmentation_type>
 						<horizontal_fov>${90.0 * M_PI/180.0}</horizontal_fov>

File: urdf/astra_stereo_s_u3.urdf.xacro (robot description, xacro)
@@ -32,33 +32,5 @@
             </collision>
         </link>
-        <!-- Camera RGB sensor -->
-        <link name="${name}_rgb_link"/>
-        <joint name="${name}_rgb_joint" type="fixed">
-            <origin xyz="0.014 0.01 0" rpy="0 0 0" />
-            <parent link="${name}_link" />
-            <child link="${name}_rgb_link" />
-        </joint>
-        <!-- Camera Depth sensor -->
-        <!-- Assuming the depth image is published in the same frame as the rgb image -->
-        <link name="${name}_depth_link"/>
-        <joint name="${name}_depth_joint" type="fixed">
-            <origin xyz="0.014 0.01 0" rpy="0 0 0" />
-            <parent link="${name}_link" />
-            <child link="${name}_depth_link" />
-        </joint>
-        <!-- Camera Optical Frame -->
-        <link name="${name}_rgb_optical_frame"/>
-        <joint name="${name}_rgb_optical_joint" type="fixed">
-            <origin xyz="0 0 0" rpy="-${M_PI/2.0} 0 -${M_PI/2.0}" />
-            <parent link="${name}_rgb_link" />
-            <child link="${name}_rgb_optical_frame" />
-        </joint>
-        <!-- Camera Depth Optical Frame -->
-        <link name="${name}_depth_optical_frame"/>
-        <joint name="${name}_depth_optical_joint" type="fixed">
-            <origin xyz="0 0 0" rpy="-${M_PI/2.0} 0 -${M_PI/2.0}" />
-            <parent link="${name}_depth_link" />
-            <child link="${name}_depth_optical_frame" />
-        </joint>
+    <!-- optical frames are published by driver, use launch file for simulation -->
     </xacro:macro>
 </robot>

Commit message: adjusted gemini2 and astra_stereo_s_u3 to have correct rgbd frames

File: gazebo/astra_stereo_s_u3.gazebo.xacro (robot description, xacro)
@@ -14,8 +14,9 @@
 					<camera_info_topic>/$(arg robot_name)/${name}/rgb/camera_info</camera_info_topic>
 					<optical_frame_id>${name}_rgb_optical_frame</optical_frame_id>
-					<horizontal_fov>${90.0 * M_PI/180.0}</horizontal_fov>
+					<horizontal_fov>${71.5 * M_PI/180.0}</horizontal_fov>
+					<vertical_fov>${56.7 * M_PI/180.0}</vertical_fov>
 					<image>
 						<format>R8G8B8</format>
-						<width>720</width>
+						<width>640</width>
 						<height>480</height>
 					</image>
@@ -26,4 +27,5 @@
 				</camera>
 			</sensor>
+            <!-- Depth Image of real camera is already registered to RGB image and has the same camera info -->
 			<sensor type="depth_camera" name="${name}_depth">
 				<always_on>true</always_on>
@@ -35,5 +37,6 @@
 					<camera_info_topic>/$(arg robot_name)/${name}/depth/camera_info</camera_info_topic>
 					<optical_frame_id>${name}_depth_optical_frame</optical_frame_id>
-					<horizontal_fov>1.047</horizontal_fov>
+					<horizontal_fov>${71.5 * M_PI/180.0}</horizontal_fov>
+                    <vertical_fov>${56.7 * M_PI/180.0}</vertical_fov>
 					<image>
 						<format>R_FLOAT32</format>
@@ -43,5 +46,5 @@
 					<depth_camera>
 						<clip>
-							<near>0.1</near>
+							<near>0.25</near>
 							<far>10.0</far>
 						</clip>

File: gazebo/orbbec_gemini2.gazebo.xacro (robot description, xacro)
@@ -10,12 +10,13 @@
 				<update_rate>15</update_rate>
 				<topic>/$(arg robot_name)/${name}/rgb/image_raw</topic>
-				<gz_frame_id>${name}_rgb_link</gz_frame_id>
+				<gz_frame_id>${name}_rgb_frame</gz_frame_id>
 				<camera name="${name}_camera">
 					<camera_info_topic>/$(arg robot_name)/${name}/rgb/camera_info</camera_info_topic>
 					<optical_frame_id>${name}_rgb_optical_frame</optical_frame_id>
-					<horizontal_fov>${90.0 * M_PI/180.0}</horizontal_fov>
+					<horizontal_fov>${63.0 * M_PI/180.0}</horizontal_fov>
+					<vertical_fov>${50.0 * M_PI/180.0}</vertical_fov>
 					<image>
 						<format>R8G8B8</format>
-						<width>720</width>
+						<width>640</width>
 						<height>480</height>
 					</image>
@@ -26,4 +27,5 @@
 				</camera>
 			</sensor>
+            <!-- Depth Image of real camera is already registered to RGB image and has the same camera info -->
 			<sensor type="depth_camera" name="${name}_depth">
 				<always_on>true</always_on>
@@ -31,9 +33,10 @@
 				<update_rate>15</update_rate>
 				<topic>/$(arg robot_name)/${name}/depth/image_raw</topic>
-				<gz_frame_id>${name}_depth_link</gz_frame_id>
+				<gz_frame_id>${name}_depth_frame</gz_frame_id>
 				<camera>
 					<camera_info_topic>/$(arg robot_name)/${name}/depth/camera_info</camera_info_topic>
 					<optical_frame_id>${name}_depth_optical_frame</optical_frame_id>
-					<horizontal_fov>1.047</horizontal_fov>
+					<horizontal_fov>${63.0 * M_PI/180.0}</horizontal_fov>
+                    <vertical_fov>${50.0 * M_PI/180.0}</vertical_fov>
 					<image>
 						<format>R_FLOAT32</format>
@@ -43,5 +46,5 @@
 					<depth_camera>
 						<clip>
-							<near>0.1</near>
+							<near>0.15</near>
 							<far>10.0</far>
 						</clip>
@@ -57,15 +60,16 @@
 				<sensor name="gemini2_${name}_segmentation_camera" type="segmentation">
 					<topic>/$(arg robot_name)/${name}/segmentation</topic>
-					<gz_frame_id>${name}_link</gz_frame_id>
+					<gz_frame_id>${name}_rgb_link</gz_frame_id>
 					<camera>
-						<optical_frame_id>${name}_optical_frame</optical_frame_id>
+						<optical_frame_id>${name}_rgb_optical_frame</optical_frame_id>
 						<segmentation_type>instance</segmentation_type>
-						<horizontal_fov>${90.0 * M_PI/180.0}</horizontal_fov>
+					    <horizontal_fov>${63.0 * M_PI/180.0}</horizontal_fov>
+					    <vertical_fov>${50.0 * M_PI/180.0}</vertical_fov>
 						<image>
-							<width>720</width>
+							<width>640</width>
 							<height>480</height>
 						</image>
 						<clip>
-							<near>0.1</near>
+							<near>0.05</near>
 							<far>10</far>
 						</clip>

File: urdf/orbbec_gemini2.urdf.xacro (robot description, xacro)
@@ -32,30 +32,5 @@
             </collision>
         </link>
-        <!-- Camera RGB sensor -->
-        <link name="${name}_rgb_link"/>
-        <joint name="${name}_rgb_joint" type="fixed">
-            <origin xyz="0.01682 0.010995 0" rpy="0 0 0" />
-            <parent link="${name}_link" />
-            <child link="${name}_rgb_link" />
-        </joint>
-        <!-- Optical Frame for ros (in z direction) -->
-        <link name="${name}_rgb_optical_frame"/>
-        <joint name="${name}_rgb_optical_joint" type="fixed">
-            <origin xyz="0 0 0" rpy="-${M_PI/2.0} 0 -${M_PI/2.0}" />
-            <parent link="${name}_rgb_link" />
-            <child link="${name}_rgb_optical_frame" />
-        </joint>
-        <link name="${name}_depth_link"/>
-        <joint name="${name}_depth_joint" type="fixed">
-            <origin xyz="0.01491 0.025 0" rpy="0 0 0" />
-            <parent link="${name}_link" />
-            <child link="${name}_depth_link" />
-        </joint>
-        <link name="${name}_depth_optical_frame"/>
-        <joint name="${name}_depth_optical_joint" type="fixed">
-            <origin xyz="0 0 0" rpy="-${M_PI/2.0} 0 -${M_PI/2.0}" />
-            <parent link="${name}_depth_link" />
-            <child link="${name}_depth_optical_frame" />
-        </joint>
+    <!-- optical frames are published by driver, use launch file for simulation -->
     </xacro:macro>
 </robot>
