Commit message: Added extended ci

File: gazebo/astra_stereo_s_u3.gazebo.xacro (robot description, xacro)
@@ -1,7 +1,6 @@
-<?xml version="1.0"?>
+<?xml version="1.0" encoding="UTF-8"?>
 <robot xmlns:xacro="http://ros.org/wiki/xacro">
-  <xacro:arg name="semantic_segmentation" default="false" />
-  <xacro:macro name="orbbec_astra_stereo_s_u3_gazebo"
-    params="name:=default semantic_segmentation:=false">
+  <xacro:arg name="semantic_segmentation" default="false"/>
+  <xacro:macro name="orbbec_astra_stereo_s_u3_gazebo" params="name:=default semantic_segmentation:=false">
     <gazebo reference="${name}_link">
       <sensor type="camera" name="${name}_rgb">

File: gazebo/flir_a65_camera.gazebo.xacro (robot description, xacro)
@@ -1,26 +1,26 @@
-<?xml version="1.0"?>
+<?xml version="1.0" encoding="UTF-8"?>
 <robot xmlns:xacro="http://ros.org/wiki/xacro">
-    <xacro:macro name="flir_a65_camera_gazebo" params="robot_name">
-        <gazebo reference="${name}_frame">
-            <sensor type="thermal" name="${name}_thermal_cam">
-                <update_rate>9</update_rate>
-                <always_on>true</always_on>
-                <topic>${robot_name}/thermal_camera/image_raw</topic>
-                <gz_frame_id>${name}_optical_frame</gz_frame_id>
-                <camera name="${name}">
-                    <camera_info_topic>${robot_name}/${name}/camera_info</camera_info_topic>
-                    <horizontal_fov>${45.0*pi/180.0}</horizontal_fov>
-                    <image>
-                        <format>R8G8B8</format>
-                        <width>640</width>
-                        <height>512</height>
-                    </image>
-                    <clip>
-                        <near>0.01</near>
-                        <far>10</far>
-                    </clip>
-                </camera>
-            </sensor>
-        </gazebo>
-    </xacro:macro>
+  <xacro:macro name="flir_a65_camera_gazebo" params="robot_name">
+    <gazebo reference="${name}_frame">
+      <sensor type="thermal" name="${name}_thermal_cam">
+        <update_rate>9</update_rate>
+        <always_on>true</always_on>
+        <topic>${robot_name}/thermal_camera/image_raw</topic>
+        <gz_frame_id>${name}_optical_frame</gz_frame_id>
+        <camera name="${name}">
+          <camera_info_topic>${robot_name}/${name}/camera_info</camera_info_topic>
+          <horizontal_fov>${45.0*pi/180.0}</horizontal_fov>
+          <image>
+            <format>R8G8B8</format>
+            <width>640</width>
+            <height>512</height>
+          </image>
+          <clip>
+            <near>0.01</near>
+            <far>10</far>
+          </clip>
+        </camera>
+      </sensor>
+    </gazebo>
+  </xacro:macro>
 </robot>

File: gazebo/generic_camera.gazebo.xacro (robot description, xacro)
@@ -1,6 +1,5 @@
-<?xml version="1.0"?>
+<?xml version="1.0" encoding="UTF-8"?>
 <robot xmlns:xacro="http://ros.org/wiki/xacro">
-  <xacro:macro name="generic_camera_gazebo"
-    params="name robot_name update_rate res_x res_y hfov image_format">
+  <xacro:macro name="generic_camera_gazebo" params="name robot_name update_rate res_x res_y hfov image_format">
     <gazebo reference="${name}_link">
       <sensor type="camera" name="${name}_camera_sensor">

File: gazebo/generic_wide_angle_camera.gazebo.xacro (robot description, xacro)
@@ -1,6 +1,5 @@
-<?xml version="1.0"?>
+<?xml version="1.0" encoding="UTF-8"?>
 <robot xmlns:xacro="http://ros.org/wiki/xacro">
-  <xacro:macro name="generic_wide_angle_camera_gazebo"
-    params="name robot_name update_rate res_x res_y hfov image_format">
+  <xacro:macro name="generic_wide_angle_camera_gazebo" params="name robot_name update_rate res_x res_y hfov image_format">
     <gazebo reference="${name}_link">
       <sensor type="wideanglecamera" name="${name}_camera_sensor">

File: gazebo/insta360_air.gazebo.xacro (robot description, xacro)
@@ -1,3 +1,3 @@
-<?xml version="1.0"?>
+<?xml version="1.0" encoding="UTF-8"?>
 <robot xmlns:xacro="http://ros.org/wiki/xacro">
   <xacro:macro name="insta360_air_gazebo" params="name:=default">

File: gazebo/insta360_pro2.gazebo.xacro (robot description, xacro)
@@ -1,6 +1,5 @@
-<?xml version="1.0"?>
+<?xml version="1.0" encoding="UTF-8"?>
 <robot xmlns:xacro="http://ros.org/wiki/xacro">
-  <xacro:macro name="insta360_pro2_gazebo"
-    params="camera_name robot_name ros_topic update_rate fov image_format res_x res_y">
+  <xacro:macro name="insta360_pro2_gazebo" params="camera_name robot_name ros_topic update_rate fov image_format res_x res_y">
     <gazebo reference="${camera_name}_link">
       <sensor type="wideanglecamera" name="${camera_name}_camera_sensor">

File: gazebo/intel_realsense_d435.gazebo.xacro (robot description, xacro)
@@ -1,7 +1,6 @@
-<?xml version="1.0"?>
+<?xml version="1.0" encoding="UTF-8"?>
 <robot xmlns:xacro="http://ros.org/wiki/xacro">
-  <xacro:arg name="semantic_segmentation" default="false" />
-  <xacro:macro name="intel_realsense_d435_gazebo"
-    params="name:=default semantic_segmentation:=false">
+  <xacro:arg name="semantic_segmentation" default="false"/>
+  <xacro:macro name="intel_realsense_d435_gazebo" params="name:=default semantic_segmentation:=false">
     <gazebo reference="${name}_link">
       <sensor type="camera" name="${name}_rgb">

File: gazebo/livox_mid360.gazebo.xacro (robot description, xacro)
@@ -1,8 +1,8 @@
-<?xml version="1.0"?>
+<?xml version="1.0" encoding="UTF-8"?>
 <robot xmlns:xacro="http://ros.org/wiki/xacro">
   <xacro:macro name="livox_mid360_gazebo" params="visualize:=True name:=default">
     <gazebo reference="${name}_laser_frame">
-      <sensor name='gpu_lidar_${name}' type='gpu_lidar'>
-        <pose relative_to='${name}_laser_frame'>0 0 0 0 0 0</pose>
+      <sensor name="gpu_lidar_${name}" type="gpu_lidar">
+        <pose relative_to="${name}_laser_frame">0 0 0 0 0 0</pose>
         <topic>/$(arg robot_name)/${name}</topic>
         <update_rate>10</update_rate>

File: gazebo/orbbec_astra2.gazebo.xacro (robot description, xacro)
@@ -1,5 +1,5 @@
-<?xml version="1.0"?>
+<?xml version="1.0" encoding="UTF-8"?>
 <robot xmlns:xacro="http://ros.org/wiki/xacro">
-  <xacro:arg name="semantic_segmentation" default="false" />
+  <xacro:arg name="semantic_segmentation" default="false"/>
   <xacro:macro name="orbbec_astra2_gazebo" params="name:=default semantic_segmentation:=false">
     <gazebo reference="${name}_link">

File: gazebo/orbbec_gemini2.gazebo.xacro (robot description, xacro)
@@ -1,5 +1,5 @@
-<?xml version="1.0"?>
+<?xml version="1.0" encoding="UTF-8"?>
 <robot xmlns:xacro="http://ros.org/wiki/xacro">
-  <xacro:arg name="semantic_segmentation" default="false" />
+  <xacro:arg name="semantic_segmentation" default="false"/>
   <xacro:macro name="orbbec_gemini2_gazebo" params="name:=default semantic_segmentation:=false">
     <gazebo reference="${name}_link">

File: gazebo/os0_128.gazebo.xacro (robot description, xacro)
@@ -1,9 +1,8 @@
-<?xml version="1.0"?>
+<?xml version="1.0" encoding="UTF-8"?>
 <robot xmlns:xacro="http://ros.org/wiki/xacro">
-  <xacro:macro name="os0_128_gazebo"
-    params="name update_rate horizontal_samples vertical_samples min_range max_range min_angle max_angle">
+  <xacro:macro name="os0_128_gazebo" params="name update_rate horizontal_samples vertical_samples min_range max_range min_angle max_angle">
     <gazebo reference="${name}_laser_frame">
       <sensor name="gpu_lidar_${name}" type="gpu_lidar">
-        <pose relative_to='${name}_laser_frame'>0 0 0 0 0 0</pose>
+        <pose relative_to="${name}_laser_frame">0 0 0 0 0 0</pose>
         <topic>/$(arg robot_name)/${name}</topic>
         <update_rate>${update_rate}</update_rate>

File: gazebo/seek_thermal_xr.gazebo.xacro (robot description, xacro)
@@ -1,3 +1,3 @@
-<?xml version="1.0"?>
+<?xml version="1.0" encoding="UTF-8"?>
 <robot xmlns:xacro="http://ros.org/wiki/xacro">
   <xacro:macro name="seek_thermal_xr_gazebo" params="name:=default">

File: urdf/arducam_wideangle_v2.urdf.xacro (robot description, xacro)
@@ -1,8 +1,8 @@
-<?xml version="1.0"?>
+<?xml version="1.0" encoding="UTF-8"?>
 <robot xmlns:xacro="http://www.ros.org/wiki/xacro">
   <xacro:include filename="$(find hector_sensors_description)/gazebo/generic_wide_angle_camera.gazebo.xacro"/>
   <xacro:macro name="arducam_wideangle_v2" params="name parent robot_name *origin ros_topic cam_info_topic update_rate res_x res_y image_format hfov">
     <joint name="${name}_joint" type="fixed">
-      <xacro:insert_block name="origin" />
+      <xacro:insert_block name="origin"/>
       <parent link="${parent}"/>
       <child link="${name}_link"/>
@@ -10,25 +10,25 @@
     <link name="${name}_link">
       <visual>
-        <origin xyz="0 0 0" rpy="0 0 0" />
+        <origin xyz="0 0 0" rpy="0 0 0"/>
         <geometry>
-          <mesh filename="package://hector_sensors_description/meshes/arducam_wideangle_v2/arducam_wideangle_v2.glb" />
+          <mesh filename="package://hector_sensors_description/meshes/arducam_wideangle_v2/arducam_wideangle_v2.glb"/>
         </geometry>
       </visual>
       <collision>
-        <origin xyz="0.006 -0.0001 0" rpy="0 0 0" />
+        <origin xyz="0.006 -0.0001 0" rpy="0 0 0"/>
         <geometry>
-          <box size="0.0209 0.0319 0.032" />
+          <box size="0.0209 0.0319 0.032"/>
         </geometry>
       </collision>
       <inertial>
-        <mass value="0.001" />
-        <origin xyz="0 0 0" rpy="0 0 0" />
-        <inertia ixx="0.0001" ixy="0" ixz="0" iyy="0.0001" iyz="0" izz="0.0001" />
+        <mass value="0.001"/>
+        <origin xyz="0 0 0" rpy="0 0 0"/>
+        <inertia ixx="0.0001" ixy="0" ixz="0" iyy="0.0001" iyz="0" izz="0.0001"/>
       </inertial>
     </link>
     <link name="${name}_optical_frame"/>
     <joint name="${name}_optical_joint" type="fixed">
-      <origin xyz="0.016 0 0" rpy="${-pi/2} 0 ${-pi/2}" />
-      <parent link="${name}_link" />
+      <origin xyz="0.016 0 0" rpy="${-pi/2} 0 ${-pi/2}"/>
+      <parent link="${name}_link"/>
       <child link="${name}_optical_frame"/>
     </joint>

File: urdf/astra_stereo_s_u3.urdf.xacro (robot description, xacro)
@@ -1,36 +1,33 @@
-<?xml version="1.0"?>
+<?xml version="1.0" encoding="UTF-8"?>
 <!-- datasheet:
 https://www.sodavision.com/wp-content/uploads/2023/12/2023.07-astra-stereo-s-u3-datasheet-_v2.0_en.pdf -->
 <robot xmlns:xacro="http://ros.org/wiki/xacro">
-  <xacro:include filename="$(find hector_xacro_tools)/urdf/inertia_tensors.urdf.xacro" />
-  <xacro:include filename="$(find hector_sensors_description)/gazebo/astra_stereo_s_u3.gazebo.xacro" />
+  <xacro:include filename="$(find hector_xacro_tools)/urdf/inertia_tensors.urdf.xacro"/>
+  <xacro:include filename="$(find hector_sensors_description)/gazebo/astra_stereo_s_u3.gazebo.xacro"/>
   <xacro:macro name="orbbec_astra_stereo_s_u3" params="name *origin *parent">
-    <xacro:orbbec_astra_stereo_s_u3_gazebo name="${name}" />
-    <xacro:property name="orbbec_astra_stereo_s_u3_mass" value="0.05" /> <!-- estimated, needs to be checked -->
-    <xacro:property name="orbbec_astra_stereo_s_u3_length" value="0.0653" />
-    <xacro:property name="orbbec_astra_stereo_s_u3_width" value="0.0123" />
-    <xacro:property name="orbbec_astra_stereo_s_u3_height" value="0.0225" />
+    <xacro:orbbec_astra_stereo_s_u3_gazebo name="${name}"/>
+    <xacro:property name="orbbec_astra_stereo_s_u3_mass" value="0.05"/>
+    <!-- estimated, needs to be checked -->
+    <xacro:property name="orbbec_astra_stereo_s_u3_length" value="0.0653"/>
+    <xacro:property name="orbbec_astra_stereo_s_u3_width" value="0.0123"/>
+    <xacro:property name="orbbec_astra_stereo_s_u3_height" value="0.0225"/>
     <joint name="${name}_joint" type="fixed">
-      <child link="${name}_link" />
-      <xacro:insert_block name="origin" />
-      <xacro:insert_block name="parent" />
+      <child link="${name}_link"/>
+      <xacro:insert_block name="origin"/>
+      <xacro:insert_block name="parent"/>
     </joint>
     <!-- Camera base -->
     <link name="${name}_link">
-      <xacro:inertial_cuboid
-        mass="${orbbec_astra_stereo_s_u3_mass}"
-        x_length="${orbbec_astra_stereo_s_u3_width}"
-        y_length="${orbbec_astra_stereo_s_u3_length}"
-        z_length="${orbbec_astra_stereo_s_u3_height}" />
+      <xacro:inertial_cuboid mass="${orbbec_astra_stereo_s_u3_mass}" x_length="${orbbec_astra_stereo_s_u3_width}" y_length="${orbbec_astra_stereo_s_u3_length}" z_length="${orbbec_astra_stereo_s_u3_height}"/>
       <visual>
-        <origin xyz="0 0 0" rpy="0 0 0" />
+        <origin xyz="0 0 0" rpy="0 0 0"/>
         <geometry>
-          <mesh filename="package://hector_sensors_description/meshes/orbbec_astra_stereo_s_u3/orbbec_astra_stereo_s_u3.dae" />
+          <mesh filename="package://hector_sensors_description/meshes/orbbec_astra_stereo_s_u3/orbbec_astra_stereo_s_u3.dae"/>
         </geometry>
       </visual>
       <collision>
-        <origin xyz="0.006 0 0.001" rpy="0 0 0" />
+        <origin xyz="0.006 0 0.001" rpy="0 0 0"/>
         <geometry>
-          <box size="0.021 0.07 0.025" />
+          <box size="0.021 0.07 0.025"/>
         </geometry>
       </collision>

File: urdf/enrich_radiation_sensor.urdf.xacro (robot description, xacro)
@@ -1,11 +1,9 @@
-<?xml version="1.0"?>
+<?xml version="1.0" encoding="UTF-8"?>
 <!-- A rough description of a thermo scientific personal radiation detector packed in a box -->
 <robot xmlns:xacro="http://ros.org/wiki/xacro">
-  <xacro:property name="rs_size_x" value="0.103" />
-  <xacro:property name="rs_size_y" value="0.078" />
-  <xacro:property name="rs_size_z" value="0.049" />
-  <xacro:macro
-    name="radiation_sensor"
-    params="name:='radiation_sensor' *origin parent">
+  <xacro:property name="rs_size_x" value="0.103"/>
+  <xacro:property name="rs_size_y" value="0.078"/>
+  <xacro:property name="rs_size_z" value="0.049"/>
+  <xacro:macro name="radiation_sensor" params="name:='radiation_sensor' *origin parent">
     <joint name="${name}_base_joint" type="fixed">
       <xacro:insert_block name="origin"/>
@@ -15,22 +13,22 @@
     <link name="${name}_base_link"/>
     <joint name="${name}_joint" type="fixed">
-      <origin xyz="0 0 ${rs_size_z / 2}" />
-      <parent link="${name}_base_link" />
-      <child link="radiation_sensor_link" />
+      <origin xyz="0 0 ${rs_size_z / 2}"/>
+      <parent link="${name}_base_link"/>
+      <child link="radiation_sensor_link"/>
     </joint>
     <link name="${name}_link">
       <visual>
-        <origin xyz="0 0 0" rpy="0 0 0" />
+        <origin xyz="0 0 0" rpy="0 0 0"/>
         <geometry>
-          <box size="${rs_size_x} ${rs_size_y} ${rs_size_z}" />
+          <box size="${rs_size_x} ${rs_size_y} ${rs_size_z}"/>
         </geometry>
         <material name="Black">
-          <color rgba="0.01 0.01 0.01 1.0" />
+          <color rgba="0.01 0.01 0.01 1.0"/>
         </material>
       </visual>
       <collision>
-        <origin xyz="0 0 0" rpy="0 0 0" />
+        <origin xyz="0 0 0" rpy="0 0 0"/>
         <geometry>
-          <box size="${rs_size_x} ${rs_size_y} ${rs_size_z}" />
+          <box size="${rs_size_x} ${rs_size_y} ${rs_size_z}"/>
         </geometry>
       </collision>

File: urdf/flir_a65_camera.urdf.xacro (robot description, xacro)
@@ -1,29 +1,29 @@
-<?xml version="1.0"?>
+<?xml version="1.0" encoding="UTF-8"?>
 <robot xmlns:xacro="http://www.ros.org/wiki/xacro">
-  <xacro:include filename="$(find hector_xacro_tools)/urdf/sensor_macros.urdf.xacro" />
+  <xacro:include filename="$(find hector_xacro_tools)/urdf/sensor_macros.urdf.xacro"/>
   <xacro:include filename="$(find hector_sensors_description)/gazebo/flir_a65_camera.gazebo.xacro"/>
   <!--Dimensions taken from http://www.flir.com/automation/display/?id=56341-->
   <xacro:macro name="flir_a65_camera_model" params="name parent *origin">
     <joint name="${name}_joint" type="fixed">
-      <xacro:insert_block name="origin" />
+      <xacro:insert_block name="origin"/>
       <parent link="${parent}"/>
       <child link="${name}_frame"/>
     </joint>
     <link name="${name}_frame">
-      <xacro:inertial_sphere mass="0.21" diameter="0.07" />
+      <xacro:inertial_sphere mass="0.21" diameter="0.07"/>
       <visual>
-        <origin xyz="0 0 0" rpy="0 0 0" />
+        <origin xyz="0 0 0" rpy="0 0 0"/>
         <geometry>
-          <mesh filename="package://hector_sensors_description/meshes/flir_ax5_camera/flir_ax5_camera.glb" />
+          <mesh filename="package://hector_sensors_description/meshes/flir_ax5_camera/flir_ax5_camera.glb"/>
         </geometry>
       </visual>
       <collision>
-        <origin xyz="-0.05205 0 -0.0015" rpy="0 0 0" />
+        <origin xyz="-0.05205 0 -0.0015" rpy="0 0 0"/>
         <geometry>
-          <box size="0.1041 0.04 0.043" />
+          <box size="0.1041 0.04 0.043"/>
         </geometry>
       </collision>
     </link>
-    <xacro:add_optical_frame name="${name}" />
+    <xacro:add_optical_frame name="${name}"/>
     <gazebo reference="${name}_frame">
       <material>Gazebo/Grey</material>
@@ -32,5 +32,5 @@
   <xacro:macro name="flir_a65_camera" params="name parent robot_name *origin">
     <xacro:flir_a65_camera_model name="${name}" parent="${parent}">
-      <xacro:insert_block name="origin" />
+      <xacro:insert_block name="origin"/>
     </xacro:flir_a65_camera_model>
     <xacro:flir_a65_camera_gazebo robot_name="${robot_name}"/>

File: urdf/generic_camera.urdf.xacro (robot description, xacro)
@@ -1,12 +1,10 @@
-<?xml version="1.0"?>
+<?xml version="1.0" encoding="UTF-8"?>
 <robot xmlns:xacro="http://www.ros.org/wiki/xacro">
-  <xacro:include filename="$(find hector_sensors_description)/gazebo/generic_camera.gazebo.xacro" />
-  <xacro:macro
-    name="generic_camera"
-    params="name parent robot_name *origin ros_topic cam_info_topic update_rate res_x res_y image_format hfov">
+  <xacro:include filename="$(find hector_sensors_description)/gazebo/generic_camera.gazebo.xacro"/>
+  <xacro:macro name="generic_camera" params="name parent robot_name *origin ros_topic cam_info_topic update_rate res_x res_y image_format hfov">
     <joint name="${name}_joint" type="fixed">
-      <xacro:insert_block name="origin" />
-      <parent link="${parent}" />
-      <child link="${name}_link" />
+      <xacro:insert_block name="origin"/>
+      <parent link="${parent}"/>
+      <child link="${name}_link"/>
     </joint>
     <link name="${name}_link">
@@ -32,18 +30,11 @@
       </collision>-->
     </link>
-    <link name="${name}_optical_frame" />
+    <link name="${name}_optical_frame"/>
     <joint name="${name}_optical_joint" type="fixed">
-      <origin xyz="0 0 0" rpy="${-pi/2} 0 ${-pi/2}" />
-      <parent link="${name}_link" />
-      <child link="${name}_optical_frame" />
+      <origin xyz="0 0 0" rpy="${-pi/2} 0 ${-pi/2}"/>
+      <parent link="${name}_link"/>
+      <child link="${name}_optical_frame"/>
     </joint>
-    <xacro:generic_camera_gazebo
-      name="${name}"
-      robot_name="${robot_name}"
-      update_rate="${update_rate}"
-      res_x="${res_x}"
-      res_y="${res_y}"
-      hfov="${hfov}"
-      image_format="${image_format}" />
+    <xacro:generic_camera_gazebo name="${name}" robot_name="${robot_name}" update_rate="${update_rate}" res_x="${res_x}" res_y="${res_y}" hfov="${hfov}" image_format="${image_format}"/>
   </xacro:macro>
 </robot>

File: urdf/generic_wide_angle_camera.urdf.xacro (robot description, xacro)
@@ -1,21 +1,19 @@
-<?xml version="1.0"?>
+<?xml version="1.0" encoding="UTF-8"?>
 <robot xmlns:xacro="http://www.ros.org/wiki/xacro">
-  <xacro:include filename="$(find hector_sensors_description)/gazebo/generic_wide_angle_camera.gazebo.xacro" />
-  <xacro:macro
-    name="generic_wide_angle_camera"
-    params="name parent robot_name *origin ros_topic cam_info_topic update_rate res_x res_y image_format hfov">
+  <xacro:include filename="$(find hector_sensors_description)/gazebo/generic_wide_angle_camera.gazebo.xacro"/>
+  <xacro:macro name="generic_wide_angle_camera" params="name parent robot_name *origin ros_topic cam_info_topic update_rate res_x res_y image_format hfov">
     <joint name="${name}_joint" type="fixed">
-      <xacro:insert_block name="origin" />
-      <parent link="${parent}" />
-      <child link="${name}_link" />
+      <xacro:insert_block name="origin"/>
+      <parent link="${parent}"/>
+      <child link="${name}_link"/>
     </joint>
     <link name="${name}_link">
       <inertial>
-        <mass value="0.01" />
-        <origin xyz="0 0 0" rpy="0 0 0" />
-        <inertia ixx="0.000001" ixy="0" ixz="0" iyy="0.000001" iyz="0" izz="0.000001" />
+        <mass value="0.01"/>
+        <origin xyz="0 0 0" rpy="0 0 0"/>
+        <inertia ixx="0.000001" ixy="0" ixz="0" iyy="0.000001" iyz="0" izz="0.000001"/>
       </inertial>
       <visual>
-	    <origin xyz="0 0 0" rpy="0 0 0" />
+        <origin xyz="0 0 0" rpy="0 0 0"/>
         <geometry>
           <box size="0.0017 0.032 0.032"/>
@@ -26,7 +24,7 @@
       </visual>
       <visual>
-        <origin xyz="0.00725 0 0" rpy="0 ${pi/2} 0" />
+        <origin xyz="0.00725 0 0" rpy="0 ${pi/2} 0"/>
         <geometry>
-          <cylinder radius="0.0086" length="0.0145" />
+          <cylinder radius="0.0086" length="0.0145"/>
         </geometry>
         <material name="Black">
@@ -35,24 +33,17 @@
       </visual>
       <collision>
-        <origin xyz="0.00725 0 0" rpy="0 0 0" />
+        <origin xyz="0.00725 0 0" rpy="0 0 0"/>
         <geometry>
-          <box size="0.016 0.032 0.032" />
+          <box size="0.016 0.032 0.032"/>
         </geometry>
       </collision>
     </link>
-    <link name="${name}_optical_frame" />
+    <link name="${name}_optical_frame"/>
     <joint name="${name}_optical_joint" type="fixed">
-      <origin xyz="0 0 0" rpy="${-pi/2} 0 ${-pi/2}" />
-      <parent link="${name}_link" />
-      <child link="${name}_optical_frame" />
+      <origin xyz="0 0 0" rpy="${-pi/2} 0 ${-pi/2}"/>
+      <parent link="${name}_link"/>
+      <child link="${name}_optical_frame"/>
     </joint>
-    <xacro:generic_wide_angle_camera_gazebo
-      name="${name}"
-      robot_name="${robot_name}"
-      update_rate="${update_rate}"
-      res_x="${res_x}"
-      res_y="${res_y}"
-      hfov="${hfov}"
-      image_format="${image_format}" />
+    <xacro:generic_wide_angle_camera_gazebo name="${name}" robot_name="${robot_name}" update_rate="${update_rate}" res_x="${res_x}" res_y="${res_y}" hfov="${hfov}" image_format="${image_format}"/>
   </xacro:macro>
 </robot>
