Commit message: Added extended ci

File: urdf/insta360_air.urdf.xacro (robot description, xacro)
@@ -1,63 +1,60 @@
-<?xml version="1.0"?>
+<?xml version="1.0" encoding="UTF-8"?>
 <robot xmlns:xacro="http://ros.org/wiki/xacro">
   <!-- TODO: datsheet: https://www.insta360.com/product/insta360-air -->
-  <xacro:property name="insta360_air_mass" value="0.05" /> <!-- estimated value -->
-  <xacro:property name="insta360_air_length" value="0.021" />
-  <xacro:property name="insta360_air_width" value="0.07" />
-  <xacro:property name="insta360_air_height" value="0.025" />
-  <xacro:include filename="$(find hector_xacro_tools)/urdf/inertia_tensors.urdf.xacro" />
-  <xacro:include filename="$(find hector_sensors_description)/gazebo/insta360_air.gazebo.xacro" />
+  <xacro:property name="insta360_air_mass" value="0.05"/>
+  <!-- estimated value -->
+  <xacro:property name="insta360_air_length" value="0.021"/>
+  <xacro:property name="insta360_air_width" value="0.07"/>
+  <xacro:property name="insta360_air_height" value="0.025"/>
+  <xacro:include filename="$(find hector_xacro_tools)/urdf/inertia_tensors.urdf.xacro"/>
+  <xacro:include filename="$(find hector_sensors_description)/gazebo/insta360_air.gazebo.xacro"/>
   <xacro:macro name="insta360_air" params="name *origin *parent">
-    <xacro:insta360_air_gazebo name="${name}" />
+    <xacro:insta360_air_gazebo name="${name}"/>
     <joint name="${name}_joint" type="fixed">
-      <child link="${name}_link" />
-      <xacro:insert_block name="origin" />
-      <xacro:insert_block name="parent" />
+      <child link="${name}_link"/>
+      <xacro:insert_block name="origin"/>
+      <xacro:insert_block name="parent"/>
     </joint>
     <!-- Camera base -->
     <link name="${name}_link">
-      <xacro:inertial_cuboid
-        mass="${insta360_air_mass}"
-        x_length="${insta360_air_length}"
-        y_length="${insta360_air_width}"
-        z_length="${insta360_air_height}" />
+      <xacro:inertial_cuboid mass="${insta360_air_mass}" x_length="${insta360_air_length}" y_length="${insta360_air_width}" z_length="${insta360_air_height}"/>
       <visual>
-        <origin xyz="0 0 0" rpy="0 0 0" />
+        <origin xyz="0 0 0" rpy="0 0 0"/>
         <geometry>
-          <box size="${insta360_air_length} ${insta360_air_width} ${insta360_air_height}" />
+          <box size="${insta360_air_length} ${insta360_air_width} ${insta360_air_height}"/>
         </geometry>
       </visual>
       <collision>
-        <origin xyz="0 0 0" rpy="0 0 0" />
+        <origin xyz="0 0 0" rpy="0 0 0"/>
         <geometry>
-          <box size="${insta360_air_length} ${insta360_air_width} ${insta360_air_height}" />
+          <box size="${insta360_air_length} ${insta360_air_width} ${insta360_air_height}"/>
         </geometry>
       </collision>
     </link>
     <!-- Camera RGB sensor -->
-    <link name="${name}_rgb_left" />
+    <link name="${name}_rgb_left"/>
     <joint name="${name}_rgb_left_joint" type="fixed">
-      <origin xyz="0 0 0" rpy="0 0 0" />
-      <parent link="${name}_link" />
-      <child link="${name}_rgb_left" />
+      <origin xyz="0 0 0" rpy="0 0 0"/>
+      <parent link="${name}_link"/>
+      <child link="${name}_rgb_left"/>
     </joint>
-    <link name="${name}_rgb_right" />
+    <link name="${name}_rgb_right"/>
     <joint name="${name}_rgb_right_joint" type="fixed">
-      <origin xyz="0 0 0" rpy="0 0 ${pi}" />
-      <parent link="${name}_link" />
-      <child link="${name}_rgb_right" />
+      <origin xyz="0 0 0" rpy="0 0 ${pi}"/>
+      <parent link="${name}_link"/>
+      <child link="${name}_rgb_right"/>
     </joint>
     <!-- Camera Optical Frame -->
-    <link name="${name}_left_optical_frame" />
+    <link name="${name}_left_optical_frame"/>
     <joint name="${name}_left_optical_joint" type="fixed">
-      <origin xyz="0 0 0" rpy="-${pi/2} 0 -${pi/2}" />
-      <parent link="${name}_rgb_left" />
-      <child link="${name}_left_optical_frame" />
+      <origin xyz="0 0 0" rpy="-${pi/2} 0 -${pi/2}"/>
+      <parent link="${name}_rgb_left"/>
+      <child link="${name}_left_optical_frame"/>
     </joint>
-    <link name="${name}_right_optical_frame" />
+    <link name="${name}_right_optical_frame"/>
     <joint name="${name}_right_optical_joint" type="fixed">
-      <origin xyz="0 0 0" rpy="-${pi/2} 0 -${pi/2}" />
-      <parent link="${name}_rgb_right" />
-      <child link="${name}_right_optical_frame" />
+      <origin xyz="0 0 0" rpy="-${pi/2} 0 -${pi/2}"/>
+      <parent link="${name}_rgb_right"/>
+      <child link="${name}_right_optical_frame"/>
     </joint>
   </xacro:macro>

File: urdf/insta360_pro2.urdf.xacro (robot description, xacro)
@@ -1,14 +1,14 @@
-<?xml version="1.0"?>
+<?xml version="1.0" encoding="UTF-8"?>
 <robot xmlns:xacro="http://www.ros.org/wiki/xacro">
   <xacro:include filename="$(find hector_sensors_description)/gazebo/insta360_pro2.gazebo.xacro"/>
-  <xacro:property name="camera_frame_center_distance" value="0.06" />
+  <xacro:property name="camera_frame_center_distance" value="0.06"/>
   <material name="Grey">
-    <color rgba="0.5 0.5 0.5 1" />
+    <color rgba="0.5 0.5 0.5 1"/>
   </material>
   <xacro:macro name="insta360_pro2" params="name parent robot_name *origin ros_topic update_rate res_x res_y image_format fov">
     <joint name="${name}_center_joint" type="fixed">
-      <xacro:insert_block name="origin" />
-      <parent link="${parent}" />
-      <child link="${name}_center_link" />
+      <xacro:insert_block name="origin"/>
+      <parent link="${parent}"/>
+      <child link="${name}_center_link"/>
     </joint>
     <link name="${name}_center_link">
@@ -16,45 +16,51 @@
       <visual>
         <geometry>
-          <mesh filename="package://hector_sensors_description/meshes/insta360_pro2/insta_pro2.glb" />
+          <mesh filename="package://hector_sensors_description/meshes/insta360_pro2/insta_pro2.glb"/>
         </geometry>
       </visual>
       <collision>
-        <origin xyz="0 0 0" rpy="0 0 0" />
+        <origin xyz="0 0 0" rpy="0 0 0"/>
         <geometry>
-          <sphere radius="0.075" />
+          <sphere radius="0.075"/>
         </geometry>
-        <material name="Grey" />
+        <material name="Grey"/>
       </collision>
       <collision>
-        <origin xyz="0 0 -0.0875" rpy="0 0 0" />
+        <origin xyz="0 0 -0.0875" rpy="0 0 0"/>
         <geometry>
-          <cylinder length="0.05" radius="0.04" />
+          <cylinder length="0.05" radius="0.04"/>
         </geometry>
       </collision>
     </link>
     <xacro:insta360_pro2_camera parent="${name}_center_link" camera_number="1" ros_topic="${ros_topic}" update_rate="${update_rate}" res_x="${res_x}" res_y="${res_y}" image_format="${image_format}" fov="${fov}">
-      <origin xyz="${camera_frame_center_distance} 0 0" rpy="${-pi/2} 0 ${-pi/2}" /> <!-- extrinsic calibration -->
+      <origin xyz="${camera_frame_center_distance} 0 0" rpy="${-pi/2} 0 ${-pi/2}"/>
+      <!-- extrinsic calibration -->
     </xacro:insta360_pro2_camera>
     <xacro:insta360_pro2_camera parent="${name}_origin1_optical_frame" camera_number="2" ros_topic="${ros_topic}" update_rate="${update_rate}" res_x="${res_x}" res_y="${res_y}" image_format="${image_format}" fov="${fov}">
-      <origin xyz="${camera_frame_center_distance * cos(radians(210))} 0 ${-camera_frame_center_distance * sin(radians(210))-camera_frame_center_distance} " rpy="0 ${radians(-60)} 0" /> <!-- extrinsic calibration -->
+      <origin xyz="${camera_frame_center_distance * cos(radians(210))} 0 ${-camera_frame_center_distance * sin(radians(210))-camera_frame_center_distance} " rpy="0 ${radians(-60)} 0"/>
+      <!-- extrinsic calibration -->
     </xacro:insta360_pro2_camera>
     <xacro:insta360_pro2_camera parent="${name}_origin1_optical_frame" camera_number="3" ros_topic="${ros_topic}" update_rate="${update_rate}" res_x="${res_x}" res_y="${res_y}" image_format="${image_format}" fov="${fov}">
-      <origin xyz="${camera_frame_center_distance * cos(radians(150))} 0 ${-camera_frame_center_distance * sin(radians(150))-camera_frame_center_distance} " rpy="0 ${radians(-120)} 0" /> <!-- extrinsic calibration -->
+      <origin xyz="${camera_frame_center_distance * cos(radians(150))} 0 ${-camera_frame_center_distance * sin(radians(150))-camera_frame_center_distance} " rpy="0 ${radians(-120)} 0"/>
+      <!-- extrinsic calibration -->
     </xacro:insta360_pro2_camera>
     <xacro:insta360_pro2_camera parent="${name}_origin1_optical_frame" camera_number="4" ros_topic="${ros_topic}" update_rate="${update_rate}" res_x="${res_x}" res_y="${res_y}" image_format="${image_format}" fov="${fov}">
-      <origin xyz="${camera_frame_center_distance * cos(radians(90))} 0 ${-camera_frame_center_distance * sin(radians(90))-camera_frame_center_distance} " rpy="0 ${radians(-180)} 0" /> <!-- extrinsic calibration -->
+      <origin xyz="${camera_frame_center_distance * cos(radians(90))} 0 ${-camera_frame_center_distance * sin(radians(90))-camera_frame_center_distance} " rpy="0 ${radians(-180)} 0"/>
+      <!-- extrinsic calibration -->
     </xacro:insta360_pro2_camera>
     <xacro:insta360_pro2_camera parent="${name}_origin1_optical_frame" camera_number="5" ros_topic="${ros_topic}" update_rate="${update_rate}" res_x="${res_x}" res_y="${res_y}" image_format="${image_format}" fov="${fov}">
-      <origin xyz="${camera_frame_center_distance * cos(radians(30))} 0 ${-camera_frame_center_distance * sin(radians(30))-camera_frame_center_distance} " rpy="0 ${radians(-240)} 0" /> <!-- extrinsic calibration -->
+      <origin xyz="${camera_frame_center_distance * cos(radians(30))} 0 ${-camera_frame_center_distance * sin(radians(30))-camera_frame_center_distance} " rpy="0 ${radians(-240)} 0"/>
+      <!-- extrinsic calibration -->
     </xacro:insta360_pro2_camera>
     <xacro:insta360_pro2_camera parent="${name}_origin1_optical_frame" camera_number="6" ros_topic="${ros_topic}" update_rate="${update_rate}" res_x="${res_x}" res_y="${res_y}" image_format="${image_format}" fov="${fov}">
-      <origin xyz="${camera_frame_center_distance * cos(radians(-30))} 0 ${-camera_frame_center_distance * sin(radians(-30))-camera_frame_center_distance} " rpy="0 ${radians(-300)} 0" /> <!-- extrinsic calibration -->
+      <origin xyz="${camera_frame_center_distance * cos(radians(-30))} 0 ${-camera_frame_center_distance * sin(radians(-30))-camera_frame_center_distance} " rpy="0 ${radians(-300)} 0"/>
+      <!-- extrinsic calibration -->
     </xacro:insta360_pro2_camera>
   </xacro:macro>
   <xacro:macro name="insta360_pro2_with_calibration" params="name parent robot_name *origin *calibration1 *calibration2 *calibration3 *calibration4 *calibration5 *calibration6 ros_topic update_rate res_x res_y image_format fov">
     <joint name="${name}_center_joint" type="fixed">
-      <xacro:insert_block name="origin" />
-      <parent link="${parent}" />
-      <child link="${name}_center_link" />
+      <xacro:insert_block name="origin"/>
+      <parent link="${parent}"/>
+      <child link="${name}_center_link"/>
     </joint>
     <link name="${name}_center_link">
@@ -62,55 +68,55 @@
       <visual>
         <geometry>
-          <mesh filename="package://hector_sensors_description/meshes/insta360_pro2/insta_pro2.glb" />
+          <mesh filename="package://hector_sensors_description/meshes/insta360_pro2/insta_pro2.glb"/>
         </geometry>
       </visual>
       <collision>
-        <origin xyz="0 0 0" rpy="0 0 0" />
+        <origin xyz="0 0 0" rpy="0 0 0"/>
         <geometry>
-          <sphere radius="0.075" />
+          <sphere radius="0.075"/>
         </geometry>
-        <material name="Grey" />
+        <material name="Grey"/>
       </collision>
       <collision>
-        <origin xyz="0 0 -0.0875" rpy="0 0 0" />
+        <origin xyz="0 0 -0.0875" rpy="0 0 0"/>
         <geometry>
-          <cylinder length="0.05" radius="0.04" />
+          <cylinder length="0.05" radius="0.04"/>
         </geometry>
       </collision>
     </link>
     <xacro:insta360_pro2_camera parent="${name}_origin2_optical_frame" robot_name="${robot_name}" camera_number="1" ros_topic="${ros_topic}" update_rate="${update_rate}" res_x="${res_x}" res_y="${res_y}" image_format="${image_format}" fov="${fov}">
-      <xacro:insert_block name="calibration1" />
+      <xacro:insert_block name="calibration1"/>
     </xacro:insta360_pro2_camera>
     <xacro:insta360_pro2_camera parent="${name}_origin3_optical_frame" robot_name="${robot_name}" camera_number="2" ros_topic="${ros_topic}" update_rate="${update_rate}" res_x="${res_x}" res_y="${res_y}" image_format="${image_format}" fov="${fov}">
-      <xacro:insert_block name="calibration2" />
+      <xacro:insert_block name="calibration2"/>
     </xacro:insta360_pro2_camera>
     <xacro:insta360_pro2_camera parent="${name}_origin4_optical_frame" robot_name="${robot_name}" camera_number="3" ros_topic="${ros_topic}" update_rate="${update_rate}" res_x="${res_x}" res_y="${res_y}" image_format="${image_format}" fov="${fov}">
-      <xacro:insert_block name="calibration3" />
+      <xacro:insert_block name="calibration3"/>
     </xacro:insta360_pro2_camera>
     <xacro:insta360_pro2_camera parent="${name}_origin5_optical_frame" robot_name="${robot_name}" camera_number="4" ros_topic="${ros_topic}" update_rate="${update_rate}" res_x="${res_x}" res_y="${res_y}" image_format="${image_format}" fov="${fov}">
-      <xacro:insert_block name="calibration4" />
+      <xacro:insert_block name="calibration4"/>
     </xacro:insta360_pro2_camera>
     <xacro:insta360_pro2_camera parent="${name}_origin6_optical_frame" robot_name="${robot_name}" camera_number="5" ros_topic="${ros_topic}" update_rate="${update_rate}" res_x="${res_x}" res_y="${res_y}" image_format="${image_format}" fov="${fov}">
-      <xacro:insert_block name="calibration5" />
+      <xacro:insert_block name="calibration5"/>
     </xacro:insta360_pro2_camera>
     <xacro:insta360_pro2_camera parent="${name}_center_link" robot_name="${robot_name}" camera_number="6" ros_topic="${ros_topic}" update_rate="${update_rate}" res_x="${res_x}" res_y="${res_y}" image_format="${image_format}" fov="${fov}">
-      <xacro:insert_block name="calibration6" />
+      <xacro:insert_block name="calibration6"/>
     </xacro:insta360_pro2_camera>
   </xacro:macro>
   <xacro:macro name="insta360_pro2_camera" params="camera_number robot_name parent *calibration ros_topic update_rate res_x res_y image_format fov">
-    <xacro:property name="camera_name" value="${name}_origin${camera_number}" />
+    <xacro:property name="camera_name" value="${name}_origin${camera_number}"/>
     <joint name="${camera_name}_optical_joint" type="fixed">
-      <xacro:insert_block name="calibration" />
-      <parent link="${parent}" />
-      <child link="${camera_name}_optical_frame" />
+      <xacro:insert_block name="calibration"/>
+      <parent link="${parent}"/>
+      <child link="${camera_name}_optical_frame"/>
     </joint>
     <joint name="${camera_name}_joint" type="fixed">
-      <origin xyz="0 0 0" rpy="0 ${-pi/2} ${pi/2}" />
-      <parent link="${camera_name}_optical_frame" />
-      <child link="${camera_name}_link" />
+      <origin xyz="0 0 0" rpy="0 ${-pi/2} ${pi/2}"/>
+      <parent link="${camera_name}_optical_frame"/>
+      <child link="${camera_name}_link"/>
     </joint>
-    <link name="${camera_name}_link" />
-    <link name="${camera_name}_optical_frame" />
-    <xacro:insta360_pro2_gazebo camera_name="${camera_name}" robot_name="${robot_name}" ros_topic="${ros_topic}" update_rate="${update_rate}" fov="${fov}" image_format="${image_format}" res_x="${res_x}" res_y="${res_y}" />
+    <link name="${camera_name}_link"/>
+    <link name="${camera_name}_optical_frame"/>
+    <xacro:insta360_pro2_gazebo camera_name="${camera_name}" robot_name="${robot_name}" ros_topic="${ros_topic}" update_rate="${update_rate}" fov="${fov}" image_format="${image_format}" res_x="${res_x}" res_y="${res_y}"/>
   </xacro:macro>
 </robot>
