Commit message: Applied topic fix from rgb to color and also frame fix for ec-swift rgbd

File: gazebo/orbbec_astra2.gazebo.xacro (robot description, xacro)
@@ -4,13 +4,13 @@
   <xacro:macro name="orbbec_astra2_gazebo" params="name:=default semantic_segmentation:=false">
     <gazebo reference="${name}_link">
-      <sensor type="camera" name="${name}_rgb">
+      <sensor type="camera" name="${name}_color">
         <always_on>true</always_on>
         <visualize>true</visualize>
         <update_rate>15</update_rate>
-        <topic>/$(arg robot_name)/${name}/rgb/image_raw</topic>
-        <gz_frame_id>${name}_rgb_link</gz_frame_id>
+        <topic>/$(arg robot_name)/${name}/color/image_raw</topic>
+        <gz_frame_id>${name}_color_frame</gz_frame_id>
         <camera name="${name}_camera">
-          <camera_info_topic>/$(arg robot_name)/${name}/rgb/camera_info</camera_info_topic>
-          <optical_frame_id>${name}_rgb_optical_frame</optical_frame_id>
+          <camera_info_topic>/$(arg robot_name)/${name}/color/camera_info</camera_info_topic>
+          <optical_frame_id>${name}_color_optical_frame</optical_frame_id>
           <horizontal_fov>${radians(90.0)}</horizontal_fov>
           <image>
@@ -30,5 +30,5 @@
         <update_rate>15</update_rate>
         <topic>/$(arg robot_name)/${name}/depth/image_raw</topic>
-        <gz_frame_id>${name}_depth_link</gz_frame_id>
+        <gz_frame_id>${name}_depth_frame</gz_frame_id>
         <camera>
           <camera_info_topic>/$(arg robot_name)/${name}/depth/camera_info</camera_info_topic>
@@ -56,5 +56,5 @@
         <sensor name="astra2_${name}_segmentation_camera" type="segmentation">
           <topic>/$(arg robot_name)/${name}/segmentation</topic>
-          <gz_frame_id>${name}_link</gz_frame_id>
+          <gz_frame_id>${name}_frame</gz_frame_id>
           <camera>
             <optical_frame_id>${name}_optical_frame</optical_frame_id>

File: gazebo/orbbec_gemini2.gazebo.xacro (robot description, xacro)
@@ -60,5 +60,5 @@
         <sensor name="gemini2_${name}_segmentation_camera" type="segmentation">
           <topic>/$(arg robot_name)/${name}/segmentation</topic>
-          <gz_frame_id>${name}_color_link</gz_frame_id>
+          <gz_frame_id>${name}_color_frame</gz_frame_id>
           <camera>
             <optical_frame_id>${name}_color_optical_frame</optical_frame_id>

File: urdf/orbbec_astra2.urdf.xacro (robot description, xacro)
@@ -32,30 +32,5 @@
       </collision>
     </link>
-    <!-- Camera RGB sensor -->
-    <link name="${name}_rgb_link"/>
-    <joint name="${name}_rgb_joint" type="fixed">
-      <origin xyz="0.033 0.022 0" rpy="0 0 0"/>
-      <parent link="${name}_link"/>
-      <child link="${name}_rgb_link"/>
-    </joint>
-    <!-- Optical Frame for ros (in z direction) -->
-    <link name="${name}_rgb_optical_frame"/>
-    <joint name="${name}_rgb_optical_joint" type="fixed">
-      <origin xyz="0 0 0" rpy="-${pi/2.0} 0 -${pi/2.0}"/>
-      <parent link="${name}_link"/>
-      <child link="${name}_rgb_optical_frame"/>
-    </joint>
-    <link name="${name}_depth_link"/>
-    <joint name="${name}_depth_joint" type="fixed">
-      <origin xyz="0.033 0.022 0" rpy="0 0 0"/>
-      <parent link="${name}_link"/>
-      <child link="${name}_depth_link"/>
-    </joint>
-    <link name="${name}_depth_optical_frame"/>
-    <joint name="${name}_depth_optical_joint" type="fixed">
-      <origin xyz="0 0 0" rpy="-${pi/2.0} 0 -${pi/2.0}"/>
-      <parent link="${name}_link"/>
-      <child link="${name}_depth_optical_frame"/>
-    </joint>
+    <!-- optical frames are published by driver, use launch file for simulation -->
   </xacro:macro>
 </robot>
