Commit message: Add livox_mid360_base_link and optical_frame link

File: gazebo/livox_mid360.gazebo.xacro (robot description, xacro)
@@ -3,10 +3,10 @@
 	<xacro:property name="M_PI" value="3.14159"/>
 	<xacro:macro name="livox_mid360_gazebo" params="visualize:=True name:=default">
-		<gazebo reference="livox_mid360_${name}_link">
+		<gazebo reference="livox_mid360_${name}_optical_frame">
 			<sensor name='gpu_lidar_${name}' type='gpu_lidar'>"
-				<pose relative_to='livox_mid360_${name}_link'>0 0 0 0 0 0</pose>
+				<pose relative_to='livox_mid360_${name}_optical_frame'>0 0 0 0 0 0</pose>
 				<topic>/$(arg robot_name)/livox_mid360_${name}</topic>
 				<update_rate>10</update_rate>
-				<gz_frame_id>livox_mid360_${name}_link</gz_frame_id>
+				<gz_frame_id>livox_mid360_${name}_optical_frame</gz_frame_id>
 				<ray>
 					<scan>

File: urdf/livox_mid360.xacro (robot description, xacro)
@@ -10,9 +10,9 @@
 	<xacro:macro name="livox_mid360" params="name:=default *origin *parent">
 		<joint name="livox_mid360_${name}_joint" type="fixed">
-			<child link="livox_mid360_${name}_link"/>
+			<child link="livox_mid360_${name}_base_link"/>
 			<xacro:insert_block name="origin"/>
 			<xacro:insert_block name="parent"/>
 		</joint>
-		<link name="livox_mid360_${name}_link">
+		<link name="livox_mid360_${name}_base_link">
 			<xacro:inertial_cuboid mass="${livox_mid360_mass}" x_length="${livox_mid360_length}" y_length="${livox_mid360_width}" z_length="${livox_mid360_height}"/>
 			<visual>
@@ -30,4 +30,10 @@
 			</collision>
 		</link>
+		<link name="livox_mid360_${name}_optical_frame"/>
+		<joint name="livox_mid360_${name}_sensor_joint_optical_frame" type="fixed">
+			<origin xyz="0 0 0" rpy="0 0 ${M_PI/2.0}" />
+            <parent link="livox_mid360_${name}_base_link" />
+            <child link="livox_mid360_${name}_optical_frame" />
+        </joint>
 	</xacro:macro>
 </robot>

Commit message: Rename optical_frame to laser_frame

File: gazebo/livox_mid360.gazebo.xacro (robot description, xacro)
@@ -3,10 +3,10 @@
 	<xacro:property name="M_PI" value="3.14159"/>
 	<xacro:macro name="livox_mid360_gazebo" params="visualize:=True name:=default">
-		<gazebo reference="livox_mid360_${name}_optical_frame">
+		<gazebo reference="livox_mid360_${name}_laser_frame">
 			<sensor name='gpu_lidar_${name}' type='gpu_lidar'>"
-				<pose relative_to='livox_mid360_${name}_optical_frame'>0 0 0 0 0 0</pose>
+				<pose relative_to='livox_mid360_${name}_laser_frame'>0 0 0 0 0 0</pose>
 				<topic>/$(arg robot_name)/livox_mid360_${name}</topic>
 				<update_rate>10</update_rate>
-				<gz_frame_id>livox_mid360_${name}_optical_frame</gz_frame_id>
+				<gz_frame_id>livox_mid360_${name}_laser_frame</gz_frame_id>
 				<ray>
 					<scan>

File: urdf/livox_mid360.xacro (robot description, xacro)
@@ -30,9 +30,9 @@
 			</collision>
 		</link>
-		<link name="livox_mid360_${name}_optical_frame"/>
-		<joint name="livox_mid360_${name}_sensor_joint_optical_frame" type="fixed">
+		<link name="livox_mid360_${name}_laser_frame"/>
+		<joint name="livox_mid360_${name}_sensor_joint_laser_frame" type="fixed">
 			<origin xyz="0 0 0" rpy="0 0 ${M_PI/2.0}" />
             <parent link="livox_mid360_${name}_base_link" />
-            <child link="livox_mid360_${name}_optical_frame" />
+            <child link="livox_mid360_${name}_laser_frame" />
         </joint>
 	</xacro:macro>

Commit message: Add laser_frame link for livox_mid360 (#3)
* Add livox_mid360_base_link and laser_frame link

File: gazebo/livox_mid360.gazebo.xacro (robot description, xacro)
@@ -3,10 +3,10 @@
 	<xacro:property name="M_PI" value="3.14159"/>
 	<xacro:macro name="livox_mid360_gazebo" params="visualize:=True name:=default">
-		<gazebo reference="livox_mid360_${name}_link">
+		<gazebo reference="livox_mid360_${name}_laser_frame">
 			<sensor name='gpu_lidar_${name}' type='gpu_lidar'>"
-				<pose relative_to='livox_mid360_${name}_link'>0 0 0 0 0 0</pose>
+				<pose relative_to='livox_mid360_${name}_laser_frame'>0 0 0 0 0 0</pose>
 				<topic>/$(arg robot_name)/livox_mid360_${name}</topic>
 				<update_rate>10</update_rate>
-				<gz_frame_id>livox_mid360_${name}_link</gz_frame_id>
+				<gz_frame_id>livox_mid360_${name}_laser_frame</gz_frame_id>
 				<ray>
 					<scan>

File: urdf/livox_mid360.xacro (robot description, xacro)
@@ -10,9 +10,9 @@
 	<xacro:macro name="livox_mid360" params="name:=default *origin *parent">
 		<joint name="livox_mid360_${name}_joint" type="fixed">
-			<child link="livox_mid360_${name}_link"/>
+			<child link="livox_mid360_${name}_base_link"/>
 			<xacro:insert_block name="origin"/>
 			<xacro:insert_block name="parent"/>
 		</joint>
-		<link name="livox_mid360_${name}_link">
+		<link name="livox_mid360_${name}_base_link">
 			<xacro:inertial_cuboid mass="${livox_mid360_mass}" x_length="${livox_mid360_length}" y_length="${livox_mid360_width}" z_length="${livox_mid360_height}"/>
 			<visual>
@@ -30,4 +30,10 @@
 			</collision>
 		</link>
+		<link name="livox_mid360_${name}_laser_frame"/>
+		<joint name="livox_mid360_${name}_sensor_joint_laser_frame" type="fixed">
+			<origin xyz="0 0 0" rpy="0 0 ${M_PI/2.0}" />
+            <parent link="livox_mid360_${name}_base_link" />
+            <child link="livox_mid360_${name}_laser_frame" />
+        </joint>
 	</xacro:macro>
 </robot>

Commit message: include gazebo in urdf for athena and ecswift sensors

File: gazebo/livox_mid360.gazebo.xacro (robot description, xacro)
@@ -6,7 +6,7 @@
 			<sensor name='gpu_lidar_${name}' type='gpu_lidar'>"
 				<pose relative_to='${name}_laser_frame'>0 0 0 0 0 0</pose>
-				<topic>/$(arg robot_name)/livox_mid360_${name}</topic>
+				<topic>/$(arg robot_name)/${name}</topic>
 				<update_rate>10</update_rate>
-				<gz_frame_id>livox_mid360_${name}_laser_frame</gz_frame_id>
+				<gz_frame_id>${name}_laser_frame</gz_frame_id>
 				<ray>
 					<scan>

File: gazebo/orbbec_astra2.gazebo.xacro (robot description, xacro)
@@ -2,5 +2,5 @@
 <robot xmlns:xacro="http://ros.org/wiki/xacro">
 	<xacro:property name="M_PI" value="3.14159"/>
-	<xacro:macro name="orbbec_astra2_gazebo" params="name:=default semantic_segmentation:=false">
+	<xacro:macro name="orbbec_astra2_gazebo" params="name:=default">
 		<gazebo reference="${name}_link">
 			<sensor type="camera" name="${name}_rgb">

File: urdf/astra_stereo_s_u3.urdf.xacro (robot description, xacro)
@@ -4,5 +4,7 @@
     <xacro:property name="M_PI" value="3.14159"/>
     <xacro:include filename="$(find hector_xacro_tools)/urdf/inertia_tensors.urdf.xacro" />
+	<xacro:include filename="$(find hector_sensors_description)/gazebo/astra_stereo_s_u3.gazebo.xacro" />
     <xacro:macro name="orbbec_astra_stereo_s_u3" params="name *origin *parent">
+        <xacro:orbbec_astra_stereo_s_u3_gazebo name="${name}" />
         <xacro:property name="orbbec_astra_stereo_s_u3_mass" value="0.05"/> <!-- estimated, needs to be checked -->
         <xacro:property name="orbbec_astra_stereo_s_u3_length" value="0.0653"/>

File: urdf/insta360_air.urdf.xacro (robot description, xacro)
@@ -8,5 +8,7 @@
     <xacro:property name="insta360_air_height" value="0.025"/>
     <xacro:include filename="$(find hector_xacro_tools)/urdf/inertia_tensors.urdf.xacro" />
+	<xacro:include filename="$(find hector_sensors_description)/gazebo/insta360_air.gazebo.xacro" />
     <xacro:macro name="insta360_air" params="name *origin *parent">
+        <xacro:insta360_air_gazebo name="${name}" />
         <joint name="${name}_joint" type="fixed">
             <child link="${name}_link"/>

File: urdf/livox_mid360.urdf.xacro (robot description, xacro)
@@ -8,5 +8,7 @@
 	<xacro:property name="livox_mid360_height" value="0.061"/>
 	<xacro:include filename="$(find hector_xacro_tools)/urdf/inertia_tensors.urdf.xacro" />
+	<xacro:include filename="$(find hector_sensors_description)/gazebo/livox_mid360.gazebo.xacro" />
 	<xacro:macro name="livox_mid360" params="name *origin *parent">
+	  	<xacro:livox_mid360_gazebo name="${name}" />
 		<joint name="${name}_joint" type="fixed">
 			<child link="${name}_link"/>
@@ -14,5 +16,5 @@
 			<xacro:insert_block name="parent"/>
 		</joint>
-		<link name="${name}_lidar_link">
+		<link name="${name}_link">
 			<xacro:inertial_cuboid mass="${livox_mid360_mass}" x_length="${livox_mid360_length}" y_length="${livox_mid360_width}" z_length="${livox_mid360_height}"/>
 			<visual>

File: urdf/orbbec_astra2.urdf.xacro (robot description, xacro)
@@ -4,5 +4,7 @@
     <xacro:property name="M_PI" value="3.14159"/>
     <xacro:include filename="$(find hector_xacro_tools)/urdf/inertia_tensors.urdf.xacro" />
+    <xacro:include filename="$(find hector_sensors_description)/gazebo/orbbec_astra2.gazebo.xacro" />
     <xacro:macro name="orbbec_astra2" params="name *origin *parent">
+        <xacro:orbbec_astra2_gazebo name="${name}" />
         <xacro:property name="orbbec_astra2_mass" value="0.195"/>
         <xacro:property name="orbbec_astra2_length" value="0.037"/>

Commit message: Added Livox Mid360 RGL-Plugin Lidar Pattern

File: gazebo/livox_mid360.gazebo.xacro (robot description, xacro)
@@ -2,35 +2,60 @@
 <robot xmlns:xacro="http://ros.org/wiki/xacro">
 	<xacro:property name="M_PI" value="3.14159"/>
-	<xacro:macro name="livox_mid360_gazebo" params="visualize:=True name:=default">
+	<xacro:macro name="livox_mid360_gazebo" params="visualize:=True name:=default use_rgl:=False">
 		<gazebo reference="${name}_laser_frame">
-			<sensor name='gpu_lidar_${name}' type='gpu_lidar'>"
-				<pose relative_to='${name}_laser_frame'>0 0 0 0 0 0</pose>
-				<topic>/$(arg robot_name)/${name}</topic>
-				<update_rate>10</update_rate>
-				<gz_frame_id>${name}_laser_frame</gz_frame_id>
-				<ray>
-					<scan>
-						<horizontal>
-							<samples>100</samples>
-							<resolution>1</resolution>
-							<min_angle>${0}</min_angle>
-							<max_angle>${2*M_PI}</max_angle>
-						</horizontal>
-						<vertical>
-							<samples>360</samples>
-							<resolution>1</resolution>
-							<min_angle>${-7.22/180*M_PI}</min_angle>
-							<max_angle>${55.22/180*M_PI}</max_angle>
-						</vertical>
-					</scan>
-					<range>
-						<min>0.08</min>
-						<max>10.0</max>
-						<resolution>0.01</resolution>
-					</range>
-				</ray>
-				<always_on>1</always_on>
-				<visualize>${visualize}</visualize>
-			</sensor>
+			<!-- ===== RGL-Variante (Livox Mid360 Preset) ===== -->
+			<xacro:if value="${use_rgl}">
+				<sensor name="rgl_lidar_${name}" type="custom">
+					<pose relative_to='${name}_laser_frame'>0 0 0 0 0 0</pose>
+					<always_on>true</always_on>
+					<update_rate>10</update_rate>
+					<visualize>${visualize}</visualize>
+					<plugin filename="RGLServerPluginInstance" name="rgl::RGLServerPluginInstance">
+						<range>
+							<min>0.1</min>
+							<max>100.0</max>
+						</range>
+						<update_rate>10</update_rate>
+						<!-- Gazebo-Transport Topic (wird via ros_gz_bridge auf PointCloud2 gemappt) -->
+						<topic>/$(arg robot_name)/${name}</topic>
+						<!-- Frame-Name, der in die Cloud geschrieben wird -->
+						<frame>${name}_laser_frame</frame>
+						<!-- Livox Scanmuster (setzt RGL_PATTERNS_DIR voraus) -->
+						<pattern_preset>Livox Mid360</pattern_preset>
+					</plugin>
+				</sensor>
+			</xacro:if>
+			<!-- ===== Fallback: bisheriger gpu_lidar ===== -->
+			<xacro:unless value="${use_rgl}">
+				<sensor name='gpu_lidar_${name}' type='gpu_lidar'>
+					<pose relative_to='${name}_laser_frame'>0 0 0 0 0 0</pose>
+					<topic>/$(arg robot_name)/${name}</topic>
+					<update_rate>10</update_rate>
+					<gz_frame_id>${name}_laser_frame</gz_frame_id>
+					<ray>
+						<scan>
+							<horizontal>
+								<samples>100</samples>
+								<resolution>1</resolution>
+								<min_angle>${0}</min_angle>
+								<max_angle>${2*M_PI}</max_angle>
+							</horizontal>
+							<vertical>
+								<samples>360</samples>
+								<resolution>1</resolution>
+								<min_angle>${-7.22/180*M_PI}</min_angle>
+								<max_angle>${55.22/180*M_PI}</max_angle>
+							</vertical>
+						</scan>
+						<range>
+							<min>0.08</min>
+							<max>10.0</max>
+							<resolution>0.01</resolution>
+						</range>
+					</ray>
+					<always_on>1</always_on>
+					<visualize>${visualize}</visualize>
+				</sensor>
+			</xacro:unless>
 		</gazebo>
 	</xacro:macro>

Commit message: Fixed the RGL Plugin Instance for the Livox Mid360 Lidar

File: gazebo/livox_mid360.gazebo.xacro (robot description, xacro)
@@ -2,29 +2,27 @@
 <robot xmlns:xacro="http://ros.org/wiki/xacro">
 	<xacro:property name="M_PI" value="3.14159"/>
-	<xacro:macro name="livox_mid360_gazebo" params="visualize:=True name:=default use_rgl:=False">
+	<xacro:macro name="livox_mid360_gazebo" params="visualize:=True name:=default use_rgl:=True">
 		<gazebo reference="${name}_laser_frame">
-			<!-- ===== RGL-Variante (Livox Mid360 Preset) ===== -->
+			<!-- ===== RGL-Variant (Livox Mid360 Preset) ===== -->
 			<xacro:if value="${use_rgl}">
-				<sensor name="rgl_lidar_${name}" type="custom">
+				<sensor name="${name}" type="custom">
 					<pose relative_to='${name}_laser_frame'>0 0 0 0 0 0</pose>
-					<always_on>true</always_on>
 					<update_rate>10</update_rate>
-					<visualize>${visualize}</visualize>
 					<plugin filename="RGLServerPluginInstance" name="rgl::RGLServerPluginInstance">
 						<range>
-							<min>0.1</min>
-							<max>100.0</max>
+							<min>0</min>
+							<max>245</max>
 						</range>
 						<update_rate>10</update_rate>
-						<!-- Gazebo-Transport Topic (wird via ros_gz_bridge auf PointCloud2 gemappt) -->
-						<topic>/$(arg robot_name)/${name}</topic>
-						<!-- Frame-Name, der in die Cloud geschrieben wird -->
+						<update_on_paused_sim>false</update_on_paused_sim>
+						<topic>/$(arg robot_name)/${name}/points</topic>
 						<frame>${name}_laser_frame</frame>
-						<!-- Livox Scanmuster (setzt RGL_PATTERNS_DIR voraus) -->
 						<pattern_preset>Livox Mid360</pattern_preset>
 					</plugin>
+					<always_on>1</always_on>
+					<visualize>${visualize}</visualize>
 				</sensor>
 			</xacro:if>
-			<!-- ===== Fallback: bisheriger gpu_lidar ===== -->
+			<!-- ===== Fallback: gpu_lidar ===== -->
 			<xacro:unless value="${use_rgl}">
 				<sensor name='gpu_lidar_${name}' type='gpu_lidar'>
