Commit message: updated lidars and scout zoom cam transform

File: gazebo/livox_mid360.gazebo.xacro (robot description, xacro)
@@ -9,4 +9,6 @@
 				<update_rate>10</update_rate>
 				<gz_frame_id>${name}_laser_frame</gz_frame_id>
+				<always_on>1</always_on>
+                <visualize>${visualize}</visualize>
 				<ray>
 					<scan>
@@ -30,6 +32,4 @@
 					</range>
 				</ray>
-				<always_on>1</always_on>
-				<visualize>${visualize}</visualize>
 			</sensor>
 		</gazebo>

File: gazebo/os0_128.gazebo.xacro (robot description, xacro)
@@ -1,25 +1,27 @@
 <?xml version="1.0"?>
 <robot xmlns:xacro="http://ros.org/wiki/xacro">
-    <xacro:macro name="os0_128_gazebo" params="name robot_name update_rate horizontal_samples vertical_samples min_range max_range">
-        <gazebo reference="${name}_frame">
-            <sensor name="${name}-OS0-128" type="gpu_lidar">
-                <visualize>false</visualize>
-                <always_on>true</always_on>
+	<xacro:property name="M_PI" value="3.14159"/>
+    <xacro:macro name="os0_128_gazebo" params="name update_rate horizontal_samples vertical_samples min_range max_range min_angle max_angle">
+        <gazebo reference="${name}_laser_frame">
+            <sensor name="gpu_lidar_${name}" type="gpu_lidar">
+            	<pose relative_to='${name}_laser_frame'>0 0 0 0 0 0</pose>
+                <topic>/$(arg robot_name)/${name}</topic>
                 <update_rate>${update_rate}</update_rate>
-                <topic>${robot_name}/${name}/scan</topic>
-                <!--gz_frame_id>${name}_frame</gz_frame_id-->
-                <lidar>
+                <gz_frame_id>${name}_laser_frame</gz_frame_id>
+                <always_on>1</always_on>
+                <visualize>True</visualize>
+                <ray>
                     <scan>
                         <horizontal>
-                        <samples>${horizontal_samples}</samples>
-                        <resolution>1</resolution>
-                        <min_angle>-${pi}</min_angle>
-                        <max_angle>${pi}</max_angle>
+                            <samples>${horizontal_samples}</samples>
+                            <resolution>1</resolution>
+                            <min_angle>-${pi}</min_angle>
+                            <max_angle>${pi}</max_angle>
                         </horizontal>
                         <vertical>
-                        <samples>${vertical_samples}</samples>
-                        <resolution>1</resolution>
-                        <min_angle>-${45.0*pi/180.0}</min_angle>
-                        <max_angle>${45.0*pi/180.0}</max_angle>
+                            <samples>${vertical_samples}</samples>
+                            <resolution>1</resolution>
+                            <min_angle>-${min_angle*pi/180.0}</min_angle>
+                            <max_angle>${max_angle*pi/180.0}</max_angle>
                         </vertical>
                     </scan>
@@ -29,10 +31,5 @@
                         <resolution>0.003</resolution>
                     </range>
-                    <noise>
-                        <type>gaussian</type>
-                        <mean>0.0</mean>
-                        <stddev>0.008</stddev>
-                    </noise>
-                </lidar>
+                </ray>
             </sensor>
         </gazebo>

File: urdf/os0_128.urdf.xacro (robot description, xacro)
@@ -1,50 +1,58 @@
 <?xml version="1.0"?>
 <robot xmlns:xacro="http://www.ros.org/wiki/xacro">
-  <xacro:include filename="$(find hector_xacro_tools)/urdf/inertia_tensors.urdf.xacro"/>
-  <xacro:include filename="$(find hector_sensors_description)/gazebo/os0_128.gazebo.xacro"/>
-  <xacro:macro name="os0_128_model" params="name parent *origin">
-    <joint name="${name}_joint" type="fixed">
-      <xacro:insert_block name="origin"/>
-      <parent link="${parent}"/>
-      <child link="${name}_frame"/>
-    </joint>
-    <link name="${name}_frame">
-      <xacro:inertial_sphere mass="0.992" diameter="0.08082"/>
-      <visual>
-        <origin xyz="0 0 -0.062825" rpy="0 0 0" />
-        <geometry>
-          <mesh filename="package://hector_sensors_description/meshes/ouster_os0/os0_baseplate.dae" scale="0.001 0.001 0.001"/>
-        </geometry>
-      </visual>
-      <visual>
-        <origin xyz="0 0 -0.040825" rpy="0 0 0" />
-        <geometry>
-          <mesh filename="package://hector_sensors_description/meshes/ouster_os0/os0.dae" scale="0.001 0.001 0.001"/>
-        </geometry>
-      </visual>
-      <collision>
-        <origin xyz="0 0 -0.000825" rpy="0 0 0" />
-        <geometry>
-          <cylinder radius="0.04041" length="0.0735"/>
-        </geometry>
-      </collision>
-      <collision>
-        <origin xyz="0 0 -0.047825" rpy="0 0 0"/>
-        <geometry>
-          <box size="0.11 0.11 0.0205"/>
-        </geometry>
-      </collision>
-    </link>
-  </xacro:macro>
-  <xacro:macro name="os0_128" params="name robot_name parent *origin ros_topic">
-    <xacro:os0_128_advanced_parameters name="${name}" robot_name="${robot_name}" parent="${parent}" update_rate="10" horizontal_samples="512" vertical_samples="128" min_range="0.45" max_range="100">
-      <xacro:insert_block name="origin"/>
-    </xacro:os0_128_advanced_parameters>
-  </xacro:macro>
-  <xacro:macro name="os0_128_advanced_parameters" params="name robot_name parent *origin update_rate horizontal_samples vertical_samples min_range max_range">
-    <xacro:os0_128_model name="${name}" parent="${parent}">
-      <xacro:insert_block name="origin"/>
-    </xacro:os0_128_model>
-    <xacro:os0_128_gazebo name="${name}" robot_name="${robot_name}" update_rate="${update_rate}" horizontal_samples="${horizontal_samples}" vertical_samples="${vertical_samples}" min_range="${min_range}" max_range="${max_range}"/>
-  </xacro:macro>
+    <xacro:include filename="$(find hector_xacro_tools)/urdf/inertia_tensors.urdf.xacro"/>
+    <xacro:include filename="$(find hector_sensors_description)/gazebo/os0_128.gazebo.xacro"/>
+    <xacro:macro name="os0_128_model" params="name *origin *parent">
+        <joint name="${name}_joint" type="fixed">
+        	<child link="${name}_link"/>
+        	<xacro:insert_block name="origin"/>
+        	<xacro:insert_block name="parent"/>
+        </joint>
+        <link name="${name}_link">
+            <xacro:inertial_sphere mass="0.992" diameter="0.08082"/>
+            <visual>
+                <origin xyz="0 0 -0.062825" rpy="0 0 0" />
+                <geometry>
+                    <mesh filename="package://hector_sensors_description/meshes/ouster_os0/os0_baseplate.dae" scale="0.001 0.001 0.001"/>
+                </geometry>
+            </visual>
+            <visual>
+                <origin xyz="0 0 -0.040825" rpy="0 0 0" />
+                <geometry>
+                    <mesh filename="package://hector_sensors_description/meshes/ouster_os0/os0.dae" scale="0.001 0.001 0.001"/>
+                </geometry>
+            </visual>
+            <collision>
+                <origin xyz="0 0 -0.000825" rpy="0 0 0" />
+                <geometry>
+                    <cylinder radius="0.04041" length="0.0735"/>
+                </geometry>
+            </collision>
+            <collision>
+                <origin xyz="0 0 -0.047825" rpy="0 0 0"/>
+                <geometry>
+                    <box size="0.11 0.11 0.0205"/>
+                </geometry>
+            </collision>
+        </link>
+        <link name="${name}_laser_frame"/>
+        <joint name="${name}_sensor_joint_laser_frame" type="fixed">
+        	<origin xyz="0 0 -0.01" rpy="0 0 ${-M_PI/2.0}" />
+            <parent link="${name}_link" />
+            <child link="${name}_laser_frame" />
+        </joint>
+    </xacro:macro>
+    <xacro:macro name="os0_128" params="name *origin *parent">
+        <xacro:os0_128_advanced_parameters name="${name}" update_rate="10" horizontal_samples="512" vertical_samples="128" min_range="0.45" max_range="100" min_angle="45" max_angle="45">
+            <xacro:insert_block name="origin"/>
+            <xacro:insert_block name="parent"/>
+        </xacro:os0_128_advanced_parameters>
+    </xacro:macro>
+    <xacro:macro name="os0_128_advanced_parameters" params="name *origin *parent update_rate horizontal_samples vertical_samples min_range max_range min_angle max_angle">
+        <xacro:os0_128_model name="${name}">
+            <xacro:insert_block name="origin"/>
+            <xacro:insert_block name="parent"/>
+        </xacro:os0_128_model>
+        <xacro:os0_128_gazebo name="${name}" update_rate="${update_rate}" horizontal_samples="${horizontal_samples}" vertical_samples="${vertical_samples}" min_range="${min_range}" max_range="${max_range}" min_angle="${min_angle}" max_angle="${max_angle}"/>
+    </xacro:macro>
 </robot>

File: urdf/tis_zoom_cam.urdf.xacro (robot description, xacro)
@@ -40,5 +40,5 @@
     </xacro:tis_zoom_camera_model>
     <xacro:generic_camera name="${name}" robot_name="${robot_name}" parent="${name}_housing_frame" ros_topic="image_raw" cam_info_topic="camera_info" update_rate="5" res_x="1920" res_y="1080" image_format="R8G8B8" hfov="70">
-      <origin xyz="0 0 0" rpy="0 0 0"/>
+      <origin xyz="0.04 0.0 0.0" rpy="0 0 0"/>
     </xacro:generic_camera>
   </xacro:macro>

Commit message: Added RGL lidar model for Livox MID-360.

File: gazebo/livox_mid360.gazebo.xacro (robot description, xacro)
@@ -1,35 +1,63 @@
 <?xml version="1.0" encoding="UTF-8"?>
 <robot xmlns:xacro="http://ros.org/wiki/xacro">
-  <xacro:macro name="livox_mid360_gazebo" params="visualize:=True name:=default">
+  <!-- When use_rgl is true the Livox Mid360 is simulated with the GPU-accelerated
+       RGL plugin (rgl::RGLServerPluginInstance), which requires the
+       rgl::RGLServerPluginManager to be loaded in the world (see base.world.xacro)
+       and a usable NVIDIA GPU at runtime. Otherwise the native gz gpu_lidar sensor
+       is used. The value is selected automatically by the launch files via
+       hector_gazebo_simulation.rgl.resolve_use_rgl; default false so the package
+       still renders standalone without the RGL plugin present. -->
+  <xacro:arg name="use_rgl" default="false"/>
+  <xacro:macro name="livox_mid360_gazebo" params="visualize:=false name:=default">
     <gazebo reference="${name}_laser_frame">
-      <sensor name="gpu_lidar_${name}" type="gpu_lidar">
-        <pose relative_to="${name}_laser_frame">0 0 0 0 0 0</pose>
-        <topic>/$(arg robot_name)/${name}</topic>
-        <update_rate>10</update_rate>
-        <gz_frame_id>${name}_laser_frame</gz_frame_id>
-        <always_on>1</always_on>
-        <visualize>${visualize}</visualize>
-        <ray>
-          <scan>
-            <horizontal>
-              <samples>100</samples>
-              <resolution>1</resolution>
-              <min_angle>${0}</min_angle>
-              <max_angle>${2*pi}</max_angle>
-            </horizontal>
-            <vertical>
-              <samples>360</samples>
-              <resolution>1</resolution>
-              <min_angle>${radians(-7.22)}</min_angle>
-              <max_angle>${radians(55.22)}</max_angle>
-            </vertical>
-          </scan>
-          <range>
-            <min>0.08</min>
-            <max>10.0</max>
-            <resolution>0.01</resolution>
-          </range>
-        </ray>
-      </sensor>
+      <xacro:if value="$(arg use_rgl)">
+        <!-- RGL publishes the cloud on the exact <topic> (gz appends nothing), so
+             the topic must carry the /points suffix the bridge expects. <frame>
+             sets the PointCloud2 header.frame_id. -->
+        <sensor name="rgl_lidar_${name}" type="custom">
+          <plugin filename="RGLServerPluginInstance" name="rgl::RGLServerPluginInstance">
+            <range>
+              <min>0.08</min>
+              <max>40.0</max>
+            </range>
+            <update_rate>10</update_rate>
+            <update_on_paused_sim>false</update_on_paused_sim>
+            <topic>/$(arg robot_name)/${name}/points</topic>
+            <frame>${name}_laser_frame</frame>
+            <pattern_preset>Livox Mid360</pattern_preset>
+          </plugin>
+        </sensor>
+      </xacro:if>
+      <xacro:unless value="$(arg use_rgl)">
+        <sensor name="gpu_lidar_${name}" type="gpu_lidar">
+          <pose relative_to="${name}_laser_frame">0 0 0 0 0 0</pose>
+          <topic>/$(arg robot_name)/${name}</topic>
+          <update_rate>10</update_rate>
+          <gz_frame_id>${name}_laser_frame</gz_frame_id>
+          <always_on>1</always_on>
+          <visualize>${visualize}</visualize>
+          <ray>
+            <scan>
+              <horizontal>
+                <samples>360</samples>
+                <resolution>1</resolution>
+                <min_angle>${0}</min_angle>
+                <max_angle>${2*pi}</max_angle>
+              </horizontal>
+              <vertical>
+                <samples>48</samples>
+                <resolution>1</resolution>
+                <min_angle>${radians(-7.22)}</min_angle>
+                <max_angle>${radians(55.22)}</max_angle>
+              </vertical>
+            </scan>
+            <range>
+              <min>0.08</min>
+              <max>40.0</max>
+              <resolution>0.01</resolution>
+            </range>
+          </ray>
+        </sensor>
+      </xacro:unless>
     </gazebo>
   </xacro:macro>

Commit message: Added RGL lidar model for Livox MID-360 gated by use_rgl argument. (#22)
* Added RGL lidar model for Livox MID-360.

File: gazebo/livox_mid360.gazebo.xacro (robot description, xacro)
@@ -1,35 +1,60 @@
 <?xml version="1.0" encoding="UTF-8"?>
 <robot xmlns:xacro="http://ros.org/wiki/xacro">
-  <xacro:macro name="livox_mid360_gazebo" params="visualize:=True name:=default">
+  <!-- When use_rgl is true the Livox Mid360 is simulated with the GPU-accelerated
+       RGL plugin (rgl::RGLServerPluginInstance), which requires the
+       rgl::RGLServerPluginManager to be loaded in the world and a usable NVIDIA
+       GPU at runtime. Otherwise the native gz gpu_lidar sensor is used. -->
+  <xacro:arg name="use_rgl" default="false"/>
+  <xacro:macro name="livox_mid360_gazebo" params="visualize:=false name:=default">
     <gazebo reference="${name}_laser_frame">
-      <sensor name="gpu_lidar_${name}" type="gpu_lidar">
-        <pose relative_to="${name}_laser_frame">0 0 0 0 0 0</pose>
-        <topic>/$(arg robot_name)/${name}</topic>
-        <update_rate>10</update_rate>
-        <gz_frame_id>${name}_laser_frame</gz_frame_id>
-        <always_on>1</always_on>
-        <visualize>${visualize}</visualize>
-        <ray>
-          <scan>
-            <horizontal>
-              <samples>100</samples>
-              <resolution>1</resolution>
-              <min_angle>${0}</min_angle>
-              <max_angle>${2*pi}</max_angle>
-            </horizontal>
-            <vertical>
-              <samples>360</samples>
-              <resolution>1</resolution>
-              <min_angle>${radians(-7.22)}</min_angle>
-              <max_angle>${radians(55.22)}</max_angle>
-            </vertical>
-          </scan>
-          <range>
-            <min>0.08</min>
-            <max>10.0</max>
-            <resolution>0.01</resolution>
-          </range>
-        </ray>
-      </sensor>
+      <xacro:if value="$(arg use_rgl)">
+        <!-- RGL publishes the cloud on the exact <topic> (gz appends nothing), so
+             the topic must carry the /points suffix the bridge expects. <frame>
+             sets the PointCloud2 header.frame_id. -->
+        <sensor name="rgl_lidar_${name}" type="custom">
+          <plugin filename="RGLServerPluginInstance" name="rgl::RGLServerPluginInstance">
+            <range>
+              <min>0.08</min>
+              <max>40.0</max>
+            </range>
+            <update_rate>10</update_rate>
+            <update_on_paused_sim>false</update_on_paused_sim>
+            <topic>/$(arg robot_name)/${name}/points</topic>
+            <frame>${name}_laser_frame</frame>
+            <pattern_preset>Livox Mid360</pattern_preset>
+          </plugin>
+        </sensor>
+      </xacro:if>
+      <xacro:unless value="$(arg use_rgl)">
+        <sensor name="gpu_lidar_${name}" type="gpu_lidar">
+          <pose relative_to="${name}_laser_frame">0 0 0 0 0 0</pose>
+          <topic>/$(arg robot_name)/${name}</topic>
+          <update_rate>10</update_rate>
+          <gz_frame_id>${name}_laser_frame</gz_frame_id>
+          <always_on>1</always_on>
+          <visualize>${visualize}</visualize>
+          <ray>
+            <scan>
+              <horizontal>
+                <samples>360</samples>
+                <resolution>1</resolution>
+                <min_angle>${0}</min_angle>
+                <max_angle>${2*pi}</max_angle>
+              </horizontal>
+              <vertical>
+                <samples>48</samples>
+                <resolution>1</resolution>
+                <min_angle>${radians(-7.22)}</min_angle>
+                <max_angle>${radians(55.22)}</max_angle>
+              </vertical>
+            </scan>
+            <range>
+              <min>0.08</min>
+              <max>40.0</max>
+              <resolution>0.01</resolution>
+            </range>
+          </ray>
+        </sensor>
+      </xacro:unless>
     </gazebo>
   </xacro:macro>
